File: Recovery PCB/Relay.sch (KiCad schematic (older format))
At the start: 13 parts, among them J2 Screw_Terminal_01x03, J3 Screw_Terminal_01x03, K1 SANYOU_SRD_Form_C, K2 SANYOU_SRD_Form_C, Q1 BC547, Q2 BC547, U4 LTV-827S

Commit message: Updated recovery board with new connections.
Parts:
- removed D1, D2: D, Diode_SMD:D_SMA_Handsoldering, symbol Device:D
- removed J2, J3: Screw_Terminal_01x03, TerminalBlock:TerminalBlock_bornier-3_P5.08mm, symbol Connector:Screw_Terminal_01x03
- removed K1, K2: SANYOU_SRD_Form_C, Relay_THT:Relay_SPDT_SANYOU_SRD_Series_Form_C, symbol Relay:SANYOU_SRD_Form_C
- removed Q1, Q2: BC547, Package_TO_SOT_THT:TO-92_Inline, symbol Transistor_BJT:BC547
- removed R10, R8: 1k, Resistor_SMD:R_0603_1608Metric, symbol Device:R_US
- removed R7, R9: 510, Resistor_SMD:R_0603_1608Metric, symbol Device:R_US
- removed U4: LTV-827S, Package_DIP:SMDIP-8_W9.53mm, symbol Isolator:LTV-827S
- added K?: SANYOU_SRD_Form_C, Relay_THT:Relay_SPDT_SANYOU_SRD_Series_Form_C, symbol Relay:SANYOU_SRD_Form_C
- added Q?: BSS138, Package_TO_SOT_SMD:SOT-23, symbol Transistor_FET:BSS138
- added R?: R_US, symbol Device:R_US
- added U?: LTV-827S, Package_DIP:SMDIP-8_W9.53mm, symbol Isolator:LTV-827S
Connections:
- wire segments 44 -> 10

Commit message: Update relays on recovery board.
Parts:
- removed Q?: BSS138, Package_TO_SOT_SMD:SOT-23, symbol Transistor_FET:BSS138
- removed R?: R_US, symbol Device:R_US
- removed U?: LTV-827S, Package_DIP:SMDIP-8_W9.53mm, symbol Isolator:LTV-827S
- added D? (x2): D, symbol Device:D
- added J? (x2): Screw_Terminal_01x03, symbol Connector:Screw_Terminal_01x03
- added K?: SANYOU_SRD_Form_C, Relay_THT:Relay_SPDT_SANYOU_SRD_Series_Form_C, symbol Relay:SANYOU_SRD_Form_C
- added R? (x2): R_US, symbol Device:R_US
- added U? (x2): LTV-847, Package_DIP:DIP-16_W7.62mm, symbol Isolator:LTV-847
Connections:
- wire segments 10 -> 38

Commit message: Update relays and re-annotate entire schematic. Review needed before layout.
Parts:
- added D1, D2: LED, symbol Device:LED
- gave numbers to parts that had none: 9
Connections:
- wire segments 38 -> 40
Changed lines of the file:
@@
 	4900 2300 4900 2050
 $Comp
-L power:+5V #PWR?
+L power:+5V #PWR027
 U 1 1 5E643112
 P 4900 2050
-F 0 "#PWR?" H 4900 1900 50  0001 C CNN
+F 0 "#PWR027" H 4900 1900 50  0001 C CNN
 F 1 "+5V" H 4915 2223 50  0000 C CNN
 F 2 "" H 4900 2050 50  0001 C CNN
@@
 Wire Wire Line
 	4100 2500 4000 2500
-Wire Wire Line
-	4000 2500 4000 2700
-$Comp
-L power:GND #PWR?
+$Comp
+L power:GND #PWR023
 U 1 1 5E651774
-P 4000 2700
-F 0 "#PWR?" H 4000 2450 50  0001 C CNN
-F 1 "GND" H 4005 2527 50  0000 C CNN
-F 2 "" H 4000 2700 50  0001 C CNN
-F 3 "" H 4000 2700 50  0001 C CNN
-	1    4000 2700
-	1    0    0    -1
-$EndComp
-$Comp
-L Relay:SANYOU_SRD_Form_C K?
+P 4000 3050
+F 0 "#PWR023" H 4000 2800 50  0001 C CNN
+F 1 "GND" H 4005 2877 50  0000 C CNN
+F 2 "" H 4000 3050 50  0001 C CNN
+F 3 "" H 4000 3050 50  0001 C CNN
+	1    4000 3050
+	1    0    0    -1
+$EndComp
+$Comp
+L Relay:SANYOU_SRD_Form_C K1
 U 1 1 5E651D90
 P 5650 2800
-F 0 "K?" H 6080 2846 50  0000 L CNN
+F 0 "K1" H 6080 2846 50  0000 L CNN
 F 1 "SANYOU_SRD_Form_C" H 6080 2755 50  0000 L CNN
 F 2 "Relay_THT:Relay_SPDT_SANYOU_SRD_Series_Form_C" H 6100 2750 50  0001 L CNN
@@
 	4700 3100 4850 3100
 $Comp
-L Device:D D?
+L Device:D D3
 U 1 1 5E58FAD9
 P 4700 2800
-F 0 "D?" V 4654 2879 50  0000 L CNN
+F 0 "D3" V 4654 2879 50  0000 L CNN
 F 1 "D" V 4745 2879 50  0000 L CNN
 F 2 "" H 4700 2800 50  0001 C CNN
@@
 	4700 2950 4700 3100
 $Comp
-L power:GND #PWR?
+L power:GND #PWR025
 U 1 1 5E5906D6
 P 4700 3100
-F 0 "#PWR?" H 4700 2850 50  0001 C CNN
+F 0 "#PWR025" H 4700 2850 50  0001 C CNN
 F 1 "GND" H 4705 2927 50  0000 C CNN
 F 2 "" H 4700 3100 50  0001 C CNN
@@
 Connection ~ 4700 3100
 $Comp
-L Device:R_US R?
+L Device:R_US R7
 U 1 1 5E590CAC
 P 5000 3100
-F 0 "R?" V 4795 3100 50  0000 C CNN
+F 0 "R7" V 4795 3100 50  0000 C CNN
 F 1 "R_US" V 4886 3100 50  0000 C CNN
 F 2 "" V 5040 3090 50  0001 C CNN
@@
 	5150 3100 5450 3100
 $Comp
-L Connector:Screw_Terminal_01x03 J?
+L Connector:Screw_Terminal_01x03 J3
 U 1 1 5E59311B
 P 7250 2800
-F 0 "J?" H 7330 2842 50  0000 L CNN
+F 0 "J3" H 7330 2842 50  0000 L CNN
 F 1 "Screw_Terminal_01x03" H 7330 2751 50  0000 L CNN
 F 2 "" H 7250 2800 50  0001 C CNN
@@
 	4900 4050 4900 3800
 $Comp
-L power:+5V #PWR?
+L power:+5V #PWR028
 U 1 1 5E5A3DD8
 P 4900 3800
-F 0 "#PWR?" H 4900 3650 50  0001 C CNN
+F 0 "#PWR028" H 4900 3650 50  0001 C CNN
 F 1 "+5V" H 4915 3973 50  0000 C CNN
 F 2 "" H 4900 3800 50  0001 C CNN
@@
 	1    0    0    -1
 $EndComp
-Wire Wire Line
-	4100 4250 4000 4250
-$Comp
-L power:GND #PWR?
-U 1 1 5E5A3DDF
-P 4000 4450
-F 0 "#PWR?" H 4000 4200 50  0001 C CNN
-F 1 "GND" H 4005 4277 50  0000 C CNN
-F 2 "" H 4000 4450 50  0001 C CNN
-F 3 "" H 4000 4450 50  0001 C CNN
-	1    4000 4450
-	1    0    0    -1
-$EndComp
-$Comp
-L Relay:SANYOU_SRD_Form_C K?
+$Comp
+L Relay:SANYOU_SRD_Form_C K2
 U 1 1 5E5A3DE5
 P 5650 4550
-F 0 "K?" H 6080 4596 50  0000 L CNN
+F 0 "K2" H 6080 4596 50  0000 L CNN
 F 1 "SANYOU_SRD_Form_C" H 6080 4505 50  0000 L CNN
 F 2 "Relay_THT:Relay_SPDT_SANYOU_SRD_Series_Form_C" H 6100 4500 50  0001 L CNN
@@
 	4700 4850 4850 4850
 $Comp
-L Device:D D?
+L Device:D D4
 U 1 1 5E5A3DEE
 P 4700 4550
-F 0 "D?" V 4654 4629 50  0000 L CNN
+F 0 "D4" V 4654 4629 50  0000 L CNN
 F 1 "D" V 4745 4629 50  0000 L CNN
 F 2 "" H 4700 4550 50  0001 C CNN
@@
 	4700 4700 4700 4850
 $Comp
-L power:GND #PWR?
+L power:GND #PWR026
 U 1 1 5E5A3DF5
 P 4700 4850
-F 0 "#PWR?" H 4700 4600 50  0001 C CNN
+F 0 "#PWR026" H 4700 4600 50  0001 C CNN
 F 1 "GND" H 4705 4677 50  0000 C CNN
 F 2 "" H 4700 4850 50  0001 C CNN
@@
 Connection ~ 4700 4850
 $Comp
-L Device:R_US R?
+L Device:R_US R8
 U 1 1 5E5A3DFC
 P 5000 4850
-F 0 "R?" V 4795 4850 50  0000 C CNN
+F 0 "R8" V 4795 4850 50  0000 C CNN
 F 1 "R_US" V 4886 4850 50  0000 C CNN
 F 2 "" V 5040 4840 50  0001 C CNN
@@
 	5150 4850 5450 4850
 $Comp
-L Connector:Screw_Terminal_01x03 J?
+L Connector:Screw_Terminal_01x03 J4
 U 1 1 5E5A3E04
 P 7250 4550
-F 0 "J?" H 7330 4592 50  0000 L CNN
+F 0 "J4" H 7330 4592 50  0000 L CNN
 F 1 "Screw_Terminal_01x03" H 7330 4501 50  0000 L CNN
 F 2 "" H 7250 4550 50  0001 C CNN
@@
 Wire Wire Line
 	7000 4550 7050 4550
-Wire Wire Line
-	4000 4250 4000 4450
-$Comp
-L Isolator:LTV-847 U?
+$Comp
+L Isolator:LTV-847 U4
 U 1 1 5E5A5FB7
 P 4400 2400
-F 0 "U?" H 4400 2725 50  0000 C CNN
+F 0 "U4" H 4400 2725 50  0000 C CNN
 F 1 "LTV-847" H 4400 2634 50  0000 C CNN
 F 2 "Package_DIP:DIP-16_W7.62mm" H 4200 2200 50  0001 L CIN
@@
 Connection ~ 4700 2500
 $Comp
-L Isolator:LTV-847 U?
+L Isolator:LTV-847 U4
 U 2 1 5E5A7800
 P 4400 4150
-F 0 "U?" H 4400 4475 50  0000 C CNN
+F 0 "U4" H 4400 4475 50  0000 C CNN
 F 1 "LTV-847" H 4400 4384 50  0000 C CNN
 F 2 "Package_DIP:DIP-16_W7.62mm" H 4200 3950 50  0001 L CIN
@@
 $EndComp
 Connection ~ 4700 4250
+$Comp
+L Device:LED D1
+U 1 1 5E58CA13
+P 4000 2750
+F 0 "D1" V 4039 2633 50  0000 R CNN
+F 1 "LED" V 3948 2633 50  0000 R CNN
+F 2 "" H 4000 2750 50  0001 C CNN
+F 3 "~" H 4000 2750 50  0001 C CNN
+	1    4000 2750
+	0    -1   -1   0
+$EndComp
+Wire Wire Line
+	4000 2500 4000 2600
+Wire Wire Line
+	4000 2900 4000 3050
+Wire Wire Line
+	4100 4250 4000 4250
+$Comp
+L power:GND #PWR024
+U 1 1 5E592CAD
+P 4000 4800
+F 0 "#PWR024" H 4000 4550 50  0001 C CNN
+F 1 "GND" H 4005 4627 50  0000 C CNN
+F 2 "" H 4000 4800 50  0001 C CNN
+F 3 "" H 4000 4800 50  0001 C CNN
+	1    4000 4800
+	1    0    0    -1
+$EndComp
+$Comp
+L Device:LED D2
+U 1 1 5E592CB3
+P 4000 4500
+F 0 "D2" V 4039 4383 50  0000 R CNN
+F 1 "LED" V 3948 4383 50  0000 R CNN
+F 2 "" H 4000 4500 50  0001 C CNN
+F 3 "~" H 4000 4500 50  0001 C CNN
+	1    4000 4500
+	0    -1   -1   0
+$EndComp
+Wire Wire Line
+	4000 4250 4000 4350
+Wire Wire Line
+	4000 4650 4000 4800
 $EndSCHEMATC

Commit message: Added footprints.
Added footprints for various parts. Still need to update some more and calculate some values.
Parts:
- removed J3, J4: Screw_Terminal_01x03, symbol Connector:Screw_Terminal_01x03
- removed U4: LTV-847, Package_DIP:DIP-16_W7.62mm, symbol Isolator:LTV-847
- added J3, J4: Screw_Terminal_01x02, symbol Connector:Screw_Terminal_01x02
- added R10: R_US, symbol Device:R_US
- added R7: 220, symbol Device:R_US
- added U4: TLP291-4(TP,E), Parts:SOIC127P700X229-16N, symbol TLP291-4_TP_E_:TLP291-4(TP,E)
- R8: value R_US -> 220
- renumbered R7 to R9
Connections:
- net labels added: +9V
- net labels removed: +5V, IN2
- wire segments 40 -> 28
- no-connect marks 0 -> 2
Other:
- note added: "I am calculating this resistor value. Please hold."

Commit message: Updated some footprints and re-annotated schematic.
Parts:
- D2: renamed from D1; footprint (none) -> LED_SMD:LED_0603_1608Metric
- D3: renamed from D2; footprint (none) -> LED_SMD:LED_0603_1608Metric
- D4: renamed from D3; footprint (none) -> Diode_SMD:D_0603_1608Metric
- D5: renamed from D4; footprint (none) -> Diode_SMD:D_0603_1608Metric
- J4: renamed from J3; footprint (none) -> TerminalBlock:TerminalBlock_bornier-2_P5.08mm
- J5: renamed from J4; footprint (none) -> TerminalBlock:TerminalBlock_bornier-2_P5.08mm
- R10: renamed from R9; footprint (none) -> Resistor_SMD:R_0603_1608Metric
- R11: renamed from R10; footprint (none) -> Resistor_SMD:R_0603_1608Metric
- R8: renamed from R7; footprint (none) -> Resistor_SMD:R_0603_1608Metric
- R9: renamed from R8; footprint (none) -> Resistor_SMD:R_0603_1608Metric
Changed lines of the file:
@@
 EESchema Schematic File Version 4
-LIBS:Recovery PCB-cache
-EELAYER 26 0
+EELAYER 30 0
 EELAYER END
 $Descr A4 11693 8268
@@
 	4900 2300 4900 2050
 $Comp
-L power:GND #PWR025
+L power:GND #PWR034
 U 1 1 5E651774
 P 4700 3100
-F 0 "#PWR025" H 4700 2850 50  0001 C CNN
+F 0 "#PWR034" H 4700 2850 50  0001 C CNN
 F 1 "GND" H 4705 2927 50  0000 C CNN
 F 2 "" H 4700 3100 50  0001 C CNN
@@
 	5050 3100 5200 3100
 $Comp
-L Device:D D3
+L Device:D D4
 U 1 1 5E58FAD9
 P 5050 2800
-F 0 "D3" V 5004 2879 50  0000 L CNN
+F 0 "D4" V 5004 2879 50  0000 L CNN
 F 1 "D" V 5095 2879 50  0000 L CNN
-F 2 "" H 5050 2800 50  0001 C CNN
+F 2 "Diode_SMD:D_0603_1608Metric" H 5050 2800 50  0001 C CNN
 F 3 "~" H 5050 2800 50  0001 C CNN
 	1    5050 2800
@@
 	5050 2950 5050 3100
 $Comp
-L power:GND #PWR029
+L power:GND #PWR038
 U 1 1 5E5906D6
 P 5050 3100
-F 0 "#PWR029" H 5050 2850 50  0001 C CNN
+F 0 "#PWR038" H 5050 2850 50  0001 C CNN
 F 1 "GND" H 5055 2927 50  0000 C CNN
 F 2 "" H 5050 3100 50  0001 C CNN
@@
 	5500 3100 5800 3100
 $Comp
-L Device:LED D1
+L Device:LED D2
 U 1 1 5E58CA13
 P 4700 2950
-F 0 "D1" V 4739 2833 50  0000 R CNN
+F 0 "D2" V 4739 2833 50  0000 R CNN
 F 1 "LED" V 4648 2833 50  0000 R CNN
-F 2 "" H 4700 2950 50  0001 C CNN
+F 2 "LED_SMD:LED_0603_1608Metric" H 4700 2950 50  0001 C CNN
 F 3 "~" H 4700 2950 50  0001 C CNN
 	1    4700 2950
@@
 $EndComp
 $Comp
-L Device:R_US R9
+L Device:R_US R10
 U 1 1 5E590CAC
 P 5350 3100
-F 0 "R9" V 5145 3100 50  0000 C CNN
+F 0 "R10" V 5145 3100 50  0000 C CNN
 F 1 "R_US" V 5236 3100 50  0000 C CNN
-F 2 "" V 5390 3090 50  0001 C CNN
+F 2 "Resistor_SMD:R_0603_1608Metric" V 5390 3090 50  0001 C CNN
 F 3 "~" H 5350 3100 50  0001 C CNN
 	1    5350 3100
@@
 	5050 2500 5050 2650
 $Comp
-L Device:R_US R7
+L Device:R_US R8
 U 1 1 5E65853B
 P 4700 2650
-F 0 "R7" H 4768 2696 50  0000 L CNN
+F 0 "R8" H 4768 2696 50  0000 L CNN
 F 1 "220" H 4768 2605 50  0000 L CNN
-F 2 "" V 4740 2640 50  0001 C CNN
+F 2 "Resistor_SMD:R_0603_1608Metric" V 4740 2640 50  0001 C CNN
 F 3 "~" H 4700 2650 50  0001 C CNN
 	1    4700 2650
@@
 	4900 3950 4900 3700
 $Comp
-L power:GND #PWR026
+L power:GND #PWR035
 U 1 1 5E662729
 P 4700 4750
-F 0 "#PWR026" H 4700 4500 50  0001 C CNN
+F 0 "#PWR035" H 4700 4500 50  0001 C CNN
 F 1 "GND" H 4705 4577 50  0000 C CNN
 F 2 "" H 4700 4750 50  0001 C CNN
@@
 	5050 4750 5200 4750
 $Comp
-L Device:D D4
+L Device:D D5
 U 1 1 5E662736
 P 5050 4450
-F 0 "D4" V 5004 4529 50  0000 L CNN
+F 0 "D5" V 5004 4529 50  0000 L CNN
 F 1 "D" V 5095 4529 50  0000 L CNN
-F 2 "" H 5050 4450 50  0001 C CNN
+F 2 "Diode_SMD:D_0603_1608Metric" H 5050 4450 50  0001 C CNN
 F 3 "~" H 5050 4450 50  0001 C CNN
 	1    5050 4450
@@
 	5050 4600 5050 4750
 $Comp
-L power:GND #PWR030
+L power:GND #PWR039
 U 1 1 5E66273D
 P 5050 4750
-F 0 "#PWR030" H 5050 4500 50  0001 C CNN
+F 0 "#PWR039" H 5050 4500 50  0001 C CNN
 F 1 "GND" H 5055 4577 50  0000 C CNN
 F 2 "" H 5050 4750 50  0001 C CNN
@@
 	5500 4750 5800 4750
 $Comp
-L Device:LED D2
+L Device:LED D3
 U 1 1 5E662754
 P 4700 4600
-F 0 "D2" V 4739 4483 50  0000 R CNN
+F 0 "D3" V 4739 4483 50  0000 R CNN
 F 1 "LED" V 4648 4483 50  0000 R CNN
-F 2 "" H 4700 4600 50  0001 C CNN
+F 2 "LED_SMD:LED_0603_1608Metric" H 4700 4600 50  0001 C CNN
 F 3 "~" H 4700 4600 50  0001 C CNN
 	1    4700 4600
@@
 $EndComp
 $Comp
-L Device:R_US R10
+L Device:R_US R11
 U 1 1 5E66275A
 P 5350 4750
-F 0 "R10" V 5145 4750 50  0000 C CNN
+F 0 "R11" V 5145 4750 50  0000 C CNN
 F 1 "R_US" V 5236 4750 50  0000 C CNN
-F 2 "" V 5390 4740 50  0001 C CNN
+F 2 "Resistor_SMD:R_0603_1608Metric" V 5390 4740 50  0001 C CNN
 F 3 "~" H 5350 4750 50  0001 C CNN
 	1    5350 4750
@@
 	5050 4150 5050 4300
 $Comp
-L Device:R_US R8
+L Device:R_US R9
 U 1 1 5E662768
 P 4700 4300
-F 0 "R8" H 4768 4346 50  0000 L CNN
+F 0 "R9" H 4768 4346 50  0000 L CNN
 F 1 "220" H 4768 4255 50  0000 L CNN
-F 2 "" V 4740 4290 50  0001 C CNN
+F 2 "Resistor_SMD:R_0603_1608Metric" V 4740 4290 50  0001 C CNN
 F 3 "~" H 4700 4300 50  0001 C CNN
 	1    4700 4300
@@
 	4000 4150 4000 4200
 $Comp
-L power:GND #PWR024
+L power:GND #PWR033
 U 1 1 5E67CE4B
 P 4000 4200
-F 0 "#PWR024" H 4000 3950 50  0001 C CNN
+F 0 "#PWR033" H 4000 3950 50  0001 C CNN
 F 1 "GND" H 4005 4027 50  0000 C CNN
 F 2 "" H 4000 4200 50  0001 C CNN
@@
 $EndComp
 $Comp
-L power:GND #PWR023
+L power:GND #PWR032
 U 1 1 5E67DABF
 P 4000 2600
-F 0 "#PWR023" H 4000 2350 50  0001 C CNN
+F 0 "#PWR032" H 4000 2350 50  0001 C CNN
 F 1 "GND" H 4005 2427 50  0000 C CNN
 F 2 "" H 4000 2600 50  0001 C CNN
@@
 Connection ~ 4700 4150
 $Comp
-L power:+9V #PWR027
+L power:+9V #PWR036
 U 1 1 5E699433
 P 4900 2050
-F 0 "#PWR027" H 4900 1900 50  0001 C CNN
+F 0 "#PWR036" H 4900 1900 50  0001 C CNN
 F 1 "+9V" H 4915 2223 50  0000 C CNN
 F 2 "" H 4900 2050 50  0001 C CNN
@@
 $EndComp
 $Comp
-L power:+9V #PWR028
+L power:+9V #PWR037
 U 1 1 5E6998CD
 P 4900 3700
-F 0 "#PWR028" H 4900 3550 50  0001 C CNN
+F 0 "#PWR037" H 4900 3550 50  0001 C CNN
 F 1 "+9V" H 4915 3873 50  0000 C CNN
 F 2 "" H 4900 3700 50  0001 C CNN
@@
 NoConn ~ 6100 2500
 $Comp
-L power:+9V #PWR031
+L power:+9V #PWR040
 U 1 1 5E69B629
 P 6300 2500
-F 0 "#PWR031" H 6300 2350 50  0001 C CNN
+F 0 "#PWR040" H 6300 2350 50  0001 C CNN
 F 1 "+9V" H 6315 2673 50  0000 C CNN
 F 2 "" H 6300 2500 50  0001 C CNN
@@
 $EndComp
 $Comp
-L Connector:Screw_Terminal_01x02 J3
+L Connector:Screw_Terminal_01x02 J4
 U 1 1 5E69C0D8
 P 7700 2750
-F 0 "J3" H 7780 2742 50  0000 L CNN
+F 0 "J4" H 7780 2742 50  0000 L CNN
 F 1 "Screw_Terminal_01x02" H 7780 2651 50  0000 L CNN
-F 2 "" H 7700 2750 50  0001 C CNN
+F 2 "TerminalBlock:TerminalBlock_bornier-2_P5.08mm" H 7700 2750 50  0001 C CNN
 F 3 "~" H 7700 2750 50  0001 C CNN
 	1    7700 2750
@@
 $EndComp
 $Comp
-L power:GND #PWR033
+L power:GND #PWR042
 U 1 1 5E6A105C
 P 7500 2850
-F 0 "#PWR033" H 7500 2600 50  0001 C CNN
+F 0 "#PWR042" H 7500 2600 50  0001 C CNN
 F 1 "GND" H 7505 2677 50  0000 C CNN
 F 2 "" H 7500 2850 50  0001 C CNN
@@
 NoConn ~ 6100 4150
 $Comp
-L power:+9V #PWR032
+L power:+9V #PWR041
 U 1 1 5E6A3657
 P 6300 4150
-F 0 "#PWR032" H 6300 4000 50  0001 C CNN
+F 0 "#PWR041" H 6300 4000 50  0001 C CNN
 F 1 "+9V" H 6315 4323 50  0000 C CNN
 F 2 "" H 6300 4150 50  0001 C CNN
@@
 $EndComp
 $Comp
-L Connector:Screw_Terminal_01x02 J4
+L Connector:Screw_Terminal_01x02 J5
 U 1 1 5E6A427F
 P 7700 4400
-F 0 "J4" H 7780 4392 50  0000 L CNN
+F 0 "J5" H 7780 4392 50  0000 L CNN
 F 1 "Screw_Terminal_01x02" H 7780 4301 50  0000 L CNN
-F 2 "" H 7700 4400 50  0001 C CNN
+F 2 "TerminalBlock:TerminalBlock_bornier-2_P5.08mm" H 7700 4400 50  0001 C CNN
 F 3 "~" H 7700 4400 50  0001 C CNN
 	1    7700 4400
@@
 $EndComp
 $Comp
-L power:GND #PWR034
+L power:GND #PWR043
 U 1 1 5E6A4285
 P 7500 4500
-F 0 "#PWR034" H 7500 4250 50  0001 C CNN
+F 0 "#PWR043" H 7500 4250 50  0001 C CNN
 F 1 "GND" H 7505 4327 50  0000 C CNN
 F 2 "" H 7500 4500 50  0001 C CNN

Commit message: Added missing footprints and replaced GPS module.
Parts:
- D4, D5: footprint Diode_SMD:D_0603_1608Metric -> Diode_SMD:D_SMB
- R10, R11: value R_US -> 300
- renumbered U4 to U5
Changed lines of the file:
@@
 F 0 "D4" V 5004 2879 50  0000 L CNN
 F 1 "D" V 5095 2879 50  0000 L CNN
-F 2 "Diode_SMD:D_0603_1608Metric" H 5050 2800 50  0001 C CNN
+F 2 "Diode_SMD:D_SMB" H 5050 2800 50  0001 C CNN
 F 3 "~" H 5050 2800 50  0001 C CNN
 	1    5050 2800
@@
 P 5350 3100
 F 0 "R10" V 5145 3100 50  0000 C CNN
-F 1 "R_US" V 5236 3100 50  0000 C CNN
+F 1 "300" V 5236 3100 50  0000 C CNN
 F 2 "Resistor_SMD:R_0603_1608Metric" V 5390 3090 50  0001 C CNN
 F 3 "~" H 5350 3100 50  0001 C CNN
@@
 Connection ~ 5050 3100
 $Comp
-L TLP291-4_TP_E_:TLP291-4(TP,E) U4
+L TLP291-4_TP_E_:TLP291-4(TP,E) U5
 U 1 1 5E646F0C
 P 4400 2400
-F 0 "U4" H 4400 2765 50  0000 C CNN
+F 0 "U5" H 4400 2765 50  0000 C CNN
 F 1 "TLP291-4(TP,E)" H 4400 2674 50  0000 C CNN
 F 2 "Parts:SOIC127P700X229-16N" H 3900 2000 50  0001 L BNN
@@
 F 0 "D5" V 5004 4529 50  0000 L CNN
 F 1 "D" V 5095 4529 50  0000 L CNN
-F 2 "Diode_SMD:D_0603_1608Metric" H 5050 4450 50  0001 C CNN
+F 2 "Diode_SMD:D_SMB" H 5050 4450 50  0001 C CNN
 F 3 "~" H 5050 4450 50  0001 C CNN
 	1    5050 4450
@@
 P 5350 4750
 F 0 "R11" V 5145 4750 50  0000 C CNN
-F 1 "R_US" V 5236 4750 50  0000 C CNN
+F 1 "300" V 5236 4750 50  0000 C CNN
 F 2 "Resistor_SMD:R_0603_1608Metric" V 5390 4740 50  0001 C CNN
 F 3 "~" H 5350 4750 50  0001 C CNN
@@
 $EndComp
 $Comp
-L TLP291-4_TP_E_:TLP291-4(TP,E) U4
+L TLP291-4_TP_E_:TLP291-4(TP,E) U5
 U 2 1 5E67ED73
 P 4400 4050
-F 0 "U4" H 4400 4415 50  0000 C CNN
+F 0 "U5" H 4400 4415 50  0000 C CNN
 F 1 "TLP291-4(TP,E)" H 4400 4324 50  0000 C CNN
 F 2 "Parts:SOIC127P700X229-16N" H 3900 3650 50  0001 L BNN

Commit message: Finished Revision 1 of the Recovery PCB.
Parts:
- D4, D5: footprint Diode_SMD:D_SMB -> Diode_SMD:D_SOT-23_ANK
Connections:
- net labels added: IN2
Changed lines of the file:
@@
 Wire Wire Line
 	5050 3100 5200 3100
-$Comp
-L Device:D D4
-U 1 1 5E58FAD9
-P 5050 2800
-F 0 "D4" V 5004 2879 50  0000 L CNN
-F 1 "D" V 5095 2879 50  0000 L CNN
-F 2 "Diode_SMD:D_SMB" H 5050 2800 50  0001 C CNN
-F 3 "~" H 5050 2800 50  0001 C CNN
-	1    5050 2800
-	0    1    1    0
-$EndComp
 Wire Wire Line
 	5050 2950 5050 3100
@@
 	1    0    0    -1
 $EndComp
-Wire Wire Line
-	5050 2500 5800 2500
 Wire Wire Line
 	5500 3100 5800 3100
@@
 	1    0    0    -1
 $EndComp
-Wire Wire Line
-	5050 2500 5050 2650
 $Comp
 L Device:R_US R8
@@
 	1    0    0    -1
 $EndComp
-Wire Wire Line
-	4700 2500 5050 2500
 Connection ~ 4700 2500
-Connection ~ 5050 2500
 Text HLabel 4000 3950 0    50   Input ~ 0
-IN1
+IN2
 Wire Wire Line
 	4000 3950 4100 3950
@@
 Wire Wire Line
 	5050 4750 5200 4750
-$Comp
-L Device:D D5
-U 1 1 5E662736
-P 5050 4450
-F 0 "D5" V 5004 4529 50  0000 L CNN
-F 1 "D" V 5095 4529 50  0000 L CNN
-F 2 "Diode_SMD:D_SMB" H 5050 4450 50  0001 C CNN
-F 3 "~" H 5050 4450 50  0001 C CNN
-	1    5050 4450
-	0    1    1    0
-$EndComp
 Wire Wire Line
 	5050 4600 5050 4750
@@
 	1    0    0    -1
 $EndComp
-Wire Wire Line
-	5050 4150 5800 4150
 Wire Wire Line
 	5500 4750 5800 4750
@@
 $EndComp
 Connection ~ 5050 4750
-Wire Wire Line
-	5050 4150 5050 4300
 $Comp
 L Device:R_US R9
@@
 $EndComp
 Wire Wire Line
-	4700 4150 5050 4150
-Connection ~ 5050 4150
-Wire Wire Line
 	4100 2500 4000 2500
 Wire Wire Line
@@
 Text Notes 5250 4950 0    50   ~ 0
 I am calculating this resistor value. Please hold.
+Wire Wire Line
+	4700 4150 5050 4150
+Wire Wire Line
+	5050 4150 5800 4150
+Connection ~ 5050 4150
+Wire Wire Line
+	5050 4150 5050 4300
+$Comp
+L Device:D D5
+U 1 1 5E662736
+P 5050 4450
+F 0 "D5" V 5004 4529 50  0000 L CNN
+F 1 "D" V 5095 4529 50  0000 L CNN
+F 2 "Diode_SMD:D_SOT-23_ANK" H 5050 4450 50  0001 C CNN
+F 3 "~" H 5050 4450 50  0001 C CNN
+	1    5050 4450
+	0    1    1    0
+$EndComp
+Wire Wire Line
+	4700 2500 5050 2500
+Wire Wire Line
+	5050 2500 5800 2500
+Connection ~ 5050 2500
+Wire Wire Line
+	5050 2500 5050 2650
+$Comp
+L Device:D D4
+U 1 1 5E58FAD9
+P 5050 2800
+F 0 "D4" V 5004 2879 50  0000 L CNN
+F 1 "D" V 5095 2879 50  0000 L CNN
+F 2 "Diode_SMD:D_SOT-23_ANK" H 5050 2800 50  0001 C CNN
+F 3 "~" H 5050 2800 50  0001 C CNN
+	1    5050 2800
+	0    1    1    0
+$EndComp
 $EndSCHEMATC
