File: Recovery PCB/Relay.sch (KiCad schematic (older format))
At the start: 13 parts, among them J4 Screw_Terminal_01x02, J5 Screw_Terminal_01x02, K1 SANYOU_SRD_Form_C, K2 SANYOU_SRD_Form_C, U5 TLP291-4(TP,E)

Commit message: Finished Rev 2 of the Recovery PCB. Optimized trace lengths and relays.
Parts:
- removed U5: TLP291-4(TP,E), Parts:SOIC127P700X229-16N, symbol TLP291-4_TP_E_:TLP291-4(TP,E)
- added J10: Conn_01x02_Male, Connector_JST:JST_XH_B2B-XH-A_1x02_P2.50mm_Vertical, symbol Connector:Conn_01x02_Male
- added Q2, Q3: BSS138, Package_TO_SOT_SMD:SOT-23, symbol Transistor_FET:BSS138
- added R1, R22: 1M, Resistor_SMD:R_0603_1608Metric, symbol Device:R_US
Connections:
- net labels added: +3.3V, GNDPWR
- wire segments 28 -> 40
- no-connect marks 2 -> 0

Commit message: Recovery PCB: Redraw schematics
Redrew Recover PCB schematics to be more easily readable and fixed board
outline, adding netclasses to ease trace placement.
Parts:
- J10: value Conn_01x02_Male -> 9V_INPUT
Connections:
- wire segments 40 -> 34
Other:
- note removed: "I am calculating this resistor value. Please hold."
Changed lines of the file:
@@
 Comment4 ""
 $EndDescr
-Text HLabel 4000 3350 0    50   Input ~ 0
+Text HLabel 4250 3350 0    50   Input ~ 0
 IN1
 $Comp
@@
 	1    0    0    -1
 $EndComp
-Text HLabel 4000 5000 0    50   Input ~ 0
+Text HLabel 4250 5000 0    50   Input ~ 0
 IN2
 $Comp
@@
 L Connector:Screw_Terminal_01x02 J4
 U 1 1 5E69C0D8
-P 7700 2750
-F 0 "J4" H 7780 2742 50  0000 L CNN
-F 1 "Screw_Terminal_01x02" H 7780 2651 50  0000 L CNN
-F 2 "TerminalBlock:TerminalBlock_bornier-2_P5.08mm" H 7700 2750 50  0001 C CNN
-F 3 "~" H 7700 2750 50  0001 C CNN
-	1    7700 2750
+P 6750 3100
+F 0 "J4" H 6830 3092 50  0000 L CNN
+F 1 "Screw_Terminal_01x02" H 6830 3001 50  0000 L CNN
+F 2 "TerminalBlock:TerminalBlock_bornier-2_P5.08mm" H 6750 3100 50  0001 C CNN
+F 3 "~" H 6750 3100 50  0001 C CNN
+	1    6750 3100
 	1    0    0    -1
 $EndComp
@@
 L Connector:Screw_Terminal_01x02 J5
 U 1 1 5E6A427F
-P 7700 4400
-F 0 "J5" H 7780 4392 50  0000 L CNN
-F 1 "Screw_Terminal_01x02" H 7780 4301 50  0000 L CNN
-F 2 "TerminalBlock:TerminalBlock_bornier-2_P5.08mm" H 7700 4400 50  0001 C CNN
-F 3 "~" H 7700 4400 50  0001 C CNN
-	1    7700 4400
-	1    0    0    -1
-$EndComp
-Text Notes 5200 3300 0    50   ~ 0
-I am calculating this resistor value. Please hold.
-Text Notes 5250 4950 0    50   ~ 0
-I am calculating this resistor value. Please hold.
+P 6750 4750
+F 0 "J5" H 6830 4742 50  0000 L CNN
+F 1 "Screw_Terminal_01x02" H 6830 4651 50  0000 L CNN
+F 2 "TerminalBlock:TerminalBlock_bornier-2_P5.08mm" H 6750 4750 50  0001 C CNN
+F 3 "~" H 6750 4750 50  0001 C CNN
+	1    6750 4750
+	1    0    0    -1
+$EndComp
 Wire Wire Line
 	4700 4150 5050 4150
@@
 L power:GNDPWR #PWR042
 U 1 1 5FFC7614
-P 7500 2850
-F 0 "#PWR042" H 7500 2650 50  0001 C CNN
-F 1 "GNDPWR" H 7504 2696 50  0000 C CNN
-F 2 "" H 7500 2800 50  0001 C CNN
-F 3 "" H 7500 2800 50  0001 C CNN
-	1    7500 2850
+P 6550 3200
+F 0 "#PWR042" H 6550 3000 50  0001 C CNN
+F 1 "GNDPWR" H 6554 3046 50  0000 C CNN
+F 2 "" H 6550 3150 50  0001 C CNN
+F 3 "" H 6550 3150 50  0001 C CNN
+	1    6550 3200
 	1    0    0    -1
 $EndComp
@@
 L power:GNDPWR #PWR043
 U 1 1 5FFCCA77
-P 7500 4500
-F 0 "#PWR043" H 7500 4300 50  0001 C CNN
-F 1 "GNDPWR" H 7504 4346 50  0000 C CNN
-F 2 "" H 7500 4450 50  0001 C CNN
-F 3 "" H 7500 4450 50  0001 C CNN
-	1    7500 4500
+P 6550 4850
+F 0 "#PWR043" H 6550 4650 50  0001 C CNN
+F 1 "GNDPWR" H 6554 4696 50  0000 C CNN
+F 2 "" H 6550 4800 50  0001 C CNN
+F 3 "" H 6550 4800 50  0001 C CNN
+	1    6550 4850
 	1    0    0    -1
 $EndComp
@@
 	1    0    0    -1
 $EndComp
-Wire Wire Line
-	7300 2750 7300 3100
-Wire Wire Line
-	7300 2750 7500 2750
-Wire Wire Line
-	7300 3100 6200 3100
-Wire Wire Line
-	7300 4400 7300 4750
-Wire Wire Line
-	7300 4400 7500 4400
-Wire Wire Line
-	7300 4750 6200 4750
 $Comp
 L Device:R_US R?
 U 1 1 5FFFD96D
-P 4100 3500
+P 4350 3500
 AR Path="/5FFFD96D" Ref="R?"  Part="1"
 AR Path="/5DEFE67E/5FFFD96D" Ref="R1"  Part="1"
-F 0 "R1" H 4168 3546 50  0000 L CNN
-F 1 "1M" H 4168 3455 50  0000 L CNN
-F 2 "Resistor_SMD:R_0603_1608Metric" V 4140 3490 50  0001 C CNN
-F 3 "~" H 4100 3500 50  0001 C CNN
-	1    4100 3500
-	1    0    0    -1
-$EndComp
-Wire Wire Line
-	4100 3350 4150 3350
-Wire Wire Line
-	4450 3550 4450 3650
+F 0 "R1" H 4418 3546 50  0000 L CNN
+F 1 "1M" H 4418 3455 50  0000 L CNN
+F 2 "Resistor_SMD:R_0603_1608Metric" V 4390 3490 50  0001 C CNN
+F 3 "~" H 4350 3500 50  0001 C CNN
+	1    4350 3500
+	1    0    0    -1
+$EndComp
+Wire Wire Line
+	4350 3350 4400 3350
+Wire Wire Line
+	4700 3550 4700 3650
 $Comp
 L Transistor_FET:BSS138 Q?
 U 1 1 5FFFD975
-P 4350 3350
+P 4600 3350
 AR Path="/5FFFD975" Ref="Q?"  Part="1"
 AR Path="/5DEFE67E/5FFFD975" Ref="Q2"  Part="1"
-F 0 "Q2" H 4554 3396 50  0000 L CNN
-F 1 "BSS138" H 4554 3305 50  0000 L CNN
-F 2 "Package_TO_SOT_SMD:SOT-23" H 4550 3275 50  0001 L CIN
-F 3 "https://www.onsemi.com/pub/Collateral/BSS138-D.PDF" H 4350 3350 50  0001 L CNN
-	1    4350 3350
+F 0 "Q2" H 4804 3396 50  0000 L CNN
+F 1 "BSS138" H 4804 3305 50  0000 L CNN
+F 2 "Package_TO_SOT_SMD:SOT-23" H 4800 3275 50  0001 L CIN
+F 3 "https://www.onsemi.com/pub/Collateral/BSS138-D.PDF" H 4600 3350 50  0001 L CNN
+	1    4600 3350
 	1    0    0    -1
 $EndComp
@@
 L power:GND #PWR?
 U 1 1 5FFFD97C
-P 4450 3650
+P 4700 3650
 AR Path="/5FFFD97C" Ref="#PWR?"  Part="1"
 AR Path="/5DEFE67E/5FFFD97C" Ref="#PWR032"  Part="1"
-F 0 "#PWR032" H 4450 3400 50  0001 C CNN
-F 1 "GND" H 4455 3477 50  0000 C CNN
-F 2 "" H 4450 3650 50  0001 C CNN
-F 3 "" H 4450 3650 50  0001 C CNN
-	1    4450 3650
-	1    0    0    -1
-$EndComp
-Wire Wire Line
-	4100 3650 4450 3650
-Connection ~ 4450 3650
+F 0 "#PWR032" H 4700 3400 50  0001 C CNN
+F 1 "GND" H 4705 3477 50  0000 C CNN
+F 2 "" H 4700 3650 50  0001 C CNN
+F 3 "" H 4700 3650 50  0001 C CNN
+	1    4700 3650
+	1    0    0    -1
+$EndComp
+Wire Wire Line
+	4350 3650 4700 3650
+Connection ~ 4700 3650
 Wire Wire Line
 	4700 3100 4700 3150
-Wire Wire Line
-	4700 3150 5050 3150
 Wire Wire Line
 	5050 2950 5050 3150
@@
 Wire Wire Line
 	5800 3150 5800 3100
-Wire Wire Line
-	4450 3150 4700 3150
 Connection ~ 4700 3150
 Connection ~ 4700 2500
 Wire Wire Line
-	4000 3350 4100 3350
-Connection ~ 4100 3350
+	4250 3350 4350 3350
+Connection ~ 4350 3350
 Connection ~ 4700 4150
 Wire Wire Line
@@
 Wire Wire Line
 	5800 4800 5800 4750
-Wire Wire Line
-	4700 4800 5050 4800
 $Comp
 L Transistor_FET:BSS138 Q3
 U 1 1 6004A37A
-P 4350 5000
-F 0 "Q3" H 4554 5046 50  0000 L CNN
-F 1 "BSS138" H 4554 4955 50  0000 L CNN
-F 2 "Package_TO_SOT_SMD:SOT-23" H 4550 4925 50  0001 L CIN
-F 3 "https://www.fairchildsemi.com/datasheets/BS/BSS138.pdf" H 4350 5000 50  0001 L CNN
-	1    4350 5000
+P 4600 5000
+F 0 "Q3" H 4804 5046 50  0000 L CNN
+F 1 "BSS138" H 4804 4955 50  0000 L CNN
+F 2 "Package_TO_SOT_SMD:SOT-23" H 4800 4925 50  0001 L CIN
+F 3 "https://www.fairchildsemi.com/datasheets/BS/BSS138.pdf" H 4600 5000 50  0001 L CNN
+	1    4600 5000
 	1    0    0    -1
 $EndComp
@@
 L power:GND #PWR033
 U 1 1 5E67CE4B
-P 4450 5300
-F 0 "#PWR033" H 4450 5050 50  0001 C CNN
-F 1 "GND" H 4455 5127 50  0000 C CNN
-F 2 "" H 4450 5300 50  0001 C CNN
-F 3 "" H 4450 5300 50  0001 C CNN
-	1    4450 5300
+P 4700 5300
+F 0 "#PWR033" H 4700 5050 50  0001 C CNN
+F 1 "GND" H 4705 5127 50  0000 C CNN
+F 2 "" H 4700 5300 50  0001 C CNN
+F 3 "" H 4700 5300 50  0001 C CNN
+	1    4700 5300
 	1    0    0    -1
 $EndComp
@@
 	0    -1   -1   0
 $EndComp
-Wire Wire Line
-	4700 4800 4450 4800
 Connection ~ 4700 4800
 $Comp
 L Device:R_US R22
 U 1 1 60068336
-P 4100 5150
-F 0 "R22" H 4168 5196 50  0000 L CNN
-F 1 "1M" H 4168 5105 50  0000 L CNN
-F 2 "Resistor_SMD:R_0603_1608Metric" V 4140 5140 50  0001 C CNN
-F 3 "~" H 4100 5150 50  0001 C CNN
-	1    4100 5150
-	1    0    0    -1
-$EndComp
-Connection ~ 4100 5000
-Wire Wire Line
-	4100 5000 4150 5000
-Wire Wire Line
-	4100 5300 4450 5300
-Wire Wire Line
-	4450 5300 4450 5200
-Connection ~ 4450 5300
-Wire Wire Line
-	4000 5000 4100 5000
+P 4350 5150
+F 0 "R22" H 4418 5196 50  0000 L CNN
+F 1 "1M" H 4418 5105 50  0000 L CNN
+F 2 "Resistor_SMD:R_0603_1608Metric" V 4390 5140 50  0001 C CNN
+F 3 "~" H 4350 5150 50  0001 C CNN
+	1    4350 5150
+	1    0    0    -1
+$EndComp
+Connection ~ 4350 5000
+Wire Wire Line
+	4350 5000 4400 5000
+Wire Wire Line
+	4350 5300 4700 5300
+Wire Wire Line
+	4700 5300 4700 5200
+Connection ~ 4700 5300
+Wire Wire Line
+	4250 5000 4350 5000
 $Comp
 L Connector:Conn_01x02_Male J10
@@
 P 4650 1800
 F 0 "J10" H 4758 1981 50  0000 C CNN
-F 1 "Conn_01x02_Male" H 4758 1890 50  0000 C CNN
+F 1 "9V_INPUT" H 4758 1890 50  0000 C CNN
 F 2 "Connector_JST:JST_XH_B2B-XH-A_1x02_P2.50mm_Vertical" H 4650 1800 50  0001 C CNN
 F 3 "~" H 4650 1800 50  0001 C CNN
@@
 L power:+9V #PWR034
 U 1 1 6008E69C
-P 5300 1800
-F 0 "#PWR034" H 5300 1650 50  0001 C CNN
-F 1 "+9V" H 5315 1973 50  0000 C CNN
-F 2 "" H 5300 1800 50  0001 C CNN
-F 3 "" H 5300 1800 50  0001 C CNN
-	1    5300 1800
-	1    0    0    -1
-$EndComp
-Wire Wire Line
-	4850 1800 5300 1800
-Wire Wire Line
-	4850 1900 5300 1900
+P 5000 1800
+F 0 "#PWR034" H 5000 1650 50  0001 C CNN
+F 1 "+9V" H 5015 1973 50  0000 C CNN
+F 2 "" H 5000 1800 50  0001 C CNN
+F 3 "" H 5000 1800 50  0001 C CNN
+	1    5000 1800
+	1    0    0    -1
+$EndComp
 $Comp
 L power:GNDPWR #PWR035
 U 1 1 6009988C
-P 5300 1900
-F 0 "#PWR035" H 5300 1700 50  0001 C CNN
-F 1 "GNDPWR" H 5304 1746 50  0000 C CNN
-F 2 "" H 5300 1850 50  0001 C CNN
-F 3 "" H 5300 1850 50  0001 C CNN
-	1    5300 1900
+P 5000 1900
+F 0 "#PWR035" H 5000 1700 50  0001 C CNN
+F 1 "GNDPWR" H 5004 1746 50  0000 C CNN
+F 2 "" H 5000 1850 50  0001 C CNN
+F 3 "" H 5000 1850 50  0001 C CNN
+	1    5000 1900
 	1    0    0    -1
 $EndComp
@@
 Wire Wire Line
 	6100 3850 6100 4150
+Wire Wire Line
+	4700 3150 5050 3150
+Wire Wire Line
+	4700 4800 5050 4800
+Wire Wire Line
+	6550 3100 6200 3100
+Wire Wire Line
+	6550 4750 6200 4750
+Wire Wire Line
+	5000 1900 4850 1900
+Wire Wire Line
+	4850 1800 5000 1800
 $EndSCHEMATC

Commit message: Recovery PCB: Reannotate
Reannotated schematic to fix reference numbering and keep reference
designators consistent.
Parts:
- renumbered D4 to D2, D2 to D3, D5 to D4, D3 to D5, J10 to J4, J4 to J5, J5 to J6, R9 to R10, R22 to R12, R8 to R7, R10 to R8, R1 to R9
Changed lines of the file:
@@
 $EndComp
 $Comp
-L Device:LED D2
+L Device:LED D3
 U 1 1 5E58CA13
 P 4700 2950
-F 0 "D2" V 4739 2833 50  0000 R CNN
+F 0 "D3" V 4739 2833 50  0000 R CNN
 F 1 "LED" V 4648 2833 50  0000 R CNN
 F 2 "LED_SMD:LED_0603_1608Metric" H 4700 2950 50  0001 C CNN
@@
 $EndComp
 $Comp
-L Device:R_US R10
+L Device:R_US R8
 U 1 1 5E590CAC
 P 5350 3150
-F 0 "R10" V 5145 3150 50  0000 C CNN
+F 0 "R8" V 5145 3150 50  0000 C CNN
 F 1 "300" V 5236 3150 50  0000 C CNN
 F 2 "Resistor_SMD:R_0603_1608Metric" V 5390 3140 50  0001 C CNN
@@
 $EndComp
 $Comp
-L Device:R_US R8
+L Device:R_US R7
 U 1 1 5E65853B
 P 4700 2650
-F 0 "R8" H 4768 2696 50  0000 L CNN
+F 0 "R7" H 4768 2696 50  0000 L CNN
 F 1 "220" H 4768 2605 50  0000 L CNN
 F 2 "Resistor_SMD:R_0603_1608Metric" V 4740 2640 50  0001 C CNN
@@
 $EndComp
 $Comp
-L Device:R_US R9
+L Device:R_US R10
 U 1 1 5E662768
 P 4700 4300
-F 0 "R9" H 4768 4346 50  0000 L CNN
+F 0 "R10" H 4768 4346 50  0000 L CNN
 F 1 "220" H 4768 4255 50  0000 L CNN
 F 2 "Resistor_SMD:R_0603_1608Metric" V 4740 4290 50  0001 C CNN
@@
 $EndComp
 $Comp
-L power:+9V #PWR040
+L power:+9V #PWR046
 U 1 1 5E69B629
 P 6300 2500
-F 0 "#PWR040" H 6300 2350 50  0001 C CNN
+F 0 "#PWR046" H 6300 2350 50  0001 C CNN
 F 1 "+9V" H 6315 2673 50  0000 C CNN
 F 2 "" H 6300 2500 50  0001 C CNN
@@
 $EndComp
 $Comp
-L Connector:Screw_Terminal_01x02 J4
+L Connector:Screw_Terminal_01x02 J5
 U 1 1 5E69C0D8
 P 6750 3100
-F 0 "J4" H 6830 3092 50  0000 L CNN
+F 0 "J5" H 6830 3092 50  0000 L CNN
 F 1 "Screw_Terminal_01x02" H 6830 3001 50  0000 L CNN
 F 2 "TerminalBlock:TerminalBlock_bornier-2_P5.08mm" H 6750 3100 50  0001 C CNN
@@
 $EndComp
 $Comp
-L power:+9V #PWR041
+L power:+9V #PWR051
 U 1 1 5E6A3657
 P 6300 4150
-F 0 "#PWR041" H 6300 4000 50  0001 C CNN
+F 0 "#PWR051" H 6300 4000 50  0001 C CNN
 F 1 "+9V" H 6315 4323 50  0000 C CNN
 F 2 "" H 6300 4150 50  0001 C CNN
@@
 $EndComp
 $Comp
-L Connector:Screw_Terminal_01x02 J5
+L Connector:Screw_Terminal_01x02 J6
 U 1 1 5E6A427F
 P 6750 4750
-F 0 "J5" H 6830 4742 50  0000 L CNN
+F 0 "J6" H 6830 4742 50  0000 L CNN
 F 1 "Screw_Terminal_01x02" H 6830 4651 50  0000 L CNN
 F 2 "TerminalBlock:TerminalBlock_bornier-2_P5.08mm" H 6750 4750 50  0001 C CNN
@@
 	5050 4150 5050 4300
 $Comp
-L Device:D D5
+L Device:D D4
 U 1 1 5E662736
 P 5050 4450
-F 0 "D5" V 5004 4529 50  0000 L CNN
+F 0 "D4" V 5004 4529 50  0000 L CNN
 F 1 "D" V 5095 4529 50  0000 L CNN
 F 2 "Diode_SMD:D_SOT-23_ANK" H 5050 4450 50  0001 C CNN
@@
 	5050 2500 5050 2650
 $Comp
-L Device:D D4
+L Device:D D2
 U 1 1 5E58FAD9
 P 5050 2800
-F 0 "D4" V 5004 2879 50  0000 L CNN
+F 0 "D2" V 5004 2879 50  0000 L CNN
 F 1 "D" V 5095 2879 50  0000 L CNN
 F 2 "Diode_SMD:D_SOT-23_ANK" H 5050 2800 50  0001 C CNN
@@
 $EndComp
 $Comp
-L power:GNDPWR #PWR042
+L power:GNDPWR #PWR047
 U 1 1 5FFC7614
 P 6550 3200
-F 0 "#PWR042" H 6550 3000 50  0001 C CNN
+F 0 "#PWR047" H 6550 3000 50  0001 C CNN
 F 1 "GNDPWR" H 6554 3046 50  0000 C CNN
 F 2 "" H 6550 3150 50  0001 C CNN
@@
 $EndComp
 $Comp
-L power:GNDPWR #PWR043
+L power:GNDPWR #PWR052
 U 1 1 5FFCCA77
 P 6550 4850
-F 0 "#PWR043" H 6550 4650 50  0001 C CNN
+F 0 "#PWR052" H 6550 4650 50  0001 C CNN
 F 1 "GNDPWR" H 6554 4696 50  0000 C CNN
 F 2 "" H 6550 4800 50  0001 C CNN
@@
 $EndComp
 $Comp
-L power:+3.3V #PWR036
+L power:+3.3V #PWR045
 U 1 1 5FFCE97E
 P 4700 2500
-F 0 "#PWR036" H 4700 2350 50  0001 C CNN
+F 0 "#PWR045" H 4700 2350 50  0001 C CNN
 F 1 "+3.3V" H 4715 2673 50  0000 C CNN
 F 2 "" H 4700 2500 50  0001 C CNN
@@
 $EndComp
 $Comp
-L power:+3.3V #PWR037
+L power:+3.3V #PWR050
 U 1 1 5FFCF2F1
 P 4700 4150
-F 0 "#PWR037" H 4700 4000 50  0001 C CNN
+F 0 "#PWR050" H 4700 4000 50  0001 C CNN
 F 1 "+3.3V" H 4715 4323 50  0000 C CNN
 F 2 "" H 4700 4150 50  0001 C CNN
@@
 P 4350 3500
 AR Path="/5FFFD96D" Ref="R?"  Part="1"
-AR Path="/5DEFE67E/5FFFD96D" Ref="R1"  Part="1"
-F 0 "R1" H 4418 3546 50  0000 L CNN
+AR Path="/5DEFE67E/5FFFD96D" Ref="R9"  Part="1"
+F 0 "R9" H 4418 3546 50  0000 L CNN
 F 1 "1M" H 4418 3455 50  0000 L CNN
 F 2 "Resistor_SMD:R_0603_1608Metric" V 4390 3490 50  0001 C CNN
@@
 P 4700 3650
 AR Path="/5FFFD97C" Ref="#PWR?"  Part="1"
-AR Path="/5DEFE67E/5FFFD97C" Ref="#PWR032"  Part="1"
-F 0 "#PWR032" H 4700 3400 50  0001 C CNN
+AR Path="/5DEFE67E/5FFFD97C" Ref="#PWR048"  Part="1"
+F 0 "#PWR048" H 4700 3400 50  0001 C CNN
 F 1 "GND" H 4705 3477 50  0000 C CNN
 F 2 "" H 4700 3650 50  0001 C CNN
@@
 $EndComp
 $Comp
-L power:GND #PWR033
+L power:GND #PWR053
 U 1 1 5E67CE4B
 P 4700 5300
-F 0 "#PWR033" H 4700 5050 50  0001 C CNN
+F 0 "#PWR053" H 4700 5050 50  0001 C CNN
 F 1 "GND" H 4705 5127 50  0000 C CNN
 F 2 "" H 4700 5300 50  0001 C CNN
@@
 $EndComp
 $Comp
-L Device:LED D3
+L Device:LED D5
 U 1 1 5E662754
 P 4700 4600
-F 0 "D3" V 4739 4483 50  0000 R CNN
+F 0 "D5" V 4739 4483 50  0000 R CNN
 F 1 "LED" V 4648 4483 50  0000 R CNN
 F 2 "LED_SMD:LED_0603_1608Metric" H 4700 4600 50  0001 C CNN
@@
 Connection ~ 4700 4800
 $Comp
-L Device:R_US R22
+L Device:R_US R12
 U 1 1 60068336
 P 4350 5150
-F 0 "R22" H 4418 5196 50  0000 L CNN
+F 0 "R12" H 4418 5196 50  0000 L CNN
 F 1 "1M" H 4418 5105 50  0000 L CNN
 F 2 "Resistor_SMD:R_0603_1608Metric" V 4390 5140 50  0001 C CNN
@@
 	4250 5000 4350 5000
 $Comp
-L Connector:Conn_01x02_Male J10
+L Connector:Conn_01x02_Male J4
 U 1 1 6008C622
 P 4650 1800
-F 0 "J10" H 4758 1981 50  0000 C CNN
+F 0 "J4" H 4758 1981 50  0000 C CNN
 F 1 "9V_INPUT" H 4758 1890 50  0000 C CNN
 F 2 "Connector_JST:JST_XH_B2B-XH-A_1x02_P2.50mm_Vertical" H 4650 1800 50  0001 C CNN
@@
 $EndComp
 $Comp
-L power:+9V #PWR034
+L power:+9V #PWR042
 U 1 1 6008E69C
 P 5000 1800
-F 0 "#PWR034" H 5000 1650 50  0001 C CNN
+F 0 "#PWR042" H 5000 1650 50  0001 C CNN
 F 1 "+9V" H 5015 1973 50  0000 C CNN
 F 2 "" H 5000 1800 50  0001 C CNN
@@
 $EndComp
 $Comp
-L power:GNDPWR #PWR035
+L power:GNDPWR #PWR043
 U 1 1 6009988C
 P 5000 1900
-F 0 "#PWR035" H 5000 1700 50  0001 C CNN
+F 0 "#PWR043" H 5000 1700 50  0001 C CNN
 F 1 "GNDPWR" H 5004 1746 50  0000 C CNN
 F 2 "" H 5000 1850 50  0001 C CNN
@@
 $EndComp
 $Comp
-L power:GNDPWR #PWR038
+L power:GNDPWR #PWR044
 U 1 1 600B3A6E
 P 5900 2200
-F 0 "#PWR038" H 5900 2000 50  0001 C CNN
+F 0 "#PWR044" H 5900 2000 50  0001 C CNN
 F 1 "GNDPWR" H 5904 2046 50  0000 C CNN
 F 2 "" H 5900 2150 50  0001 C CNN
@@
 	6100 2200 6100 2500
 $Comp
-L power:GNDPWR #PWR039
+L power:GNDPWR #PWR049
 U 1 1 600BDC8C
 P 5900 3850
-F 0 "#PWR039" H 5900 3650 50  0001 C CNN
+F 0 "#PWR049" H 5900 3650 50  0001 C CNN
 F 1 "GNDPWR" H 5904 3696 50  0000 C CNN
 F 2 "" H 5900 3800 50  0001 C CNN

Commit message: Recovery PCB: Fix relay
Replaced unavailable relay with a correct part and replaced voltage
regulator with an easier to solder alternative.
Parts:
- K1, K2: value SANYOU_SRD_Form_C -> G6RL-14-ASI-DC3; footprint Relay_THT:Relay_SPDT_SANYOU_SRD_Series_Form_C -> Parts:RELAY_G6RL-1; symbol Relay:SANYOU_SRD_Form_C -> recovery-custom:G6RL-14-ASI-DC3
- R11, R8: value 300 -> 5
Other:
- note added: "Coil resistance: 40Ohms @ 3v3\nI_rated: 0.0733\nI_rated = Vcc/(R_coil+R_limit)\nAt rated voltage, minimal resistance needed"
Changed lines of the file:
@@
 IN1
 $Comp
-L Relay:SANYOU_SRD_Form_C K1
+L recovery-custom:G6RL-14-ASI-DC3 K1
 U 1 1 5E651D90
 P 6000 2800
 F 0 "K1" H 6430 2846 50  0000 L CNN
-F 1 "SANYOU_SRD_Form_C" H 6430 2755 50  0000 L CNN
-F 2 "Relay_THT:Relay_SPDT_SANYOU_SRD_Series_Form_C" H 6450 2750 50  0001 L CNN
-F 3 "http://www.sanyourelay.ca/public/products/pdf/SRD.pdf" H 6000 2800 50  0001 C CNN
+F 1 "G6RL-14-ASI-DC3" H 6430 2755 50  0000 L CNN
+F 2 "Parts:RELAY_G6RL-1" H 6450 2750 50  0001 L CNN
+F 3 "https://omronfs.omron.com/en_US/ecb/products/pdf/en-g6rl.pdf" H 6000 2800 50  0001 C CNN
 	1    6000 2800
 	1    0    0    -1
@@
 P 5350 3150
 F 0 "R8" V 5145 3150 50  0000 C CNN
-F 1 "300" V 5236 3150 50  0000 C CNN
+F 1 "5" V 5236 3150 50  0000 C CNN
 F 2 "Resistor_SMD:R_0603_1608Metric" V 5390 3140 50  0001 C CNN
 F 3 "~" H 5350 3150 50  0001 C CNN
@@
 IN2
 $Comp
-L Relay:SANYOU_SRD_Form_C K2
+L recovery-custom:G6RL-14-ASI-DC3 K2
 U 1 1 5E66272F
 P 6000 4450
 F 0 "K2" H 6430 4496 50  0000 L CNN
-F 1 "SANYOU_SRD_Form_C" H 6430 4405 50  0000 L CNN
-F 2 "Relay_THT:Relay_SPDT_SANYOU_SRD_Series_Form_C" H 6450 4400 50  0001 L CNN
-F 3 "http://www.sanyourelay.ca/public/products/pdf/SRD.pdf" H 6000 4450 50  0001 C CNN
+F 1 "G6RL-14-ASI-DC3" H 6430 4405 50  0000 L CNN
+F 2 "Parts:RELAY_G6RL-1" H 6450 4400 50  0001 L CNN
+F 3 "https://omronfs.omron.com/en_US/ecb/products/pdf/en-g6rl.pdf" H 6000 4450 50  0001 C CNN
 	1    6000 4450
 	1    0    0    -1
@@
 P 5350 4800
 F 0 "R11" V 5145 4800 50  0000 C CNN
-F 1 "300" V 5236 4800 50  0000 C CNN
+F 1 "5" V 5236 4800 50  0000 C CNN
 F 2 "Resistor_SMD:R_0603_1608Metric" V 5390 4790 50  0001 C CNN
 F 3 "~" H 5350 4800 50  0001 C CNN
@@
 Wire Wire Line
 	4850 1800 5000 1800
+Text Notes 5150 3700 0    50   ~ 0
+Coil resistance: 40Ohms @ 3v3\nI_rated: 0.0733\nI_rated = Vcc/(R_coil+R_limit)\nAt rated voltage, minimal resistance needed
+$Comp
+L power:PWR_FLAG #FLG?
+U 1 1 60045E18
+P 5000 1800
+F 0 "#FLG?" H 5000 1875 50  0001 C CNN
+F 1 "PWR_FLAG" V 5000 1928 50  0000 L CNN
+F 2 "" H 5000 1800 50  0001 C CNN
+F 3 "~" H 5000 1800 50  0001 C CNN
+	1    5000 1800
+	0    1    1    0
+$EndComp
+Connection ~ 5000 1800
+$Comp
+L power:PWR_FLAG #FLG?
+U 1 1 6004749E
+P 5000 1900
+F 0 "#FLG?" H 5000 1975 50  0001 C CNN
+F 1 "PWR_FLAG" V 5000 2028 50  0000 L CNN
+F 2 "" H 5000 1900 50  0001 C CNN
+F 3 "~" H 5000 1900 50  0001 C CNN
+	1    5000 1900
+	0    1    1    0
+$EndComp
 $EndSCHEMATC

Commit message: Replaced IMU, relays, and power regulator with new components. Modified schematic accordingly.
Parts:
- removed K1, K2: G6RL-14-ASI-DC3, Parts:RELAY_G6RL-1, symbol recovery-custom:G6RL-14-ASI-DC3
- added U5, U6: Panasonic-PA-N, symbol Panasonic-PA-N:Panasonic-PA-N
Connections:
- wire segments 34 -> 30

Commit message: Reperformed board layout with new components.
Parts:
- R11, R8: value 5 -> 10
- U5, U6: footprint (none) -> Parts:Panasonic-PA-N
Other:
- note added: "Coil resistance: 82Ohms @ 3V\nI_rated: 0.0367\nI_rated = Vcc/(R_coil+R_limit)\nAt rated voltage, minimal resistance needed"
- note removed: "Coil resistance: 40Ohms @ 3v3\nI_rated: 0.0733\nI_rated = Vcc/(R_coil+R_limit)\nAt rated voltage, minimal resistance needed"
Changed lines of the file:
@@
 P 5350 3250
 F 0 "R8" V 5145 3250 50  0000 C CNN
-F 1 "5" V 5236 3250 50  0000 C CNN
+F 1 "10" V 5236 3250 50  0000 C CNN
 F 2 "Resistor_SMD:R_0603_1608Metric" V 5390 3240 50  0001 C CNN
 F 3 "~" H 5350 3250 50  0001 C CNN
@@
 P 5350 4950
 F 0 "R11" V 5145 4950 50  0000 C CNN
-F 1 "5" V 5236 4950 50  0000 C CNN
+F 1 "10" V 5236 4950 50  0000 C CNN
 F 2 "Resistor_SMD:R_0603_1608Metric" V 5390 4940 50  0001 C CNN
 F 3 "~" H 5350 4950 50  0001 C CNN
@@
 	4850 1800 5000 1800
 Text Notes 5250 3900 0    50   ~ 0
-Coil resistance: 40Ohms @ 3v3\nI_rated: 0.0733\nI_rated = Vcc/(R_coil+R_limit)\nAt rated voltage, minimal resistance needed
+Coil resistance: 82Ohms @ 3V\nI_rated: 0.0367\nI_rated = Vcc/(R_coil+R_limit)\nAt rated voltage, minimal resistance needed
 $Comp
 L power:PWR_FLAG #FLG01
@@
 F 0 "U5" V 6000 2500 50  0000 C CNN
 F 1 "Panasonic-PA-N" V 5900 2250 50  0000 C CNN
-F 2 "" H 5900 2950 50  0001 C CNN
+F 2 "Parts:Panasonic-PA-N" H 5900 2950 50  0001 C CNN
 F 3 "" H 5900 2950 50  0001 C CNN
 	1    5900 2950
@@
 F 0 "U6" V 6000 4200 50  0000 C CNN
 F 1 "Panasonic-PA-N" V 5900 3950 50  0000 C CNN
-F 2 "" H 5900 4650 50  0001 C CNN
+F 2 "Parts:Panasonic-PA-N" H 5900 4650 50  0001 C CNN
 F 3 "" H 5900 4650 50  0001 C CNN
 	1    5900 4650
