File: Recovery PCB/Recovery PCB.sch (KiCad schematic (older format))
At the start: 17 parts, among them J4 Rotary_Switch_Header

Commit message: Updated recovery board with new connections.
Parts:
- removed R?: 330, symbol Device:R
- added J?: Conn_02x05_Odd_Even, symbol Connector_Generic:Conn_02x05_Odd_Even
- added J?: Conn_01x04_Male, symbol Connector:Conn_01x04_Male
- added Q?: BSS138, Package_TO_SOT_SMD:SOT-23, symbol Transistor_FET:BSS138
- added R?: 10k, symbol Device:R_US
- added R?: 330, symbol Device:R_US
- added R?: 1k, symbol Device:R_US
- added R?: 1M, symbol Device:R_US
Connections:
- net labels added: +3V3, +5V, BUZZER, CLK, IMU_INT, IMU_RESET, IN1, IN2, MISO, MOSI, RADIO_CS, RADIO_IO, RADIO_RESET, SCL, SDA, SD_CS, Xout, Yout, Zout
- wire segments 37 -> 102
- no-connect marks 0 -> 6

Commit message: Update relays and re-annotate entire schematic. Review needed before layout.
Parts:
- removed J4: Rotary_Switch_Header, Connector_PinHeader_1.00mm:PinHeader_1x02_P1.00mm_Vertical, symbol Connector:Conn_01x02_Male
- gave numbers to parts that had none: 21
Other:
- note added: "Add rotary switch. Figure out what it does."
Changed lines of the file:
@@
 F3 "IN1" I L 3200 1350 50
 $EndSheet
-$Comp
-L Connector:Conn_01x02_Male J4
-U 1 1 5DF4E3A8
-P 3400 4100
-F 0 "J4" H 3508 4281 50  0000 C CNN
-F 1 "Rotary_Switch_Header" H 3508 4190 50  0000 C CNN
-F 2 "Connector_PinHeader_1.00mm:PinHeader_1x02_P1.00mm_Vertical" H 3400 4100 50  0001 C CNN
-F 3 "~" H 3400 4100 50  0001 C CNN
-	1    3400 4100
-	1    0    0    -1
-$EndComp
 $Sheet
 S 3200 1900 550  500
@@
 $EndSheet
 $Comp
-L Device:Crystal Y?
+L Device:Crystal Y1
 U 1 1 5E27B68E
 P 5400 2550
-F 0 "Y?" V 5354 2681 50  0000 L CNN
+F 0 "Y1" V 5354 2681 50  0000 L CNN
 F 1 "32.768kHz" V 5445 2681 50  0000 L CNN
 F 2 "" H 5400 2550 50  0001 C CNN
@@
 	5400 2700 5950 2700
 $Comp
-L Device:C C?
+L Device:C C2
 U 1 1 5E27B93F
 P 5400 2850
-F 0 "C?" H 5515 2896 50  0000 L CNN
+F 0 "C2" H 5515 2896 50  0000 L CNN
 F 1 "22p" H 5515 2805 50  0000 L CNN
 F 2 "" H 5438 2700 50  0001 C CNN
@@
 Connection ~ 5400 2700
 $Comp
-L Device:C C?
+L Device:C C1
 U 1 1 5E27BA52
 P 5000 2850
-F 0 "C?" H 5115 2896 50  0000 L CNN
+F 0 "C1" H 5115 2896 50  0000 L CNN
 F 1 "22p" H 5115 2805 50  0000 L CNN
 F 2 "" H 5038 2700 50  0001 C CNN
@@
 	5400 3000 5300 3000
 $Comp
-L power:GND #PWR?
+L power:GND #PWR07
 U 1 1 5E27BB25
 P 5300 3000
-F 0 "#PWR?" H 5300 2750 50  0001 C CNN
+F 0 "#PWR07" H 5300 2750 50  0001 C CNN
 F 1 "GND" H 5305 2827 50  0000 C CNN
 F 2 "" H 5300 3000 50  0001 C CNN
@@
 No, it's not done yet.
 $Comp
-L power:GND #PWR?
+L power:GND #PWR013
 U 1 1 5E2E1420
 P 7650 5900
-F 0 "#PWR?" H 7650 5650 50  0001 C CNN
+F 0 "#PWR013" H 7650 5650 50  0001 C CNN
 F 1 "GND" H 7655 5727 50  0000 C CNN
 F 2 "" H 7650 5900 50  0001 C CNN
@@
 $EndComp
 $Comp
-L MCU_Microchip_SAMD:ATSAMD21G18A-AUT U?
+L MCU_Microchip_SAMD:ATSAMD21G18A-AUT U1
 U 1 1 5E27AB92
 P 7100 4000
-F 0 "U?" H 7100 2014 50  0000 C CNN
+F 0 "U1" H 7100 2014 50  0000 C CNN
 F 1 "ATSAMD21G18A-AUT" H 7100 1923 50  0000 C CNN
 F 2 "Package_QFP:TQFP-48_7x7mm_P0.5mm" H 6150 2250 50  0001 C CNN
@@
 $EndComp
 $Comp
-L Switch:SW_Push SW?
+L Switch:SW_Push SW1
 U 1 1 5E2E1A9C
 P 5450 6350
-F 0 "SW?" V 5496 6302 50  0000 R CNN
+F 0 "SW1" V 5496 6302 50  0000 R CNN
 F 1 "SW_Push" V 5405 6302 50  0000 R CNN
 F 2 "" H 5450 6550 50  0001 C CNN
@@
 	7000 5900 7200 5900
 $Comp
-L Device:C C?
+L Device:C C9
 U 1 1 5E2E29D6
 P 7450 1950
-F 0 "C?" V 7198 1950 50  0000 C CNN
+F 0 "C9" V 7198 1950 50  0000 C CNN
 F 1 "1u" V 7289 1950 50  0000 C CNN
 F 2 "" H 7488 1800 50  0001 C CNN
@@
 $EndComp
 $Comp
-L power:GND #PWR?
+L power:GND #PWR012
 U 1 1 5E2E2A5A
 P 7600 2050
-F 0 "#PWR?" H 7600 1800 50  0001 C CNN
+F 0 "#PWR012" H 7600 1800 50  0001 C CNN
 F 1 "GND" H 7605 1877 50  0000 C CNN
 F 2 "" H 7600 2050 50  0001 C CNN
@@
 $EndComp
 $Comp
-L Device:C C?
+L Device:C C7
 U 1 1 5E2E2AE2
 P 7450 1050
-F 0 "C?" V 7198 1050 50  0000 C CNN
+F 0 "C7" V 7198 1050 50  0000 C CNN
 F 1 "10u" V 7289 1050 50  0000 C CNN
 F 2 "" H 7488 900 50  0001 C CNN
@@
 $EndComp
 $Comp
-L Device:C C?
+L Device:C C8
 U 1 1 5E2E2B89
 P 7450 1500
-F 0 "C?" V 7198 1500 50  0000 C CNN
+F 0 "C8" V 7198 1500 50  0000 C CNN
 F 1 "100n" V 7289 1500 50  0000 C CNN
 F 2 "" H 7488 1350 50  0001 C CNN
@@
 $EndComp
 $Comp
-L power:GND #PWR?
+L power:GND #PWR011
 U 1 1 5E2E2E9D
 P 6600 2050
-F 0 "#PWR?" H 6600 1800 50  0001 C CNN
+F 0 "#PWR011" H 6600 1800 50  0001 C CNN
 F 1 "GND" H 6605 1877 50  0000 C CNN
 F 2 "" H 6600 2050 50  0001 C CNN
@@
 $EndComp
 $Comp
-L Device:C C?
+L Device:C C6
 U 1 1 5E2E3FFA
 P 6750 1950
-F 0 "C?" V 6498 1950 50  0000 C CNN
+F 0 "C6" V 6498 1950 50  0000 C CNN
 F 1 "100n" V 6589 1950 50  0000 C CNN
 F 2 "" H 6788 1800 50  0001 C CNN
@@
 	6600 2050 6600 1950
 $Comp
-L Device:C C?
+L Device:C C5
 U 1 1 5E2E542C
 P 6750 1500
-F 0 "C?" V 6498 1500 50  0000 C CNN
+F 0 "C5" V 6498 1500 50  0000 C CNN
 F 1 "100n" V 6589 1500 50  0000 C CNN
 F 2 "" H 6788 1350 50  0001 C CNN
@@
 Connection ~ 6600 1950
 $Comp
-L power:+3.3V #PWR?
+L power:+3.3V #PWR08
 U 1 1 5E2E6BFA
 P 6000 1050
-F 0 "#PWR?" H 6000 900 50  0001 C CNN
+F 0 "#PWR08" H 6000 900 50  0001 C CNN
 F 1 "+3.3V" H 6015 1223 50  0000 C CNN
 F 2 "" H 6000 1050 50  0001 C CNN
@@
 $EndComp
 $Comp
-L Device:C C?
+L Device:C C4
 U 1 1 5E2E7512
 P 6300 1750
-F 0 "C?" H 6415 1796 50  0000 L CNN
+F 0 "C4" H 6415 1796 50  0000 L CNN
 F 1 "10u" H 6415 1705 50  0000 L CNN
 F 2 "" H 6338 1600 50  0001 C CNN
@@
 	6300 1950 6600 1950
 $Comp
-L pspice:INDUCTOR L?
+L pspice:INDUCTOR L1
 U 1 1 5E2E97C8
 P 6650 1050
-F 0 "L?" H 6650 1265 50  0000 C CNN
+F 0 "L1" H 6650 1265 50  0000 C CNN
 F 1 "10uH" H 6650 1174 50  0000 C CNN
 F 2 "" H 6650 1050 50  0001 C CNN
@@
 	6300 1050 6400 1050
 $Comp
-L Device:Ferrite_Bead_Small FB?
+L Device:Ferrite_Bead_Small FB1
 U 1 1 5E2EAF0E
 P 7100 1050
-F 0 "FB?" V 6863 1050 50  0000 C CNN
+F 0 "FB1" V 6863 1050 50  0000 C CNN
 F 1 "Ferrite_Bead_Small" V 6954 1050 50  0000 C CNN
 F 2 "" V 7030 1050 50  0001 C CNN
@@
 Connection ~ 7000 1500
 $Comp
-L Device:C C?
+L Device:C C3
 U 1 1 5E2EBF3D
 P 6000 6350
-F 0 "C?" H 6115 6396 50  0000 L CNN
+F 0 "C3" H 6115 6396 50  0000 L CNN
 F 1 "100n" H 6115 6305 50  0000 L CNN
 F 2 "" H 6038 6200 50  0001 C CNN
@@
 Connection ~ 7200 5900
 $Comp
-L Connector_Generic:Conn_02x05_Odd_Even J?
+L Connector_Generic:Conn_02x05_Odd_Even J2
 U 1 1 5E51F52E
 P 5150 5500
-F 0 "J?" H 5200 5917 50  0000 C CNN
+F 0 "J2" H 5200 5917 50  0000 C CNN
 F 1 "Conn_02x05_Odd_Even" H 5200 5826 50  0000 C CNN
 F 2 "" H 5150 5500 50  0001 C CNN
@@
 $EndComp
 $Comp
-L Device:R_US R?
+L Device:R_US R4
 U 1 1 5E5278AF
 P 6000 6000
-F 0 "R?" H 6068 6046 50  0000 L CNN
+F 0 "R4" H 6068 6046 50  0000 L CNN
 F 1 "10k" H 6068 5955 50  0000 L CNN
 F 2 "" V 6040 5990 50  0001 C CNN
@@
 $EndComp
 $Comp
-L power:+3.3V #PWR?
+L power:+3.3V #PWR09
 U 1 1 5E52A8BC
 P 6000 5850
-F 0 "#PWR?" H 6000 5700 50  0001 C CNN
+F 0 "#PWR09" H 6000 5700 50  0001 C CNN
 F 1 "+3.3V" H 6015 6023 50  0000 C CNN
 F 2 "" H 6000 5850 50  0001 C CNN
@@
 $EndComp
 $Comp
-L Device:R_US R?
+L Device:R_US R3
 U 1 1 5E52BCFB
 P 5650 6150
-F 0 "R?" V 5445 6150 50  0000 C CNN
+F 0 "R3" V 5445 6150 50  0000 C CNN
 F 1 "330" V 5536 6150 50  0000 C CNN
 F 2 "" V 5690 6140 50  0001 C CNN
@@
 	5850 6150 6000 6150
 $Comp
-L power:GND #PWR?
+L power:GND #PWR010
 U 1 1 5E53FD32
 P 6000 6550
-F 0 "#PWR?" H 6000 6300 50  0001 C CNN
+F 0 "#PWR010" H 6000 6300 50  0001 C CNN
 F 1 "GND" H 6005 6377 50  0000 C CNN
 F 2 "" H 6000 6550 50  0001 C CNN
@@
 	4650 5300 4650 5100
 $Comp
-L power:+3.3V #PWR?
+L power:+3.3V #PWR03
 U 1 1 5E544AF2
 P 4650 5100
-F 0 "#PWR?" H 4650 4950 50  0001 C CNN
+F 0 "#PWR03" H 4650 4950 50  0001 C CNN
 F 1 "+3.3V" H 4665 5273 50  0000 C CNN
 F 2 "" H 4650 5100 50  0001 C CNN
@@
 Connection ~ 4650 5500
 $Comp
-L power:GND #PWR?
+L power:GND #PWR04
 U 1 1 5E546F66
 P 4650 5900
-F 0 "#PWR?" H 4650 5650 50  0001 C CNN
+F 0 "#PWR04" H 4650 5650 50  0001 C CNN
 F 1 "GND" H 4655 5727 50  0000 C CNN
 F 2 "" H 4650 5900 50  0001 C CNN
@@
 	5950 3600 6100 3600
 $Comp
-L power:GND #PWR?
+L power:GND #PWR06
 U 1 1 5E53D337
 P 5050 3700
-F 0 "#PWR?" H 5050 3450 50  0001 C CNN
+F 0 "#PWR06" H 5050 3450 50  0001 C CNN
 F 1 "GND" H 5055 3527 50  0000 C CNN
 F 2 "" H 5050 3700 50  0001 C CNN
@@
 $EndComp
 $Comp
-L power:+3V3 #PWR?
+L power:+3V3 #PWR05
 U 1 1 5E53C566
 P 5050 3250
-F 0 "#PWR?" H 5050 3100 50  0001 C CNN
+F 0 "#PWR05" H 5050 3100 50  0001 C CNN
 F 1 "+3V3" H 5065 3423 50  0000 C CNN
 F 2 "" H 5050 3250 50  0001 C CNN
@@
 	4750 3400 6100 3400
 $Comp
-L Connector:Conn_01x04_Male J?
+L Connector:Conn_01x04_Male J1
 U 1 1 5E5342FD
 P 4550 3400
-F 0 "J?" H 4658 3681 50  0000 C CNN
+F 0 "J1" H 4658 3681 50  0000 C CNN
 F 1 "Conn_01x04_Male" H 4658 3590 50  0000 C CNN
 F 2 "" H 4550 3400 50  0001 C CNN
@@
 	1250 5300 1450 5300
 $Comp
-L power:GND #PWR?
+L power:GND #PWR01
 U 1 1 5E5B9E4D
 P 2100 5600
-F 0 "#PWR?" H 2100 5350 50  0001 C CNN
+F 0 "#PWR01" H 2100 5350 50  0001 C CNN
 F 1 "GND" H 2105 5427 50  0000 C CNN
 F 2 "" H 2100 5600 50  0001 C CNN
@@
 	2100 5100 2450 5100
 $Comp
-L Device:R_US R?
+L Device:R_US R1
 U 1 1 5E5C636B
 P 1600 5300
-F 0 "R?" V 1395 5300 50  0000 C CNN
+F 0 "R1" V 1395 5300 50  0000 C CNN
 F 1 "1k" V 1486 5300 50  0000 C CNN
 F 2 "" V 1640 5290 50  0001 C CNN
@@
 $EndComp
 $Comp
-L Transistor_FET:BSS138 Q?
+L Transistor_FET:BSS138 Q1
 U 1 1 5E5FD8D0
 P 2000 5300
-F 0 "Q?" H 2204 5346 50  0000 L CNN
+F 0 "Q1" H 2204 5346 50  0000 L CNN
 F 1 "BSS138" H 2204 5255 50  0000 L CNN
 F 2 "Package_TO_SOT_SMD:SOT-23" H 2200 5225 50  0001 L CIN
@@
 	1750 5300 1800 5300
 $Comp
-L Device:R_US R?
+L Device:R_US R2
 U 1 1 5E61BC5D
 P 1750 5450
-F 0 "R?" H 1818 5496 50  0000 L CNN
+F 0 "R2" H 1818 5496 50  0000 L CNN
 F 1 "1M" H 1818 5405 50  0000 L CNN
 F 2 "" V 1790 5440 50  0001 C CNN
@@
 BUZZER
 $Comp
-L power:+5V #PWR?
+L power:+5V #PWR02
 U 1 1 5E5E56E5
 P 2450 4800
-F 0 "#PWR?" H 2450 4650 50  0001 C CNN
+F 0 "#PWR02" H 2450 4650 50  0001 C CNN
 F 1 "+5V" H 2465 4973 50  0000 C CNN
 F 2 "" H 2450 4800 50  0001 C CNN
@@
 	1    0    0    -1
 $EndComp
+Text Notes 2850 4200 0    50   ~ 0
+Add rotary switch. Figure out what it does.
 $EndSCHEMATC

Commit message: Added footprints.
Added footprints for various parts. Still need to update some more and calculate some values.
Parts:
- C1, C2, C3, C4, C5, C6, C7, C8, C9: footprint (none) -> Capacitor_SMD:C_0603_1608Metric
- R1, R2, R3, R4: footprint (none) -> Resistor_SMD:R_0603_1608Metric
Other:
- note added: "UART header"
Changed lines of the file:
@@
 F 0 "C2" H 5515 2896 50  0000 L CNN
 F 1 "22p" H 5515 2805 50  0000 L CNN
-F 2 "" H 5438 2700 50  0001 C CNN
+F 2 "Capacitor_SMD:C_0603_1608Metric" H 5438 2700 50  0001 C CNN
 F 3 "~" H 5400 2850 50  0001 C CNN
 	1    5400 2850
@@
 F 0 "C1" H 5115 2896 50  0000 L CNN
 F 1 "22p" H 5115 2805 50  0000 L CNN
-F 2 "" H 5038 2700 50  0001 C CNN
+F 2 "Capacitor_SMD:C_0603_1608Metric" H 5038 2700 50  0001 C CNN
 F 3 "~" H 5000 2850 50  0001 C CNN
 	1    5000 2850
@@
 F 0 "C9" V 7198 1950 50  0000 C CNN
 F 1 "1u" V 7289 1950 50  0000 C CNN
-F 2 "" H 7488 1800 50  0001 C CNN
+F 2 "Capacitor_SMD:C_0603_1608Metric" H 7488 1800 50  0001 C CNN
 F 3 "~" H 7450 1950 50  0001 C CNN
 	1    7450 1950
@@
 F 0 "C7" V 7198 1050 50  0000 C CNN
 F 1 "10u" V 7289 1050 50  0000 C CNN
-F 2 "" H 7488 900 50  0001 C CNN
+F 2 "Capacitor_SMD:C_0603_1608Metric" H 7488 900 50  0001 C CNN
 F 3 "~" H 7450 1050 50  0001 C CNN
 	1    7450 1050
@@
 F 0 "C8" V 7198 1500 50  0000 C CNN
 F 1 "100n" V 7289 1500 50  0000 C CNN
-F 2 "" H 7488 1350 50  0001 C CNN
+F 2 "Capacitor_SMD:C_0603_1608Metric" H 7488 1350 50  0001 C CNN
 F 3 "~" H 7450 1500 50  0001 C CNN
 	1    7450 1500
@@
 F 0 "C6" V 6498 1950 50  0000 C CNN
 F 1 "100n" V 6589 1950 50  0000 C CNN
-F 2 "" H 6788 1800 50  0001 C CNN
+F 2 "Capacitor_SMD:C_0603_1608Metric" H 6788 1800 50  0001 C CNN
 F 3 "~" H 6750 1950 50  0001 C CNN
 	1    6750 1950
@@
 F 0 "C5" V 6498 1500 50  0000 C CNN
 F 1 "100n" V 6589 1500 50  0000 C CNN
-F 2 "" H 6788 1350 50  0001 C CNN
+F 2 "Capacitor_SMD:C_0603_1608Metric" H 6788 1350 50  0001 C CNN
 F 3 "~" H 6750 1500 50  0001 C CNN
 	1    6750 1500
@@
 F 0 "C4" H 6415 1796 50  0000 L CNN
 F 1 "10u" H 6415 1705 50  0000 L CNN
-F 2 "" H 6338 1600 50  0001 C CNN
+F 2 "Capacitor_SMD:C_0603_1608Metric" H 6338 1600 50  0001 C CNN
 F 3 "~" H 6300 1750 50  0001 C CNN
 	1    6300 1750
@@
 F 0 "C3" H 6115 6396 50  0000 L CNN
 F 1 "100n" H 6115 6305 50  0000 L CNN
-F 2 "" H 6038 6200 50  0001 C CNN
+F 2 "Capacitor_SMD:C_0603_1608Metric" H 6038 6200 50  0001 C CNN
 F 3 "~" H 6000 6350 50  0001 C CNN
 	1    6000 6350
@@
 F 0 "R4" H 6068 6046 50  0000 L CNN
 F 1 "10k" H 6068 5955 50  0000 L CNN
-F 2 "" V 6040 5990 50  0001 C CNN
+F 2 "Resistor_SMD:R_0603_1608Metric" V 6040 5990 50  0001 C CNN
 F 3 "~" H 6000 6000 50  0001 C CNN
 	1    6000 6000
@@
 F 0 "R3" V 5445 6150 50  0000 C CNN
 F 1 "330" V 5536 6150 50  0000 C CNN
-F 2 "" V 5690 6140 50  0001 C CNN
+F 2 "Resistor_SMD:R_0603_1608Metric" V 5690 6140 50  0001 C CNN
 F 3 "~" H 5650 6150 50  0001 C CNN
 	1    5650 6150
@@
 F 0 "R1" V 1395 5300 50  0000 C CNN
 F 1 "1k" V 1486 5300 50  0000 C CNN
-F 2 "" V 1640 5290 50  0001 C CNN
+F 2 "Resistor_SMD:R_0603_1608Metric" V 1640 5290 50  0001 C CNN
 F 3 "~" H 1600 5300 50  0001 C CNN
 	1    1600 5300
@@
 F 0 "R2" H 1818 5496 50  0000 L CNN
 F 1 "1M" H 1818 5405 50  0000 L CNN
-F 2 "" V 1790 5440 50  0001 C CNN
+F 2 "Resistor_SMD:R_0603_1608Metric" V 1790 5440 50  0001 C CNN
 F 3 "~" H 1750 5450 50  0001 C CNN
 	1    1750 5450
@@
 Text Notes 2850 4200 0    50   ~ 0
 Add rotary switch. Figure out what it does.
+Text Notes 4400 3050 0    50   ~ 0
+UART header
 $EndSCHEMATC

Commit message: Drew up power supply, test points; reworked MCU I/O
Parts:
- added C? (x2): 2.2u, symbol Device:C
- added D?: LED, symbol Device:LED
- added J?: Conn_01x02, symbol Connector_Generic:Conn_01x02
- added R?: 1k, symbol Device:R
- added SW?: SW_SPDT, symbol Switch:SW_SPDT
- added TP? (x5): TestPoint, symbol Connector:TestPoint
- added TP?: Espirus-misosu, symbol Connector:TestPoint
- added TP?: Espirus-mosi, symbol Connector:TestPoint
- added TP?: Espirus-chronos, symbol Connector:TestPoint
- added TP?: Radius-selectae, symbol Connector:TestPoint
- added TP?: Radius-reseta, symbol Connector:TestPoint
- added TP?: Radius-interruptus, symbol Connector:TestPoint
- added TP?: Sandiscus-selectae, symbol Connector:TestPoint
- added TP?: Etusi-sidae, symbol Connector:TestPoint
- added TP?: Etusi-chronos, symbol Connector:TestPoint
- added TP?: Emu-reseta, symbol Connector:TestPoint
- added TP?: Emu-interruptus, symbol Connector:TestPoint
- added U?: MIC5528-3.3YMT-TR, Package_TO_SOT_SMD:TDFN-6-1.2x1.2, symbol recovery-custom:MIC5528-3.3YMT-TR
- J2: value Conn_02x05_Odd_Even -> MCU Programming Socket; footprint (none) -> Connector_PinHeader_1.27mm:PinHeader_2x05_P1.27mm_Vertical
Connections:
- net labels added: +BATT
- net labels removed: +5V
- wire segments 102 -> 128
Other:
- note added: "Battery connector"
- note added: "Observe the variegated selection of electroflora \nassembled presently for your viewing edification."
- note added: "Power on/off switch"
- note added: "Power regulator:\nUse low-ESR ceramic capcitors --- \nsee pg. 13 of regulator datasheet."
- note added: "Power-on \nindicator lamp"
- note added: "SERCOM assignments: \nSERCOM0: UART to outside world\n PAD[2] = Tx; PAD[3] = Rx\nSERCOM2: SPI \n PAD[0] = MISO; PAD[2] = MOSI; PAD[3] = CLK\nSERCOM3: I2C\n PAD[0] = SDA; PAD[1] = SCL\n"
- note added: "Test point garden"
- note removed: "Add rotary switch. Figure out what it does."
- note removed: "No, it's not done yet."
