File: Recovery PCB/Recovery PCB.sch (KiCad schematic (older format))
At the start: 45 parts, among them J1 Conn_01x04_Male, J2 MCU Programming Socket, Q1 BSS138, SW1 SW_Push, U1 ATSAMD21G18A-AUT, Y1 32.768kHz

Commit message: Updated some footprints and re-annotated schematic.
Parts:
- C10, C11: renamed from C?; footprint (none) -> Capacitor_SMD:C_0603_1608Metric
- D1: renamed from D?; footprint (none) -> LED_SMD:LED_0603_1608Metric
- R5: renamed from R?; footprint (none) -> Resistor_SMD:R_0603_1608Metric
- gave numbers to parts that had none: 18
Changed lines of the file:
@@
 EESchema Schematic File Version 4
-LIBS:Recovery PCB-cache
-EELAYER 26 0
+EELAYER 30 0
 EELAYER END
 $Descr A4 11693 8268
@@
 $EndComp
 $Comp
-L Device:C C?
+L Device:C C10
 U 1 1 5F00EE93
 P 9000 3200
-F 0 "C?" H 9115 3246 50  0000 L CNN
+F 0 "C10" H 9115 3246 50  0000 L CNN
 F 1 "2.2u" H 9115 3155 50  0000 L CNN
-F 2 "" H 9038 3050 50  0001 C CNN
+F 2 "Capacitor_SMD:C_0603_1608Metric" H 9038 3050 50  0001 C CNN
 F 3 "~" H 9000 3200 50  0001 C CNN
 	1    9000 3200
@@
 $EndComp
 $Comp
-L Device:C C?
+L Device:C C11
 U 1 1 5F00EF43
 P 10350 3200
-F 0 "C?" H 10465 3246 50  0000 L CNN
+F 0 "C11" H 10465 3246 50  0000 L CNN
 F 1 "2.2u" H 10465 3155 50  0000 L CNN
-F 2 "" H 10388 3050 50  0001 C CNN
+F 2 "Capacitor_SMD:C_0603_1608Metric" H 10388 3050 50  0001 C CNN
 F 3 "~" H 10350 3200 50  0001 C CNN
 	1    10350 3200
@@
 Wire Wire Line
 	9350 3050 9350 3250
-Connection ~ 9350 3050
 Wire Wire Line
 	10150 3050 10350 3050
 $Comp
-L power:GND #PWR?
+L power:GND #PWR018
 U 1 1 5F023B13
 P 9750 3450
-F 0 "#PWR?" H 9750 3200 50  0001 C CNN
+F 0 "#PWR018" H 9750 3200 50  0001 C CNN
 F 1 "GND" H 9755 3277 50  0000 C CNN
 F 2 "" H 9750 3450 50  0001 C CNN
@@
 Power regulator:\nUse low-ESR ceramic capcitors --- \nsee pg. 13 of regulator datasheet.
 $Comp
-L power:+3.3V #PWR?
+L power:+3.3V #PWR021
 U 1 1 5F02E217
 P 10350 3050
-F 0 "#PWR?" H 10350 2900 50  0001 C CNN
+F 0 "#PWR021" H 10350 2900 50  0001 C CNN
 F 1 "+3.3V" H 10365 3223 50  0000 C CNN
 F 2 "" H 10350 3050 50  0001 C CNN
@@
 Connection ~ 10350 3050
 $Comp
-L Connector_Generic:Conn_01x02 J?
+L Connector_Generic:Conn_01x02 J3
 U 1 1 5F04A0E6
 P 10350 1900
-F 0 "J?" H 10430 1892 50  0000 L CNN
+F 0 "J3" H 10430 1892 50  0000 L CNN
 F 1 "Conn_01x02" H 10430 1801 50  0000 L CNN
 F 2 "" H 10350 1900 50  0001 C CNN
@@
 $EndComp
 $Comp
-L power:GND #PWR?
+L power:GND #PWR019
 U 1 1 5F04A42B
 P 10150 2000
-F 0 "#PWR?" H 10150 1750 50  0001 C CNN
+F 0 "#PWR019" H 10150 1750 50  0001 C CNN
 F 1 "GND" H 10155 1827 50  0000 C CNN
 F 2 "" H 10150 2000 50  0001 C CNN
@@
 $EndComp
 $Comp
-L power:+BATT #PWR?
+L power:+BATT #PWR017
 U 1 1 5F04A4A2
 P 9500 1800
-F 0 "#PWR?" H 9500 1650 50  0001 C CNN
+F 0 "#PWR017" H 9500 1650 50  0001 C CNN
 F 1 "+BATT" H 9515 1973 50  0000 C CNN
 F 2 "" H 9500 1800 50  0001 C CNN
@@
 $EndComp
 $Comp
-L power:+BATT #PWR?
+L power:+BATT #PWR015
 U 1 1 5F04A512
 P 9100 1900
-F 0 "#PWR?" H 9100 1750 50  0001 C CNN
+F 0 "#PWR015" H 9100 1750 50  0001 C CNN
 F 1 "+BATT" H 9115 2073 50  0000 C CNN
 F 2 "" H 9100 1900 50  0001 C CNN
@@
 $EndComp
 $Comp
-L Device:R R?
+L Device:R R5
 U 1 1 5F04A597
 P 9100 2050
-F 0 "R?" H 9170 2096 50  0000 L CNN
+F 0 "R5" H 9170 2096 50  0000 L CNN
 F 1 "1k" H 9170 2005 50  0000 L CNN
-F 2 "" V 9030 2050 50  0001 C CNN
+F 2 "Resistor_SMD:R_0603_1608Metric" V 9030 2050 50  0001 C CNN
 F 3 "~" H 9100 2050 50  0001 C CNN
 	1    9100 2050
@@
 $EndComp
 $Comp
-L Device:LED D?
+L Device:LED D1
 U 1 1 5F04A679
 P 9100 2350
-F 0 "D?" V 9138 2233 50  0000 R CNN
+F 0 "D1" V 9138 2233 50  0000 R CNN
 F 1 "LED" V 9047 2233 50  0000 R CNN
-F 2 "" H 9100 2350 50  0001 C CNN
+F 2 "LED_SMD:LED_0603_1608Metric" H 9100 2350 50  0001 C CNN
 F 3 "~" H 9100 2350 50  0001 C CNN
 	1    9100 2350
@@
 $EndComp
 $Comp
-L power:GND #PWR?
+L power:GND #PWR016
 U 1 1 5F04A80F
 P 9100 2500
-F 0 "#PWR?" H 9100 2250 50  0001 C CNN
+F 0 "#PWR016" H 9100 2250 50  0001 C CNN
 F 1 "GND" H 9105 2327 50  0000 C CNN
 F 2 "" H 9100 2500 50  0001 C CNN
@@
 Power-on \nindicator lamp
 $Comp
-L power:+BATT #PWR?
+L power:+BATT #PWR014
 U 1 1 5F05E671
 P 9000 3050
-F 0 "#PWR?" H 9000 2900 50  0001 C CNN
+F 0 "#PWR014" H 9000 2900 50  0001 C CNN
 F 1 "+BATT" H 9015 3223 50  0000 C CNN
 F 2 "" H 9000 3050 50  0001 C CNN
@@
 Battery connector
 $Comp
-L Switch:SW_SPDT SW?
+L Switch:SW_SPDT SW2
 U 1 1 5F06332F
 P 9850 1800
-F 0 "SW?" H 9850 2085 50  0000 C CNN
+F 0 "SW2" H 9850 2085 50  0000 C CNN
 F 1 "SW_SPDT" H 9850 1994 50  0000 C CNN
 F 2 "" H 9850 1800 50  0001 C CNN
@@
 	8100 2400 8300 2400
 $Comp
-L Connector:TestPoint TP?
+L Connector:TestPoint TP1
 U 1 1 5F0B5A3F
 P 1250 5450
-F 0 "TP?" H 1192 5477 50  0000 R CNN
+F 0 "TP1" H 1192 5477 50  0000 R CNN
 F 1 "TestPoint" H 1192 5568 50  0000 R CNN
 F 2 "" H 1450 5450 50  0001 C CNN
@@
 	1250 5300 1250 5450
 $Comp
-L power:+3.3V #PWR?
+L power:+3.3V #PWR02
 U 1 1 5F0BABF8
 P 2450 4800
-F 0 "#PWR?" H 2450 4650 50  0001 C CNN
+F 0 "#PWR02" H 2450 4650 50  0001 C CNN
 F 1 "+3.3V" H 2465 4973 50  0000 C CNN
 F 2 "" H 2450 4800 50  0001 C CNN
@@
 $EndComp
 $Comp
-L Connector:TestPoint TP?
+L Connector:TestPoint TP16
 U 1 1 5F0BB8C2
 P 10650 2600
-F 0 "TP?" H 10592 2627 50  0000 R CNN
+F 0 "TP16" H 10592 2627 50  0000 R CNN
 F 1 "TestPoint" H 10592 2718 50  0000 R CNN
 F 2 "" H 10850 2600 50  0001 C CNN
@@
 $EndComp
 $Comp
-L Connector:TestPoint TP?
+L Connector:TestPoint TP12
 U 1 1 5F0C0060
 P 10150 2600
-F 0 "TP?" H 10092 2627 50  0000 R CNN
+F 0 "TP12" H 10092 2627 50  0000 R CNN
 F 1 "TestPoint" H 10092 2718 50  0000 R CNN
 F 2 "" H 10350 2600 50  0001 C CNN
@@
 $EndComp
 $Comp
-L power:+3.3V #PWR?
+L power:+3.3V #PWR020
 U 1 1 5F0C015C
 P 10150 2600
-F 0 "#PWR?" H 10150 2450 50  0001 C CNN
+F 0 "#PWR020" H 10150 2450 50  0001 C CNN
 F 1 "+3.3V" H 10165 2773 50  0000 C CNN
 F 2 "" H 10150 2600 50  0001 C CNN
@@
 $EndComp
 $Comp
-L power:+BATT #PWR?
+L power:+BATT #PWR022
 U 1 1 5F0C0233
 P 10650 2600
-F 0 "#PWR?" H 10650 2450 50  0001 C CNN
+F 0 "#PWR022" H 10650 2450 50  0001 C CNN
 F 1 "+BATT" H 10665 2773 50  0000 C CNN
 F 2 "" H 10650 2600 50  0001 C CNN
@@
 Test point garden
 $Comp
-L Connector:TestPoint TP?
+L Connector:TestPoint TP4
 U 1 1 5F0D38A5
 P 8450 4650
-F 0 "TP?" V 8645 4724 50  0000 C CNN
+F 0 "TP4" V 8645 4724 50  0000 C CNN
 F 1 "Espirus-misosu" V 8554 4724 50  0000 C CNN
 F 2 "" H 8650 4650 50  0001 C CNN
@@
 	5950 5000 6100 5000
 $Comp
-L Connector:TestPoint TP?
+L Connector:TestPoint TP5
 U 1 1 5F0FD40E
 P 8450 4950
-F 0 "TP?" V 8645 5024 50  0000 C CNN
+F 0 "TP5" V 8645 5024 50  0000 C CNN
 F 1 "Espirus-mosi" V 8554 5024 50  0000 C CNN
 F 2 "" H 8650 4950 50  0001 C CNN
@@
 	8450 4950 8700 4950
 $Comp
-L Connector:TestPoint TP?
+L Connector:TestPoint TP6
 U 1 1 5F10B6AA
 P 8450 5250
-F 0 "TP?" V 8645 5324 50  0000 C CNN
+F 0 "TP6" V 8645 5324 50  0000 C CNN
 F 1 "Espirus-chronos" V 8554 5324 50  0000 C CNN
 F 2 "" H 8650 5250 50  0001 C CNN
@@
 	8450 5250 8700 5250
 $Comp
-L Connector:TestPoint TP?
+L Connector:TestPoint TP9
 U 1 1 5F110716
 P 9300 4650
-F 0 "TP?" V 9495 4724 50  0000 C CNN
+F 0 "TP9" V 9495 4724 50  0000 C CNN
 F 1 "Radius-selectae" V 9404 4724 50  0000 C CNN
 F 2 "" H 9500 4650 50  0001 C CNN
@@
 	9300 4650 9550 4650
 $Comp
-L Connector:TestPoint TP?
+L Connector:TestPoint TP10
 U 1 1 5F11071E
 P 9300 4950
-F 0 "TP?" V 9495 5024 50  0000 C CNN
+F 0 "TP10" V 9495 5024 50  0000 C CNN
 F 1 "Radius-reseta" V 9404 5024 50  0000 C CNN
 F 2 "" H 9500 4950 50  0001 C CNN
@@
 	9300 4950 9550 4950
 $Comp
-L Connector:TestPoint TP?
+L Connector:TestPoint TP11
 U 1 1 5F110726
 P 9300 5250
-F 0 "TP?" V 9495 5324 50  0000 C CNN
+F 0 "TP11" V 9495 5324 50  0000 C CNN
 F 1 "Radius-interruptus" V 9404 5324 50  0000 C CNN
 F 2 "" H 9500 5250 50  0001 C CNN
@@
 	9300 5250 9550 5250
 $Comp
-L Connector:TestPoint TP?
+L Connector:TestPoint TP13
 U 1 1 5F12A324
 P 10300 4650
-F 0 "TP?" V 10495 4724 50  0000 C CNN
+F 0 "TP13" V 10495 4724 50  0000 C CNN
 F 1 "Sandiscus-selectae" V 10404 4724 50  0000 C CNN
 F 2 "" H 10500 4650 50  0001 C CNN
@@
 	10300 4650 10550 4650
 $Comp
-L Connector:TestPoint TP?
+L Connector:TestPoint TP7
 U 1 1 5F134E33
 P 8450 5550
-F 0 "TP?" V 8645 5624 50  0000 C CNN
+F 0 "TP7" V 8645 5624 50  0000 C CNN
 F 1 "Etusi-sidae" V 8554 5624 50  0000 C CNN
 F 2 "" H 8650 5550 50  0001 C CNN
@@
 	8450 5550 8700 5550
 $Comp
-L Connector:TestPoint TP?
+L Connector:TestPoint TP8
 U 1 1 5F134E3B
 P 8450 5850
-F 0 "TP?" V 8645 5924 50  0000 C CNN
+F 0 "TP8" V 8645 5924 50  0000 C CNN
 F 1 "Etusi-chronos" V 8554 5924 50  0000 C CNN
 F 2 "" H 8650 5850 50  0001 C CNN
@@
 	8450 5850 8700 5850
 $Comp
-L Connector:TestPoint TP?
+L Connector:TestPoint TP14
 U 1 1 5F14495E
 P 10300 4950
-F 0 "TP?" V 10495 5024 50  0000 C CNN
+F 0 "TP14" V 10495 5024 50  0000 C CNN
 F 1 "Emu-reseta" V 10404 5024 50  0000 C CNN
 F 2 "" H 10500 4950 50  0001 C CNN
@@
 IMU_INT
 $Comp
-L Connector:TestPoint TP?
+L Connector:TestPoint TP15
 U 1 1 5F16BA81
 P 10300 5250
-F 0 "TP?" V 10495 5324 50  0000 C CNN
+F 0 "TP15" V 10495 5324 50  0000 C CNN
 F 1 "Emu-interruptus" V 10404 5324 50  0000 C CNN
 F 2 "" H 10500 5250 50  0001 C CNN
@@
 IMU_INT
 $Comp
-L Connector:TestPoint TP?
+L Connector:TestPoint TP3
 U 1 1 5F1726AB
 P 5600 3400
-F 0 "TP?" H 5658 3520 50  0000 L CNN
+F 0 "TP3" H 5658 3520 50  0000 L CNN
 F 1 "TestPoint" H 5658 3429 50  0000 L CNN
 F 2 "" H 5800 3400 50  0001 C CNN
@@
 	5600 3400 6100 3400
 $Comp
-L Connector:TestPoint TP?
+L Connector:TestPoint TP2
 U 1 1 5F17276B
 P 5250 3500
-F 0 "TP?" H 5192 3527 50  0000 R CNN
+F 0 "TP2" H 5192 3527 50  0000 R CNN
 F 1 "TestPoint" H 5192 3618 50  0000 R CNN
 F 2 "" H 5450 3500 50  0001 C CNN

Commit message: Added missing footprints and replaced GPS module.
Parts:
- BZ1: footprint (none) -> Buzzer_Beeper:Buzzer_TDK_PS1240P02BT_D12.2mm_H6.5mm
- FB1: footprint (none) -> Inductor_SMD:L_0603_1608Metric
- J1: footprint (none) -> Connector_PinHeader_2.54mm:PinHeader_1x04_P2.54mm_Vertical
- J3: footprint (none) -> Connector_JST:JST_XH_B2B-XH-A_1x02_P2.50mm_Vertical
- L1: footprint (none) -> Inductor_SMD:L_1008_2520Metric
- SW1: footprint (none) -> Parts:SW_SPST_PTS815
- SW2: footprint (none) -> Connector_JST:JST_XH_B3B-XH-A_1x03_P2.50mm_Vertical
- Y1: footprint (none) -> Crystal:Crystal_SMD_3215-2Pin_3.2x1.5mm
- gave numbers to parts that had none: 1
Connections:
- wire segments 128 -> 126
- no-connect marks 6 -> 20
Changed lines of the file:
@@
 F 0 "Y1" V 5354 2681 50  0000 L CNN
 F 1 "32.768kHz" V 5445 2681 50  0000 L CNN
-F 2 "" H 5400 2550 50  0001 C CNN
+F 2 "Crystal:Crystal_SMD_3215-2Pin_3.2x1.5mm" H 5400 2550 50  0001 C CNN
 F 3 "~" H 5400 2550 50  0001 C CNN
 	1    5400 2550
@@
 F 0 "SW1" V 5496 6302 50  0000 R CNN
 F 1 "SW_Push" V 5405 6302 50  0000 R CNN
-F 2 "" H 5450 6550 50  0001 C CNN
+F 2 "Parts:SW_SPST_PTS815" H 5450 6550 50  0001 C CNN
 F 3 "" H 5450 6550 50  0001 C CNN
 	1    5450 6350
@@
 F 0 "L1" H 6650 1265 50  0000 C CNN
 F 1 "10uH" H 6650 1174 50  0000 C CNN
-F 2 "" H 6650 1050 50  0001 C CNN
+F 2 "Inductor_SMD:L_1008_2520Metric" H 6650 1050 50  0001 C CNN
 F 3 "~" H 6650 1050 50  0001 C CNN
 	1    6650 1050
@@
 F 0 "FB1" V 6863 1050 50  0000 C CNN
 F 1 "Ferrite_Bead_Small" V 6954 1050 50  0000 C CNN
-F 2 "" V 7030 1050 50  0001 C CNN
+F 2 "Inductor_SMD:L_0603_1608Metric" V 7030 1050 50  0001 C CNN
 F 3 "~" H 7100 1050 50  0001 C CNN
 	1    7100 1050
@@
 F 0 "J1" H 4658 3681 50  0000 C CNN
 F 1 "Conn_01x04_Male" H 4658 3590 50  0000 C CNN
-F 2 "" H 4550 3400 50  0001 C CNN
+F 2 "Connector_PinHeader_2.54mm:PinHeader_1x04_P2.54mm_Vertical" H 4550 3400 50  0001 C CNN
 F 3 "~" H 4550 3400 50  0001 C CNN
 	1    4550 3400
@@
 Wire Wire Line
 	5000 3000 5300 3000
-Text Label 2950 3150 2    50   ~ 0
-SDA
-Text Label 2950 3250 2    50   ~ 0
-SCL
 $Sheet
 S 1450 2650 550  450
@@
 F0 "gps-module" 50
 F1 "gps-module.sch" 50
-F2 "RX" I L 3100 3000 50
-F3 "TX" O L 3100 2900 50
-F4 "GPS_SDA" B L 3100 3150 50
-F5 "GPS_SCL" I L 3100 3250 50
+F2 "GPS_SDA" B L 3100 3150 50
+F3 "GPS_SCL" I L 3100 3250 50
+F4 "~RST" I L 3100 2950 50
 $EndSheet
 Text Label 5950 4900 2    50   ~ 0
@@
 Wire Wire Line
 	5950 4400 6100 4400
-Wire Wire Line
-	3100 2900 2950 2900
-Wire Wire Line
-	3100 3000 2950 3000
-NoConn ~ 2950 2900
-NoConn ~ 2950 3000
 Connection ~ 2100 5600
 Wire Wire Line
@@
 F 0 "BZ1" H 2702 5029 50  0000 L CNN
 F 1 "Buzzer" H 2702 4938 50  0000 L CNN
-F 2 "" V 2525 5100 50  0001 C CNN
+F 2 "Buzzer_Beeper:Buzzer_TDK_PS1240P02BT_D12.2mm_H6.5mm" V 2525 5100 50  0001 C CNN
 F 3 "~" V 2525 5100 50  0001 C CNN
 	1    2550 5000
@@
 Text Notes 4400 3050 0    50   ~ 0
 UART header
-$Comp
-L recovery-custom:MIC5528-3.3YMT-TR U?
-U 1 1 5EFFFA85
-P 9750 3150
-F 0 "U?" H 9750 3517 50  0000 C CNN
-F 1 "MIC5528-3.3YMT-TR" H 9750 3426 50  0000 C CNN
-F 2 "Package_TO_SOT_SMD:TDFN-6-1.2x1.2" H 9750 2750 50  0001 C CNN
-F 3 "http://www.microchip.com/mymicrochip/filehandler.aspx?ddocname=en580311" H 9500 3400 50  0001 C CNN
-	1    9750 3150
-	1    0    0    -1
-$EndComp
 $Comp
 L Device:C C10
@@
 F 0 "J3" H 10430 1892 50  0000 L CNN
 F 1 "Conn_01x02" H 10430 1801 50  0000 L CNN
-F 2 "" H 10350 1900 50  0001 C CNN
+F 2 "Connector_JST:JST_XH_B2B-XH-A_1x02_P2.50mm_Vertical" H 10350 1900 50  0001 C CNN
 F 3 "~" H 10350 1900 50  0001 C CNN
 	1    10350 1900
@@
 F 0 "SW2" H 9850 2085 50  0000 C CNN
 F 1 "SW_SPDT" H 9850 1994 50  0000 C CNN
-F 2 "" H 9850 1800 50  0001 C CNN
+F 2 "Connector_JST:JST_XH_B3B-XH-A_1x03_P2.50mm_Vertical" H 9850 1800 50  0001 C CNN
 F 3 "" H 9850 1800 50  0001 C CNN
 	1    9850 1800
@@
 Text Label 5950 4400 2    50   ~ 0
 SD_CS
-Wire Wire Line
-	8100 2400 8300 2400
 $Comp
 L Connector:TestPoint TP1
@@
 Text Notes 9150 5600 0    50   ~ 0
 Observe the variegated selection of electroflora \nassembled presently for your viewing edification.
+NoConn ~ 6100 2600
+NoConn ~ 6100 2700
+NoConn ~ 6100 2800
+NoConn ~ 6100 3200
+NoConn ~ 6100 3300
+NoConn ~ 6100 3700
+NoConn ~ 6100 4300
+NoConn ~ 6100 4500
+NoConn ~ 6100 4800
+NoConn ~ 8100 2500
+NoConn ~ 8100 2600
+NoConn ~ 8100 2700
+NoConn ~ 8100 3000
+NoConn ~ 8100 3100
+Text Label 2950 3250 2    50   ~ 0
+SCL
+Text Label 2950 3150 2    50   ~ 0
+SDA
+NoConn ~ 8100 2400
+Wire Wire Line
+	3100 2950 2950 2950
+NoConn ~ 2950 2950
+$Comp
+L recovery-custom:MIC5528-3.3YMT-TR U2
+U 1 1 5EFFFA85
+P 9750 3150
+F 0 "U2" H 9750 3517 50  0000 C CNN
+F 1 "MIC5528-3.3YMT-TR" H 9750 3426 50  0000 C CNN
+F 2 "Package_TO_SOT_SMD:TDFN-6-1.2x1.2" H 9750 2750 50  0001 C CNN
+F 3 "http://www.microchip.com/mymicrochip/filehandler.aspx?ddocname=en580311" H 9500 3400 50  0001 C CNN
+	1    9750 3150
+	1    0    0    -1
+$EndComp
 $EndSCHEMATC

Commit message: Finished Revision 1 of the Recovery PCB.
Parts:
- TP1, TP10, TP11, TP12, TP13, TP14, TP15, TP16, TP2, TP3, TP4, TP5, TP6, TP7, TP8, TP9: footprint (none) -> TestPoint:TestPoint_Pad_D1.0mm
- U2: footprint Package_TO_SOT_SMD:TDFN-6-1.2x1.2 -> Package_DFN_QFN:DFN-6-1EP_1.2x1.2mm_P0.4mm_EP0.3x0.94mm_PullBack
Changed lines of the file:
@@
 Text Label 1250 5300 2    50   ~ 0
 BUZZER
-$Comp
-L Device:Buzzer BZ1
-U 1 1 5DEFD3F0
-P 2550 5000
-F 0 "BZ1" H 2702 5029 50  0000 L CNN
-F 1 "Buzzer" H 2702 4938 50  0000 L CNN
-F 2 "Buzzer_Beeper:Buzzer_TDK_PS1240P02BT_D12.2mm_H6.5mm" V 2525 5100 50  0001 C CNN
-F 3 "~" V 2525 5100 50  0001 C CNN
-	1    2550 5000
-	1    0    0    -1
-$EndComp
 Text Notes 4400 3050 0    50   ~ 0
 UART header
@@
 F 0 "TP1" H 1192 5477 50  0000 R CNN
 F 1 "TestPoint" H 1192 5568 50  0000 R CNN
-F 2 "" H 1450 5450 50  0001 C CNN
+F 2 "TestPoint:TestPoint_Pad_D1.0mm" H 1450 5450 50  0001 C CNN
 F 3 "~" H 1450 5450 50  0001 C CNN
 	1    1250 5450
@@
 F 0 "TP16" H 10592 2627 50  0000 R CNN
 F 1 "TestPoint" H 10592 2718 50  0000 R CNN
-F 2 "" H 10850 2600 50  0001 C CNN
+F 2 "TestPoint:TestPoint_Pad_D1.0mm" H 10850 2600 50  0001 C CNN
 F 3 "~" H 10850 2600 50  0001 C CNN
 	1    10650 2600
@@
 F 0 "TP12" H 10092 2627 50  0000 R CNN
 F 1 "TestPoint" H 10092 2718 50  0000 R CNN
-F 2 "" H 10350 2600 50  0001 C CNN
+F 2 "TestPoint:TestPoint_Pad_D1.0mm" H 10350 2600 50  0001 C CNN
 F 3 "~" H 10350 2600 50  0001 C CNN
 	1    10150 2600
@@
 F 0 "TP4" V 8645 4724 50  0000 C CNN
 F 1 "Espirus-misosu" V 8554 4724 50  0000 C CNN
-F 2 "" H 8650 4650 50  0001 C CNN
+F 2 "TestPoint:TestPoint_Pad_D1.0mm" H 8650 4650 50  0001 C CNN
 F 3 "~" H 8650 4650 50  0001 C CNN
 	1    8450 4650
@@
 F 0 "TP5" V 8645 5024 50  0000 C CNN
 F 1 "Espirus-mosi" V 8554 5024 50  0000 C CNN
-F 2 "" H 8650 4950 50  0001 C CNN
+F 2 "TestPoint:TestPoint_Pad_D1.0mm" H 8650 4950 50  0001 C CNN
 F 3 "~" H 8650 4950 50  0001 C CNN
 	1    8450 4950
@@
 F 0 "TP6" V 8645 5324 50  0000 C CNN
 F 1 "Espirus-chronos" V 8554 5324 50  0000 C CNN
-F 2 "" H 8650 5250 50  0001 C CNN
+F 2 "TestPoint:TestPoint_Pad_D1.0mm" H 8650 5250 50  0001 C CNN
 F 3 "~" H 8650 5250 50  0001 C CNN
 	1    8450 5250
@@
 F 0 "TP9" V 9495 4724 50  0000 C CNN
 F 1 "Radius-selectae" V 9404 4724 50  0000 C CNN
-F 2 "" H 9500 4650 50  0001 C CNN
+F 2 "TestPoint:TestPoint_Pad_D1.0mm" H 9500 4650 50  0001 C CNN
 F 3 "~" H 9500 4650 50  0001 C CNN
 	1    9300 4650
@@
 F 0 "TP10" V 9495 5024 50  0000 C CNN
 F 1 "Radius-reseta" V 9404 5024 50  0000 C CNN
-F 2 "" H 9500 4950 50  0001 C CNN
+F 2 "TestPoint:TestPoint_Pad_D1.0mm" H 9500 4950 50  0001 C CNN
 F 3 "~" H 9500 4950 50  0001 C CNN
 	1    9300 4950
@@
 F 0 "TP11" V 9495 5324 50  0000 C CNN
 F 1 "Radius-interruptus" V 9404 5324 50  0000 C CNN
-F 2 "" H 9500 5250 50  0001 C CNN
+F 2 "TestPoint:TestPoint_Pad_D1.0mm" H 9500 5250 50  0001 C CNN
 F 3 "~" H 9500 5250 50  0001 C CNN
 	1    9300 5250
@@
 F 0 "TP13" V 10495 4724 50  0000 C CNN
 F 1 "Sandiscus-selectae" V 10404 4724 50  0000 C CNN
-F 2 "" H 10500 4650 50  0001 C CNN
+F 2 "TestPoint:TestPoint_Pad_D1.0mm" H 10500 4650 50  0001 C CNN
 F 3 "~" H 10500 4650 50  0001 C CNN
 	1    10300 4650
@@
 F 0 "TP7" V 8645 5624 50  0000 C CNN
 F 1 "Etusi-sidae" V 8554 5624 50  0000 C CNN
-F 2 "" H 8650 5550 50  0001 C CNN
+F 2 "TestPoint:TestPoint_Pad_D1.0mm" H 8650 5550 50  0001 C CNN
 F 3 "~" H 8650 5550 50  0001 C CNN
 	1    8450 5550
@@
 F 0 "TP8" V 8645 5924 50  0000 C CNN
 F 1 "Etusi-chronos" V 8554 5924 50  0000 C CNN
-F 2 "" H 8650 5850 50  0001 C CNN
+F 2 "TestPoint:TestPoint_Pad_D1.0mm" H 8650 5850 50  0001 C CNN
 F 3 "~" H 8650 5850 50  0001 C CNN
 	1    8450 5850
@@
 F 0 "TP14" V 10495 5024 50  0000 C CNN
 F 1 "Emu-reseta" V 10404 5024 50  0000 C CNN
-F 2 "" H 10500 4950 50  0001 C CNN
+F 2 "TestPoint:TestPoint_Pad_D1.0mm" H 10500 4950 50  0001 C CNN
 F 3 "~" H 10500 4950 50  0001 C CNN
 	1    10300 4950
@@
 F 0 "TP15" V 10495 5324 50  0000 C CNN
 F 1 "Emu-interruptus" V 10404 5324 50  0000 C CNN
-F 2 "" H 10500 5250 50  0001 C CNN
+F 2 "TestPoint:TestPoint_Pad_D1.0mm" H 10500 5250 50  0001 C CNN
 F 3 "~" H 10500 5250 50  0001 C CNN
 	1    10300 5250
@@
 F 0 "TP3" H 5658 3520 50  0000 L CNN
 F 1 "TestPoint" H 5658 3429 50  0000 L CNN
-F 2 "" H 5800 3400 50  0001 C CNN
+F 2 "TestPoint:TestPoint_Pad_D1.0mm" H 5800 3400 50  0001 C CNN
 F 3 "~" H 5800 3400 50  0001 C CNN
 	1    5600 3400
@@
 F 0 "TP2" H 5192 3527 50  0000 R CNN
 F 1 "TestPoint" H 5192 3618 50  0000 R CNN
-F 2 "" H 5450 3500 50  0001 C CNN
+F 2 "TestPoint:TestPoint_Pad_D1.0mm" H 5450 3500 50  0001 C CNN
 F 3 "~" H 5450 3500 50  0001 C CNN
 	1    5250 3500
@@
 F 0 "U2" H 9750 3517 50  0000 C CNN
 F 1 "MIC5528-3.3YMT-TR" H 9750 3426 50  0000 C CNN
-F 2 "Package_TO_SOT_SMD:TDFN-6-1.2x1.2" H 9750 2750 50  0001 C CNN
+F 2 "Package_DFN_QFN:DFN-6-1EP_1.2x1.2mm_P0.4mm_EP0.3x0.94mm_PullBack" H 9750 2750 50  0001 C CNN
 F 3 "http://www.microchip.com/mymicrochip/filehandler.aspx?ddocname=en580311" H 9500 3400 50  0001 C CNN
 	1    9750 3150
 	1    0    0    -1
 $EndComp
+$Comp
+L Device:Buzzer BZ1
+U 1 1 5DEFD3F0
+P 2550 5000
+F 0 "BZ1" H 2702 5029 50  0000 L CNN
+F 1 "Buzzer" H 2702 4938 50  0000 L CNN
+F 2 "Buzzer_Beeper:Buzzer_TDK_PS1240P02BT_D12.2mm_H6.5mm" V 2525 5100 50  0001 C CNN
+F 3 "~" V 2525 5100 50  0001 C CNN
+	1    2550 5000
+	1    0    0    -1
+$EndComp

Commit message: Finished Rev 2 of the Recovery PCB. Optimized trace lengths and relays.
Parts:
- removed R1: 1k, Resistor_SMD:R_0603_1608Metric, symbol Device:R_US
Changed lines of the file:
@@
 Wire Wire Line
 	5950 4400 6100 4400
-Connection ~ 2100 5600
-Wire Wire Line
-	1750 5600 2100 5600
-Connection ~ 1750 5300
-Wire Wire Line
-	1250 5300 1450 5300
-$Comp
-L power:GND #PWR01
-U 1 1 5E5B9E4D
-P 2100 5600
-F 0 "#PWR01" H 2100 5350 50  0001 C CNN
-F 1 "GND" H 2105 5427 50  0000 C CNN
-F 2 "" H 2100 5600 50  0001 C CNN
-F 3 "" H 2100 5600 50  0001 C CNN
-	1    2100 5600
-	1    0    0    -1
-$EndComp
-Wire Wire Line
-	2100 5100 2450 5100
-$Comp
-L Device:R_US R1
-U 1 1 5E5C636B
-P 1600 5300
-F 0 "R1" V 1395 5300 50  0000 C CNN
-F 1 "1k" V 1486 5300 50  0000 C CNN
-F 2 "Resistor_SMD:R_0603_1608Metric" V 1640 5290 50  0001 C CNN
-F 3 "~" H 1600 5300 50  0001 C CNN
-	1    1600 5300
-	0    1    1    0
-$EndComp
-$Comp
-L Transistor_FET:BSS138 Q1
-U 1 1 5E5FD8D0
-P 2000 5300
-F 0 "Q1" H 2204 5346 50  0000 L CNN
-F 1 "BSS138" H 2204 5255 50  0000 L CNN
-F 2 "Package_TO_SOT_SMD:SOT-23" H 2200 5225 50  0001 L CIN
-F 3 "https://www.onsemi.com/pub/Collateral/BSS138-D.PDF" H 2000 5300 50  0001 L CNN
-	1    2000 5300
-	1    0    0    -1
-$EndComp
-Wire Wire Line
-	2100 5500 2100 5600
-Wire Wire Line
-	1750 5300 1800 5300
-$Comp
-L Device:R_US R2
-U 1 1 5E61BC5D
-P 1750 5450
-F 0 "R2" H 1818 5496 50  0000 L CNN
-F 1 "1M" H 1818 5405 50  0000 L CNN
-F 2 "Resistor_SMD:R_0603_1608Metric" V 1790 5440 50  0001 C CNN
-F 3 "~" H 1750 5450 50  0001 C CNN
-	1    1750 5450
-	1    0    0    -1
-$EndComp
 Wire Wire Line
 	2450 4900 2450 4800
@@
 	1    0    0    -1
 $EndComp
+Connection ~ 1750 5300
+Wire Wire Line
+	1250 5300 1750 5300
 $Comp
 L Device:Buzzer BZ1
@@
 	1    0    0    -1
 $EndComp
+$Comp
+L Device:R_US R2
+U 1 1 5E61BC5D
+P 1750 5450
+F 0 "R2" H 1818 5496 50  0000 L CNN
+F 1 "1M" H 1818 5405 50  0000 L CNN
+F 2 "Resistor_SMD:R_0603_1608Metric" V 1790 5440 50  0001 C CNN
+F 3 "~" H 1750 5450 50  0001 C CNN
+	1    1750 5450
+	1    0    0    -1
+$EndComp
+Wire Wire Line
+	1750 5300 1800 5300
+Wire Wire Line
+	2100 5500 2100 5600
+$Comp
+L Transistor_FET:BSS138 Q1
+U 1 1 5E5FD8D0
+P 2000 5300
+F 0 "Q1" H 2204 5346 50  0000 L CNN
+F 1 "BSS138" H 2204 5255 50  0000 L CNN
+F 2 "Package_TO_SOT_SMD:SOT-23" H 2200 5225 50  0001 L CIN
+F 3 "https://www.onsemi.com/pub/Collateral/BSS138-D.PDF" H 2000 5300 50  0001 L CNN
+	1    2000 5300
+	1    0    0    -1
+$EndComp
+Wire Wire Line
+	2100 5100 2450 5100
+$Comp
+L power:GND #PWR01
+U 1 1 5E5B9E4D
+P 2100 5600
+F 0 "#PWR01" H 2100 5350 50  0001 C CNN
+F 1 "GND" H 2105 5427 50  0000 C CNN
+F 2 "" H 2100 5600 50  0001 C CNN
+F 3 "" H 2100 5600 50  0001 C CNN
+	1    2100 5600
+	1    0    0    -1
+$EndComp
+Wire Wire Line
+	1750 5600 2100 5600
+Connection ~ 2100 5600
 $EndSCHEMATC
