File: Recovery PCB/Recovery PCB.sch (KiCad schematic (older format))
At the start: 44 parts, among them J1 Conn_01x04_Male, J2 MCU Programming Socket, J3 Conn_01x02, Q1 BSS138, SW1 SW_Push, SW2 SW_SPDT, U1 ATSAMD21G18A-AUT, U2 MIC5528-3.3YMT-TR, Y1 32.768kHz

Commit message: Recovery PCB: Redraw schematics
Redrew Recover PCB schematics to be more easily readable and fixed board
outline, adding netclasses to ease trace placement.
Parts:
- FB1: value Ferrite_Bead_Small -> Ferrite
Connections:
- wire segments 126 -> 123

Commit message: Rev 3 of Recovery PCB. Fixed decoupling caps and finalized power/ground.
Parts:
- C4, C7: footprint Capacitor_SMD:C_0603_1608Metric -> Capacitor_SMD:C_0805_2012Metric
Changed lines of the file:
@@
 F 0 "C7" H 8000 1550 50  0000 C CNN
 F 1 "10u" H 8000 1450 50  0000 C CNN
-F 2 "Capacitor_SMD:C_0603_1608Metric" H 8238 1400 50  0001 C CNN
+F 2 "Capacitor_SMD:C_0805_2012Metric" H 8238 1400 50  0001 C CNN
 F 3 "~" H 8200 1550 50  0001 C CNN
 	1    8200 1550
@@
 F 0 "C4" H 6250 1650 50  0000 L CNN
 F 1 "10u" H 6250 1550 50  0000 L CNN
-F 2 "Capacitor_SMD:C_0603_1608Metric" H 6188 1500 50  0001 C CNN
+F 2 "Capacitor_SMD:C_0805_2012Metric" H 6188 1500 50  0001 C CNN
 F 3 "~" H 6150 1650 50  0001 C CNN
 	1    6150 1650

Commit message: Recovery PCB: Optimize space
Reduced board space by shifting layout a bit.
Parts:
- removed TP2, TP3: TestPoint, TestPoint:TestPoint_Pad_D1.0mm, symbol Connector:TestPoint
- added C?: 100n, Capacitor_SMD:C_0603_1608Metric, symbol Device:C
Connections:
- net labels added: UART_RX, UART_TX
- wire segments 123 -> 122
Changed lines of the file:
@@
 L Device:C C6
 U 1 1 5E2E3FFA
-P 6450 1650
-F 0 "C6" H 6300 1650 50  0000 C CNN
-F 1 "100n" H 6300 1550 50  0000 C CNN
-F 2 "Capacitor_SMD:C_0603_1608Metric" H 6488 1500 50  0001 C CNN
-F 3 "~" H 6450 1650 50  0001 C CNN
-	1    6450 1650
+P 6150 1650
+F 0 "C6" H 6000 1650 50  0000 C CNN
+F 1 "100n" H 6000 1550 50  0000 C CNN
+F 2 "Capacitor_SMD:C_0603_1608Metric" H 6188 1500 50  0001 C CNN
+F 3 "~" H 6150 1650 50  0001 C CNN
+	1    6150 1650
 	1    0    0    -1
 $EndComp
@@
 L Device:C C4
 U 1 1 5E2E7512
-P 6150 1650
-F 0 "C4" H 6250 1650 50  0000 L CNN
-F 1 "10u" H 6250 1550 50  0000 L CNN
-F 2 "Capacitor_SMD:C_0805_2012Metric" H 6188 1500 50  0001 C CNN
-F 3 "~" H 6150 1650 50  0001 C CNN
-	1    6150 1650
+P 5850 1650
+F 0 "C4" H 5950 1650 50  0000 L CNN
+F 1 "10u" H 5950 1550 50  0000 L CNN
+F 2 "Capacitor_SMD:C_0805_2012Metric" H 5888 1500 50  0001 C CNN
+F 3 "~" H 5850 1650 50  0001 C CNN
+	1    5850 1650
 	-1   0    0    -1
 $EndComp
@@
 Wire Wire Line
 	4750 3300 5050 3300
-Wire Wire Line
-	6100 3500 5250 3500
-Wire Wire Line
-	4750 3400 5250 3400
 $Comp
 L Connector:Conn_01x04_Male J1
@@
 Text Label 10550 5250 0    50   ~ 0
 IMU_INT
-$Comp
-L Connector:TestPoint TP3
-U 1 1 5F1726AB
-P 5250 3400
-F 0 "TP3" H 5308 3520 50  0000 L CNN
-F 1 "TestPoint" H 5308 3429 50  0000 L CNN
-F 2 "TestPoint:TestPoint_Pad_D1.0mm" H 5450 3400 50  0001 C CNN
-F 3 "~" H 5450 3400 50  0001 C CNN
-	1    5250 3400
-	1    0    0    -1
-$EndComp
-$Comp
-L Connector:TestPoint TP2
-U 1 1 5F17276B
-P 5250 3500
-F 0 "TP2" H 5192 3527 50  0000 R CNN
-F 1 "TestPoint" H 5192 3618 50  0000 R CNN
-F 2 "TestPoint:TestPoint_Pad_D1.0mm" H 5450 3500 50  0001 C CNN
-F 3 "~" H 5450 3500 50  0001 C CNN
-	1    5250 3500
-	-1   0    0    1
-$EndComp
-Connection ~ 5250 3500
-Wire Wire Line
-	5250 3500 4750 3500
 Text Notes 9150 5600 0    50   ~ 0
 Observe the variegated selection of electroflora \nassembled presently for your viewing edification.
@@
 	5250 2400 5400 2400
 Connection ~ 5400 2400
-Connection ~ 5250 3400
-Wire Wire Line
-	5250 3400 6100 3400
 $Comp
 L power:+3.3V #PWR08
@@
 L power:GND #PWR0120
 U 1 1 601D693E
-P 6450 1800
-F 0 "#PWR0120" H 6450 1550 50  0001 C CNN
-F 1 "GND" H 6455 1627 50  0000 C CNN
-F 2 "" H 6450 1800 50  0001 C CNN
-F 3 "" H 6450 1800 50  0001 C CNN
-	1    6450 1800
-	1    0    0    -1
-$EndComp
-Wire Wire Line
-	6750 1500 6900 1500
-Wire Wire Line
-	6900 1500 6900 2100
-$Comp
-L power:GND #PWR0121
-U 1 1 60212EB4
 P 6150 1800
-F 0 "#PWR0121" H 6150 1550 50  0001 C CNN
+F 0 "#PWR0120" H 6150 1550 50  0001 C CNN
 F 1 "GND" H 6155 1627 50  0000 C CNN
 F 2 "" H 6150 1800 50  0001 C CNN
 F 3 "" H 6150 1800 50  0001 C CNN
 	1    6150 1800
+	1    0    0    -1
+$EndComp
+Wire Wire Line
+	6750 1500 6900 1500
+Wire Wire Line
+	6900 1500 6900 2100
+$Comp
+L power:GND #PWR0121
+U 1 1 60212EB4
+P 5850 1800
+F 0 "#PWR0121" H 5850 1550 50  0001 C CNN
+F 1 "GND" H 5855 1627 50  0000 C CNN
+F 2 "" H 5850 1800 50  0001 C CNN
+F 3 "" H 5850 1800 50  0001 C CNN
+	1    5850 1800
 	1    0    0    -1
 $EndComp
@@
 	7000 1350 7000 1400
 Wire Wire Line
+	5850 1500 5850 1400
+Wire Wire Line
 	6150 1500 6150 1400
-Connection ~ 6900 1400
-Wire Wire Line
-	6450 1500 6450 1400
-Connection ~ 6450 1400
-Wire Wire Line
-	6450 1400 6900 1400
-Wire Wire Line
-	6150 1400 6450 1400
+Connection ~ 6150 1400
+Wire Wire Line
+	5850 1400 6150 1400
 Wire Wire Line
 	7000 1400 7000 2100
@@
 	950  5300 1250 5300
 Connection ~ 1250 5300
+Wire Wire Line
+	4750 3400 6100 3400
+Wire Wire Line
+	4750 3500 6100 3500
+Text Label 5100 3400 0    50   ~ 0
+UART_TX
+Text Label 5100 3500 0    50   ~ 0
+UART_RX
+$Comp
+L power:GND #PWR?
+U 1 1 601436A5
+P 6450 1800
+F 0 "#PWR?" H 6450 1550 50  0001 C CNN
+F 1 "GND" H 6455 1627 50  0000 C CNN
+F 2 "" H 6450 1800 50  0001 C CNN
+F 3 "" H 6450 1800 50  0001 C CNN
+	1    6450 1800
+	1    0    0    -1
+$EndComp
+$Comp
+L Device:C C?
+U 1 1 601436AB
+P 6450 1650
+F 0 "C?" H 6300 1650 50  0000 C CNN
+F 1 "100n" H 6300 1750 50  0000 C CNN
+F 2 "Capacitor_SMD:C_0603_1608Metric" H 6488 1500 50  0001 C CNN
+F 3 "~" H 6450 1650 50  0001 C CNN
+	1    6450 1650
+	1    0    0    1
+$EndComp
+Wire Wire Line
+	6150 1400 6900 1400
+Connection ~ 6900 1400
+Wire Wire Line
+	6450 1500 6750 1500
+Connection ~ 6750 1500
 $EndSCHEMATC

Commit message: Recovery PCB: Reannotate
Reannotated schematic to fix reference numbering and keep reference
designators consistent.
Parts:
- gave numbers to parts that had none: 1
- renumbered C8 to C1, C3 to C12, C7 to C2, C4 to C3, C6 to C4, C5 to C6, C9 to C7, C1 to C8, C2 to C9, J3 to J1, J1 to J2, J2 to J3, R5 to R1, R4 to R3, R3 to R4, SW2 to SW1, SW1 to SW2, TP12 to TP1, TP11 to TP10, TP15 to TP11, TP1 to TP12, TP7 to TP13, TP8 to TP14, TP16 to TP2, TP4 to TP3, TP9 to TP4, TP13 to TP5, TP5 to TP6, TP10 to TP7, TP14 to TP8, TP6 to TP9, U2 to U1, U1 to U2

Commit message: Recovery PCB: Fix relay
Replaced unavailable relay with a correct part and replaced voltage
regulator with an easier to solder alternative.
Parts:
- C10, C11: value 2.2u -> 1u
- U1: value MIC5528-3.3YMT-TR -> AP7366-33W5-7; footprint Package_DFN_QFN:DFN-6-1EP_1.2x1.2mm_P0.4mm_EP0.3x0.94mm_PullBack -> Package_TO_SOT_SMD:SOT-23-5; symbol recovery-custom:MIC5528-3.3YMT-TR -> recovery-custom:AP7366-33W5-7
Connections:
- wire segments 122 -> 123
Changed lines of the file:
@@
 $EndDescr
 $Sheet
-S 1450 1300 550  250
+S 1250 1300 550  250
 U 5DEC0147
 F0 "PressureSensor" 50
 F1 "PressureSensor.sch" 50
-F2 "SDA" I L 1450 1350 50
-F3 "SCL" I L 1450 1450 50
+F2 "SCL" I L 1250 1350 50
+F3 "SDA" B L 1250 1450 50
 $EndSheet
 $Sheet
-S 1450 1900 550  350
+S 1250 1900 550  350
 U 5DED66E9
 F0 "Accelerometer" 50
 F1 "Accelerometer.sch" 50
-F2 "Xout" O R 2000 1950 50
-F3 "Yout" O R 2000 2050 50
-F4 "Zout" O R 2000 2150 50
+F2 "Xout" O R 1800 1950 50
+F3 "Yout" O R 1800 2050 50
+F4 "Zout" O R 1800 2150 50
 $EndSheet
 $Sheet
@@
 $EndSheet
 $Sheet
-S 3200 1900 550  500
+S 3200 1900 700  400
 U 5DF50C3B
 F0 "microSD" 50
@@
 F3 "SD_CLK" I L 3200 2100 50
 F4 "SD_DI" I L 3200 2200 50
-F5 "SD_DO" O L 3200 2300 50
+F5 "SD_DO" O R 3900 2000 50
 $EndSheet
 $Comp
@@
 Wire Wire Line
 	8100 2900 8300 2900
-Text Label 1300 1350 2    50   ~ 0
+Text Label 1100 1450 2    50   ~ 0
 SDA
-Text Label 1300 1450 2    50   ~ 0
+Text Label 1100 1350 2    50   ~ 0
 SCL
 Wire Wire Line
-	1300 1350 1450 1350
-Wire Wire Line
-	1300 1450 1450 1450
-Text Label 1300 2900 2    50   ~ 0
+	1100 1450 1250 1450
+Wire Wire Line
+	1100 1350 1250 1350
+Text Label 1100 2700 2    50   ~ 0
 SDA
-Text Label 1300 2800 2    50   ~ 0
+Text Label 1100 2600 2    50   ~ 0
 SCL
 Wire Wire Line
-	1300 2800 1450 2800
-Wire Wire Line
-	1300 2900 1450 2900
+	1100 2600 1250 2600
+Wire Wire Line
+	1100 2700 1250 2700
 Wire Wire Line
 	5950 3600 6100 3600
@@
 $EndComp
 $Sheet
-S 1450 2650 550  450
+S 1250 2500 550  450
 U 5DF00598
 F0 "IMU" 50
 F1 "IMU.sch" 50
-F2 "INT" I L 1450 2700 50
-F3 "SCL" I L 1450 2800 50
-F4 "SDA" I L 1450 2900 50
-F5 "nRESET" I L 1450 3000 50
+F2 "SCL" I L 1250 2600 50
+F3 "nRESET" I L 1250 2850 50
+F4 "INT" O R 1800 2600 50
+F5 "SDA" B L 1250 2700 50
 $EndSheet
-Text Label 1300 3000 2    50   ~ 0
+Text Label 1100 2850 2    50   ~ 0
 IMU_RESET
 Wire Wire Line
-	1450 3000 1300 3000
+	1250 2850 1100 2850
 Text Label 5950 5000 2    50   ~ 0
 IMU_RESET
 Wire Wire Line
-	1450 2700 1300 2700
-Text Label 1300 2700 2    50   ~ 0
+	1800 2600 1950 2600
+Text Label 1950 2600 0    50   ~ 0
 IMU_INT
 Text Label 5950 2900 2    50   ~ 0
@@
 Wire Wire Line
 	5950 3100 6100 3100
-Text Label 2300 1950 0    50   ~ 0
+Text Label 2100 1950 0    50   ~ 0
 Xout
-Text Label 2300 2050 0    50   ~ 0
+Text Label 2100 2050 0    50   ~ 0
 Yout
-Text Label 2300 2150 0    50   ~ 0
+Text Label 2100 2150 0    50   ~ 0
 Zout
 Wire Wire Line
-	2000 1950 2300 1950
-Wire Wire Line
-	2000 2050 2300 2050
-Wire Wire Line
-	2000 2150 2300 2150
-Text Label 1200 3650 2    50   ~ 0
+	1800 1950 2100 1950
+Wire Wire Line
+	1800 2050 2100 2050
+Wire Wire Line
+	1800 2150 2100 2150
+Text Label 1050 3350 2    50   ~ 0
 CLK
-Text Label 1200 3750 2    50   ~ 0
+Text Label 1050 3450 2    50   ~ 0
 MOSI
-Text Label 1200 3850 2    50   ~ 0
+Text Label 2600 3350 0    50   ~ 0
 MISO
-Text Label 1200 3950 2    50   ~ 0
+Text Label 1050 3550 2    50   ~ 0
 RADIO_CS
-Text Label 1200 4050 2    50   ~ 0
+Text Label 1050 3750 2    50   ~ 0
 RADIO_RESET
 Wire Wire Line
-	1200 3650 1400 3650
-Wire Wire Line
-	1200 3750 1400 3750
-Wire Wire Line
-	1200 3850 1400 3850
-Wire Wire Line
-	1200 3950 1400 3950
+	1050 3350 1250 3350
+Wire Wire Line
+	1050 3450 1250 3450
+Wire Wire Line
+	2600 3350 2400 3350
+Wire Wire Line
+	1050 3550 1250 3550
 $Sheet
-S 1400 3550 950  700
+S 1250 3250 1150 600
 U 5E277237
 F0 "radio-915-lora" 50
 F1 "radio-915-lora.sch" 50
-F2 "RADIO_SCK" I L 1400 3650 50
-F3 "RADIO_MOSI" I L 1400 3750 50
-F4 "RADIO_MISO" O L 1400 3850 50
-F5 "RADIO_SS" I L 1400 3950 50
-F6 "RADIO_RESET" I L 1400 4050 50
-F7 "RADIO_DIO0" O L 1400 4150 50
+F2 "RADIO_SCK" I L 1250 3350 50
+F3 "RADIO_MOSI" I L 1250 3450 50
+F4 "RADIO_MISO" O R 2400 3350 50
+F5 "RADIO_SS" I L 1250 3550 50
+F6 "RADIO_RESET" I L 1250 3750 50
+F7 "RADIO_DIO0" O R 2400 3750 50
 $EndSheet
 Wire Wire Line
-	1200 4050 1400 4050
+	1050 3750 1250 3750
 Text Label 5950 4000 2    50   ~ 0
 RADIO_CS
@@
 Text Label 5950 4200 2    50   ~ 0
 RADIO_IO
-Text Label 1200 4150 2    50   ~ 0
+Text Label 2600 3750 0    50   ~ 0
 RADIO_IO
 Wire Wire Line
-	1200 4150 1400 4150
+	2600 3750 2400 3750
 Wire Wire Line
 	5950 4000 6100 4000
@@
 Text Label 3000 2200 2    50   ~ 0
 MOSI
-Text Label 3000 2300 2    50   ~ 0
+Text Label 4100 2000 0    50   ~ 0
 MISO
 Wire Wire Line
@@
 	3000 2200 3200 2200
 Wire Wire Line
-	3000 2300 3200 2300
+	4100 2000 3900 2000
 Text Label 3000 2000 2    50   ~ 0
 SD_CS
@@
 	5950 4200 6100 4200
 Wire Wire Line
-	2950 3250 3100 3250
-Wire Wire Line
-	2950 3150 3100 3150
+	3050 2750 3200 2750
+Wire Wire Line
+	3050 2650 3200 2650
 $Sheet
-S 3100 2700 850  750
+S 3200 2550 700  450
 U 5E2DF1A9
 F0 "gps-module" 50
 F1 "gps-module.sch" 50
-F2 "GPS_SDA" B L 3100 3150 50
-F3 "GPS_SCL" I L 3100 3250 50
-F4 "~RST" I L 3100 2950 50
+F2 "GPS_SDA" B L 3200 2650 50
+F3 "GPS_SCL" I L 3200 2750 50
+F4 "~RST" I L 3200 2900 50
 $EndSheet
 Text Label 5950 4900 2    50   ~ 0
@@
 P 9000 3200
 F 0 "C10" H 9115 3246 50  0000 L CNN
-F 1 "2.2u" H 9115 3155 50  0000 L CNN
+F 1 "1u" H 9115 3155 50  0000 L CNN
 F 2 "Capacitor_SMD:C_0603_1608Metric" H 9038 3050 50  0001 C CNN
 F 3 "~" H 9000 3200 50  0001 C CNN
@@
 P 10350 3200
 F 0 "C11" H 10465 3246 50  0000 L CNN
-F 1 "2.2u" H 10465 3155 50  0000 L CNN
+F 1 "1u" H 10465 3155 50  0000 L CNN
 F 2 "Capacitor_SMD:C_0603_1608Metric" H 10388 3050 50  0001 C CNN
 F 3 "~" H 10350 3200 50  0001 C CNN
@@
 Wire Wire Line
 	9750 3450 10350 3450
-Wire Wire Line
-	9000 3050 9350 3050
-Wire Wire Line
-	9350 3050 9350 3250
-Wire Wire Line
-	10150 3050 10350 3050
 $Comp
 L power:GND #PWR019
@@
 NoConn ~ 8100 3000
 NoConn ~ 8100 3100
-Text Label 2950 3250 2    50   ~ 0
+Text Label 3050 2750 2    50   ~ 0
 SCL
-Text Label 2950 3150 2    50   ~ 0
+Text Label 3050 2650 2    50   ~ 0
 SDA
 NoConn ~ 8100 2400
 Wire Wire Line
-	3100 2950 2950 2950
-NoConn ~ 2950 2950
-$Comp
-L recovery-custom:MIC5528-3.3YMT-TR U1
+	3200 2900 3050 2900
+NoConn ~ 3050 2900
+$Comp
+L recovery-custom:AP7366-33W5-7 U1
 U 1 1 5EFFFA85
 P 9750 3150
 F 0 "U1" H 9750 3517 50  0000 C CNN
-F 1 "MIC5528-3.3YMT-TR" H 9750 3426 50  0000 C CNN
-F 2 "Package_DFN_QFN:DFN-6-1EP_1.2x1.2mm_P0.4mm_EP0.3x0.94mm_PullBack" H 9750 2750 50  0001 C CNN
-F 3 "http://www.microchip.com/mymicrochip/filehandler.aspx?ddocname=en580311" H 9500 3400 50  0001 C CNN
+F 1 "AP7366-33W5-7" H 9750 3426 50  0000 C CNN
+F 2 "Package_TO_SOT_SMD:SOT-23-5" H 9750 2750 50  0001 C CNN
+F 3 "https://www.diodes.com/assets/Datasheets/AP7366.pdf" H 9500 3400 50  0001 C CNN
 	1    9750 3150
 	1    0    0    -1
@@
 	6450 1500 6750 1500
 Connection ~ 6750 1500
+Wire Wire Line
+	9000 3050 9400 3050
+Wire Wire Line
+	9400 3050 9400 3200
+Connection ~ 9400 3050
+Wire Wire Line
+	9750 3400 9750 3450
+Wire Wire Line
+	10100 3050 10350 3050
 $EndSCHEMATC

Commit message: Recovery PCB: Deleted excess pullup resistors, redid mounting holes.
Parts:
- added H1, H2, H3, H4: MountingHole, MountingHole:MountingHole_3.2mm_M3_Pad_Via, symbol Mechanical:MountingHole
Changed lines of the file:
@@
 EESchema Schematic File Version 4
+LIBS:Recovery PCB-cache
 EELAYER 30 0
 EELAYER END
@@
 Wire Wire Line
 	10100 3050 10350 3050
+$Comp
+L Mechanical:MountingHole H1
+U 1 1 600DBB87
+P 850 7100
+F 0 "H1" H 950 7146 50  0000 L CNN
+F 1 "MountingHole" H 950 7055 50  0000 L CNN
+F 2 "MountingHole:MountingHole_3.2mm_M3_Pad_Via" H 850 7100 50  0001 C CNN
+F 3 "~" H 850 7100 50  0001 C CNN
+	1    850  7100
+	1    0    0    -1
+$EndComp
+$Comp
+L Mechanical:MountingHole H2
+U 1 1 600DC751
+P 850 7300
+F 0 "H2" H 950 7346 50  0000 L CNN
+F 1 "MountingHole" H 950 7255 50  0000 L CNN
+F 2 "MountingHole:MountingHole_3.2mm_M3_Pad_Via" H 850 7300 50  0001 C CNN
+F 3 "~" H 850 7300 50  0001 C CNN
+	1    850  7300
+	1    0    0    -1
+$EndComp
+$Comp
+L Mechanical:MountingHole H3
+U 1 1 600E19B8
+P 850 7500
+F 0 "H3" H 950 7546 50  0000 L CNN
+F 1 "MountingHole" H 950 7455 50  0000 L CNN
+F 2 "MountingHole:MountingHole_3.2mm_M3_Pad_Via" H 850 7500 50  0001 C CNN
+F 3 "~" H 850 7500 50  0001 C CNN
+	1    850  7500
+	1    0    0    -1
+$EndComp
+$Comp
+L Mechanical:MountingHole H4
+U 1 1 600E6D04
+P 850 7700
+F 0 "H4" H 950 7746 50  0000 L CNN
+F 1 "MountingHole" H 950 7655 50  0000 L CNN
+F 2 "MountingHole:MountingHole_3.2mm_M3_Pad_Via" H 850 7700 50  0001 C CNN
+F 3 "~" H 850 7700 50  0001 C CNN
+	1    850  7700
+	1    0    0    -1
+$EndComp
 $EndSCHEMATC

Commit message: Recovery PCB: Minor changes to layout.
Parts:
- C1, C12, C4, C5, C6: value 100n -> 0.1u
- L1: value 10uH -> 10u
- Y1: value 32.768kHz -> 32.768k
Changed lines of the file:
@@
 P 5400 2550
 F 0 "Y1" V 5354 2681 50  0000 L CNN
-F 1 "32.768kHz" V 5445 2681 50  0000 L CNN
+F 1 "32.768k" V 5445 2681 50  0000 L CNN
 F 2 "Crystal:Crystal_SMD_3215-2Pin_3.2x1.5mm" H 5400 2550 50  0001 C CNN
 F 3 "~" H 5400 2550 50  0001 C CNN
@@
 P 7850 1550
 F 0 "C1" H 7700 1550 50  0000 C CNN
-F 1 "100n" H 7650 1450 50  0000 C CNN
+F 1 "0.1u" H 7650 1450 50  0000 C CNN
 F 2 "Capacitor_SMD:C_0603_1608Metric" H 7888 1400 50  0001 C CNN
 F 3 "~" H 7850 1550 50  0001 C CNN
@@
 P 6150 1650
 F 0 "C4" H 6000 1650 50  0000 C CNN
-F 1 "100n" H 6000 1550 50  0000 C CNN
+F 1 "0.1u" H 6000 1550 50  0000 C CNN
 F 2 "Capacitor_SMD:C_0603_1608Metric" H 6188 1500 50  0001 C CNN
 F 3 "~" H 6150 1650 50  0001 C CNN
@@
 P 6750 1650
 F 0 "C6" H 6600 1650 50  0000 C CNN
-F 1 "100n" H 6600 1750 50  0000 C CNN
+F 1 "0.1u" H 6600 1750 50  0000 C CNN
 F 2 "Capacitor_SMD:C_0603_1608Metric" H 6788 1500 50  0001 C CNN
 F 3 "~" H 6750 1650 50  0001 C CNN
@@
 P 6000 6350
 F 0 "C12" H 6115 6396 50  0000 L CNN
-F 1 "100n" H 6115 6305 50  0000 L CNN
+F 1 "0.1u" H 6115 6305 50  0000 L CNN
 F 2 "Capacitor_SMD:C_0603_1608Metric" H 6038 6200 50  0001 C CNN
 F 3 "~" H 6000 6350 50  0001 C CNN
@@
 P 7000 1100
 F 0 "L1" V 6950 1300 50  0000 C CNN
-F 1 "10uH" V 7050 1300 50  0000 C CNN
+F 1 "10u" V 7050 1300 50  0000 C CNN
 F 2 "Inductor_SMD:L_1008_2520Metric" H 7000 1100 50  0001 C CNN
 F 3 "~" H 7000 1100 50  0001 C CNN
@@
 P 6450 1650
 F 0 "C5" H 6300 1650 50  0000 C CNN
-F 1 "100n" H 6300 1750 50  0000 C CNN
+F 1 "0.1u" H 6300 1750 50  0000 C CNN
 F 2 "Capacitor_SMD:C_0603_1608Metric" H 6488 1500 50  0001 C CNN
 F 3 "~" H 6450 1650 50  0001 C CNN
