File: Recovery PCB/gps-module.sch (KiCad schematic (older format))
At the start: 5 parts

Commit message: Update relays and re-annotate entire schematic. Review needed before layout.
Parts:
- gave numbers to parts that had none: 5
Changed lines of the file:
@@
 $EndDescr
 $Comp
-L power:+3.3V #PWR?
+L power:+3.3V #PWR048
 U 1 1 5E2DF238
 P 6450 2300
-F 0 "#PWR?" H 6450 2150 50  0001 C CNN
+F 0 "#PWR048" H 6450 2150 50  0001 C CNN
 F 1 "+3.3V" H 6465 2473 50  0000 C CNN
 F 2 "" H 6450 2300 50  0001 C CNN
@@
 $EndComp
 $Comp
-L Device:C C?
+L Device:C C22
 U 1 1 5E2E0557
 P 6450 2450
-F 0 "C?" H 6565 2496 50  0000 L CNN
+F 0 "C22" H 6565 2496 50  0000 L CNN
 F 1 "0.1u" H 6565 2405 50  0000 L CNN
 F 2 "" H 6488 2300 50  0001 C CNN
@@
 $EndComp
 $Comp
-L power:GND #PWR?
+L power:GND #PWR049
 U 1 1 5E2E05B5
 P 6450 2600
-F 0 "#PWR?" H 6450 2350 50  0001 C CNN
+F 0 "#PWR049" H 6450 2350 50  0001 C CNN
 F 1 "GND" H 6455 2427 50  0000 C CNN
 F 2 "" H 6450 2600 50  0001 C CNN
@@
 $EndComp
 $Comp
-L power:GND #PWR?
+L power:GND #PWR046
 U 1 1 5E2E05DA
 P 4150 3350
-F 0 "#PWR?" H 4150 3100 50  0001 C CNN
+F 0 "#PWR046" H 4150 3100 50  0001 C CNN
 F 1 "GND" H 4155 3177 50  0000 C CNN
 F 2 "" H 4150 3350 50  0001 C CNN
@@
 TX
 $Comp
-L RF_GPS:ublox_SAM-M8Q U?
+L RF_GPS:ublox_SAM-M8Q U7
 U 1 1 5E36093E
 P 4650 2850
-F 0 "U?" H 4650 2264 50  0000 C CNN
+F 0 "U7" H 4650 2264 50  0000 C CNN
 F 1 "ublox_SAM-M8Q" H 4650 2173 50  0000 C CNN
 F 2 "RF_Module:ublox_SAM-M8Q" H 5200 2400 50  0001 C CNN
@@
 $EndComp
 $Comp
-L power:+3.3V #PWR?
+L power:+3.3V #PWR047
 U 1 1 5E360B04
 P 4550 2300
-F 0 "#PWR?" H 4550 2150 50  0001 C CNN
+F 0 "#PWR047" H 4550 2150 50  0001 C CNN
 F 1 "+3.3V" H 4565 2473 50  0000 C CNN
 F 2 "" H 4550 2300 50  0001 C CNN
@@
 GPS_SCL
 $Comp
-L Device:R R?
+L Device:R R16
 U 1 1 5E361A27
 P 5450 2950
-F 0 "R?" V 5243 2950 50  0000 C CNN
+F 0 "R16" V 5243 2950 50  0000 C CNN
 F 1 "22" V 5334 2950 50  0000 C CNN
 F 2 "" V 5380 2950 50  0001 C CNN
@@
 $EndComp
 $Comp
-L Device:R R?
+L Device:R R17
 U 1 1 5E361A85
 P 5450 3250
-F 0 "R?" V 5243 3250 50  0000 C CNN
+F 0 "R17" V 5243 3250 50  0000 C CNN
 F 1 "22" V 5334 3250 50  0000 C CNN
 F 2 "" V 5380 3250 50  0001 C CNN
@@
 NoConn ~ 4150 2850
 $Comp
-L Connector:Conn_01x03_Female J?
+L Connector:Conn_01x03_Female J8
 U 1 1 5E3FA8A5
 P 3250 2850
-F 0 "J?" H 3144 3135 50  0000 C CNN
+F 0 "J8" H 3144 3135 50  0000 C CNN
 F 1 "Conn_01x03_Female" H 3144 3044 50  0000 C CNN
 F 2 "" H 3250 2850 50  0001 C CNN

Commit message: Added footprints.
Added footprints for various parts. Still need to update some more and calculate some values.
Parts:
- removed R16, R17: 22, symbol Device:R
- added R18, R19: 22, Resistor_SMD:R_0603_1608Metric, symbol Device:R_US
- C22: footprint (none) -> Capacitor_SMD:C_0603_1608Metric
Changed lines of the file:
@@
 $EndDescr
 $Comp
-L power:+3.3V #PWR048
+L power:+3.3V #PWR053
 U 1 1 5E2DF238
 P 6450 2300
-F 0 "#PWR048" H 6450 2150 50  0001 C CNN
+F 0 "#PWR053" H 6450 2150 50  0001 C CNN
 F 1 "+3.3V" H 6465 2473 50  0000 C CNN
 F 2 "" H 6450 2300 50  0001 C CNN
@@
 F 0 "C22" H 6565 2496 50  0000 L CNN
 F 1 "0.1u" H 6565 2405 50  0000 L CNN
-F 2 "" H 6488 2300 50  0001 C CNN
+F 2 "Capacitor_SMD:C_0603_1608Metric" H 6488 2300 50  0001 C CNN
 F 3 "~" H 6450 2450 50  0001 C CNN
 	1    6450 2450
@@
 $EndComp
 $Comp
-L power:GND #PWR049
+L power:GND #PWR054
 U 1 1 5E2E05B5
 P 6450 2600
-F 0 "#PWR049" H 6450 2350 50  0001 C CNN
+F 0 "#PWR054" H 6450 2350 50  0001 C CNN
 F 1 "GND" H 6455 2427 50  0000 C CNN
 F 2 "" H 6450 2600 50  0001 C CNN
@@
 $EndComp
 $Comp
-L power:GND #PWR046
+L power:GND #PWR051
 U 1 1 5E2E05DA
 P 4150 3350
-F 0 "#PWR046" H 4150 3100 50  0001 C CNN
+F 0 "#PWR051" H 4150 3100 50  0001 C CNN
 F 1 "GND" H 4155 3177 50  0000 C CNN
 F 2 "" H 4150 3350 50  0001 C CNN
@@
 $EndComp
 $Comp
-L power:+3.3V #PWR047
+L power:+3.3V #PWR052
 U 1 1 5E360B04
 P 4550 2300
-F 0 "#PWR047" H 4550 2150 50  0001 C CNN
+F 0 "#PWR052" H 4550 2150 50  0001 C CNN
 F 1 "+3.3V" H 4565 2473 50  0000 C CNN
 F 2 "" H 4550 2300 50  0001 C CNN
@@
 Text HLabel 5750 3050 2    50   Input ~ 0
 GPS_SCL
-$Comp
-L Device:R R16
-U 1 1 5E361A27
-P 5450 2950
-F 0 "R16" V 5243 2950 50  0000 C CNN
-F 1 "22" V 5334 2950 50  0000 C CNN
-F 2 "" V 5380 2950 50  0001 C CNN
-F 3 "~" H 5450 2950 50  0001 C CNN
-	1    5450 2950
-	0    1    1    0
-$EndComp
-$Comp
-L Device:R R17
-U 1 1 5E361A85
-P 5450 3250
-F 0 "R17" V 5243 3250 50  0000 C CNN
-F 1 "22" V 5334 3250 50  0000 C CNN
-F 2 "" V 5380 3250 50  0001 C CNN
-F 3 "~" H 5450 3250 50  0001 C CNN
-	1    5450 3250
-	0    1    1    0
-$EndComp
 Wire Wire Line
 	5300 3250 5150 3250
@@
 Wire Wire Line
 	3750 3050 4150 3050
+$Comp
+L Device:R_US R18
+U 1 1 5E68A6B9
+P 5450 2950
+F 0 "R18" V 5245 2950 50  0000 C CNN
+F 1 "22" V 5336 2950 50  0000 C CNN
+F 2 "Resistor_SMD:R_0603_1608Metric" V 5490 2940 50  0001 C CNN
+F 3 "~" H 5450 2950 50  0001 C CNN
+	1    5450 2950
+	0    1    1    0
+$EndComp
+$Comp
+L Device:R_US R19
+U 1 1 5E68AC1C
+P 5450 3250
+F 0 "R19" V 5245 3250 50  0000 C CNN
+F 1 "22" V 5336 3250 50  0000 C CNN
+F 2 "Resistor_SMD:R_0603_1608Metric" V 5490 3240 50  0001 C CNN
+F 3 "~" H 5450 3250 50  0001 C CNN
+	1    5450 3250
+	0    1    1    0
+$EndComp
 $EndSCHEMATC

Commit message: Updated some footprints and re-annotated schematic.
Parts:
- J9: renamed from J8; footprint (none) -> Connector_PinSocket_2.54mm:PinSocket_1x03_P2.54mm_Vertical
- renumbered C22 to C24, R18 to R19, R19 to R20
Changed lines of the file:
@@
 EESchema Schematic File Version 4
-LIBS:Recovery PCB-cache
-EELAYER 26 0
+EELAYER 30 0
 EELAYER END
 $Descr A4 11693 8268
@@
 $EndDescr
 $Comp
-L power:+3.3V #PWR053
+L power:+3.3V #PWR062
 U 1 1 5E2DF238
 P 6450 2300
-F 0 "#PWR053" H 6450 2150 50  0001 C CNN
+F 0 "#PWR062" H 6450 2150 50  0001 C CNN
 F 1 "+3.3V" H 6465 2473 50  0000 C CNN
 F 2 "" H 6450 2300 50  0001 C CNN
@@
 $EndComp
 $Comp
-L Device:C C22
+L Device:C C24
 U 1 1 5E2E0557
 P 6450 2450
-F 0 "C22" H 6565 2496 50  0000 L CNN
+F 0 "C24" H 6565 2496 50  0000 L CNN
 F 1 "0.1u" H 6565 2405 50  0000 L CNN
 F 2 "Capacitor_SMD:C_0603_1608Metric" H 6488 2300 50  0001 C CNN
@@
 $EndComp
 $Comp
-L power:GND #PWR054
+L power:GND #PWR063
 U 1 1 5E2E05B5
 P 6450 2600
-F 0 "#PWR054" H 6450 2350 50  0001 C CNN
+F 0 "#PWR063" H 6450 2350 50  0001 C CNN
 F 1 "GND" H 6455 2427 50  0000 C CNN
 F 2 "" H 6450 2600 50  0001 C CNN
@@
 $EndComp
 $Comp
-L power:GND #PWR051
+L power:GND #PWR060
 U 1 1 5E2E05DA
 P 4150 3350
-F 0 "#PWR051" H 4150 3100 50  0001 C CNN
+F 0 "#PWR060" H 4150 3100 50  0001 C CNN
 F 1 "GND" H 4155 3177 50  0000 C CNN
 F 2 "" H 4150 3350 50  0001 C CNN
@@
 $EndComp
 $Comp
-L power:+3.3V #PWR052
+L power:+3.3V #PWR061
 U 1 1 5E360B04
 P 4550 2300
-F 0 "#PWR052" H 4550 2150 50  0001 C CNN
+F 0 "#PWR061" H 4550 2150 50  0001 C CNN
 F 1 "+3.3V" H 4565 2473 50  0000 C CNN
 F 2 "" H 4550 2300 50  0001 C CNN
@@
 NoConn ~ 4150 2850
 $Comp
-L Connector:Conn_01x03_Female J8
+L Connector:Conn_01x03_Female J9
 U 1 1 5E3FA8A5
 P 3250 2850
-F 0 "J8" H 3144 3135 50  0000 C CNN
+F 0 "J9" H 3144 3135 50  0000 C CNN
 F 1 "Conn_01x03_Female" H 3144 3044 50  0000 C CNN
-F 2 "" H 3250 2850 50  0001 C CNN
+F 2 "Connector_PinSocket_2.54mm:PinSocket_1x03_P2.54mm_Vertical" H 3250 2850 50  0001 C CNN
 F 3 "~" H 3250 2850 50  0001 C CNN
 	1    3250 2850
@@
 	3750 3050 4150 3050
 $Comp
-L Device:R_US R18
+L Device:R_US R19
 U 1 1 5E68A6B9
 P 5450 2950
-F 0 "R18" V 5245 2950 50  0000 C CNN
+F 0 "R19" V 5245 2950 50  0000 C CNN
 F 1 "22" V 5336 2950 50  0000 C CNN
 F 2 "Resistor_SMD:R_0603_1608Metric" V 5490 2940 50  0001 C CNN
@@
 $EndComp
 $Comp
-L Device:R_US R19
+L Device:R_US R20
 U 1 1 5E68AC1C
 P 5450 3250
-F 0 "R19" V 5245 3250 50  0000 C CNN
+F 0 "R20" V 5245 3250 50  0000 C CNN
 F 1 "22" V 5336 3250 50  0000 C CNN
 F 2 "Resistor_SMD:R_0603_1608Metric" V 5490 3240 50  0001 C CNN

Commit message: Added missing footprints and replaced GPS module.
Parts:
- removed J9: Conn_01x03_Female, Connector_PinSocket_2.54mm:PinSocket_1x03_P2.54mm_Vertical, symbol Connector:Conn_01x03_Female
- removed U7: ublox_SAM-M8Q, RF_Module:ublox_SAM-M8Q, symbol RF_GPS:ublox_SAM-M8Q
- added J9: CON-SMA-EDGE-S, RFSOLUTIONS_CON-SMA-EDGE-S, symbol CON-SMA-EDGE-S:CON-SMA-EDGE-S
- added R21: 2.2k, Resistor_SMD:R_0603_1608Metric, symbol Device:R_US
- added U8: CAM-M8, CAM-M8, symbol CAM-M8:CAM-M8
- C24: value 0.1u -> 4.7u
- R19, R20: value 22 -> 2.2k
Connections:
- net labels added: ~RST
- net labels removed: RX, TX
- wire segments 16 -> 47
- no-connect marks 1 -> 8

Commit message: Finished Revision 1 of the Recovery PCB.
Parts:
- J9: footprint RFSOLUTIONS_CON-SMA-EDGE-S -> Parts:RFSOLUTIONS_CON-SMA-EDGE-S
- U8: footprint CAM-M8 -> Parts:CAM-M8
Changed lines of the file:
@@
 F 0 "U8" H 6000 3000 50  0001 L BNN
 F 1 "CAM-M8" H 6000 3000 50  0001 L BNN
-F 2 "CAM-M8" H 6000 3000 50  0001 L BNN
+F 2 "Parts:CAM-M8" H 6000 3000 50  0001 L BNN
 F 3 "" H 6000 3000 50  0001 L BNN
 	1    6000 3000
@@
 Connection ~ 6100 1800
 NoConn ~ 6900 2600
-Wire Wire Line
-	6900 2900 7500 2900
 NoConn ~ 4600 3700
 NoConn ~ 4600 3100
@@
 L CON-SMA-EDGE-S:CON-SMA-EDGE-S J9
 U 1 1 5FCDAE06
-P 7600 2900
-F 0 "J9" H 7440 2894 50  0000 R CNN
-F 1 "CON-SMA-EDGE-S" H 7440 2985 50  0000 R CNN
-F 2 "RFSOLUTIONS_CON-SMA-EDGE-S" H 7600 2900 50  0001 L BNN
-F 3 "" H 7600 2900 50  0001 L BNN
-F 4 "RF Solutions" H 7600 2900 50  0001 L BNN "MANUFACTURER"
-F 5 "1" H 7600 2900 50  0001 L BNN "PARTREV"
-F 6 "6.35mm" H 7600 2900 50  0001 L BNN "MAXIMUM_PACKAGE_HEIGHT"
-F 7 "Manufacturer Recommendations" H 7600 2900 50  0001 L BNN "STANDARD"
-	1    7600 2900
-	-1   0    0    1
+P 7300 3000
+F 0 "J9" H 7140 2994 50  0000 R CNN
+F 1 "CON-SMA-EDGE-S" H 7140 3085 50  0000 R CNN
+F 2 "Parts:RFSOLUTIONS_CON-SMA-EDGE-S" H 7300 3000 50  0001 L BNN
+F 3 "" H 7300 3000 50  0001 L BNN
+F 4 "RF Solutions" H 7300 3000 50  0001 L BNN "MANUFACTURER"
+F 5 "1" H 7300 3000 50  0001 L BNN "PARTREV"
+F 6 "6.35mm" H 7300 3000 50  0001 L BNN "MAXIMUM_PACKAGE_HEIGHT"
+F 7 "Manufacturer Recommendations" H 7300 3000 50  0001 L BNN "STANDARD"
+	1    7300 3000
+	-1   0    0    -1
 $EndComp
 $Comp
 L power:GND #PWR066
 U 1 1 5FCDC46C
-P 7500 3100
-F 0 "#PWR066" H 7500 2850 50  0001 C CNN
-F 1 "GND" H 7505 2927 50  0000 C CNN
-F 2 "" H 7500 3100 50  0001 C CNN
-F 3 "" H 7500 3100 50  0001 C CNN
-	1    7500 3100
-	1    0    0    -1
-$EndComp
-Wire Wire Line
-	7500 3100 7500 3000
+P 7200 3100
+F 0 "#PWR066" H 7200 2850 50  0001 C CNN
+F 1 "GND" H 7205 2927 50  0000 C CNN
+F 2 "" H 7200 3100 50  0001 C CNN
+F 3 "" H 7200 3100 50  0001 C CNN
+	1    7200 3100
+	1    0    0    -1
+$EndComp
+Wire Wire Line
+	7200 3100 7200 3000
 $Comp
 L power:+3.3V #PWR060
@@
 Text HLabel 3600 3900 0    50   Input ~ 0
 ~RST
+Wire Wire Line
+	6900 2900 7200 2900
 $EndSCHEMATC

Commit message: Recovery PCB: Redraw schematics
Redrew Recover PCB schematics to be more easily readable and fixed board
outline, adding netclasses to ease trace placement.
Parts:
- J9: value CON-SMA-EDGE-S -> SMA_GPS
Connections:
- net labels added: GPS_RF
- wire segments 47 -> 45
Changed lines of the file:
@@
 L Device:C C24
 U 1 1 5FCFD1D5
-P 5200 1800
-F 0 "C24" V 5452 1800 50  0000 C CNN
-F 1 "4.7u" V 5361 1800 50  0000 C CNN
-F 2 "Capacitor_SMD:C_0603_1608Metric" H 5238 1650 50  0001 C CNN
-F 3 "~" H 5200 1800 50  0001 C CNN
-	1    5200 1800
-	0    -1   -1   0
+P 5350 1650
+F 0 "C24" H 5550 1700 50  0000 C CNN
+F 1 "4.7u" H 5550 1600 50  0000 C CNN
+F 2 "Capacitor_SMD:C_0603_1608Metric" H 5388 1500 50  0001 C CNN
+F 3 "~" H 5350 1650 50  0001 C CNN
+	1    5350 1650
+	-1   0    0    -1
 $EndComp
 $Comp
 L power:GND #PWR063
 U 1 1 5FCFFDB2
-P 4900 1800
-F 0 "#PWR063" H 4900 1550 50  0001 C CNN
-F 1 "GND" H 4905 1627 50  0000 C CNN
-F 2 "" H 4900 1800 50  0001 C CNN
-F 3 "" H 4900 1800 50  0001 C CNN
-	1    4900 1800
+P 5350 1800
+F 0 "#PWR063" H 5350 1550 50  0001 C CNN
+F 1 "GND" H 5355 1627 50  0000 C CNN
+F 2 "" H 5350 1800 50  0001 C CNN
+F 3 "" H 5350 1800 50  0001 C CNN
+	1    5350 1800
 	1    0    0    -1
 $EndComp
-Wire Wire Line
-	4900 1800 5050 1800
-Wire Wire Line
-	5350 1800 5500 1800
-Wire Wire Line
-	5500 1800 5500 1900
-Wire Wire Line
-	5500 1800 5800 1800
-Wire Wire Line
-	5800 1800 5800 1900
-Connection ~ 5500 1800
-Wire Wire Line
-	5800 1800 6100 1800
-Wire Wire Line
-	6100 1800 6100 1900
-Connection ~ 5800 1800
-Wire Wire Line
-	6100 1800 6250 1800
-Connection ~ 6100 1800
 NoConn ~ 6900 2600
 NoConn ~ 4600 3700
@@
 L power:+3.3V #PWR065
 U 1 1 5FCDA81D
-P 6250 1800
-F 0 "#PWR065" H 6250 1650 50  0001 C CNN
-F 1 "+3.3V" H 6265 1973 50  0000 C CNN
-F 2 "" H 6250 1800 50  0001 C CNN
-F 3 "" H 6250 1800 50  0001 C CNN
-	1    6250 1800
+P 5500 1500
+F 0 "#PWR065" H 5500 1350 50  0001 C CNN
+F 1 "+3.3V" H 5515 1673 50  0000 C CNN
+F 2 "" H 5500 1500 50  0001 C CNN
+F 3 "" H 5500 1500 50  0001 C CNN
+	1    5500 1500
 	1    0    0    -1
 $EndComp
@@
 P 7300 3000
 F 0 "J9" H 7140 2994 50  0000 R CNN
-F 1 "CON-SMA-EDGE-S" H 7140 3085 50  0000 R CNN
+F 1 "SMA_GPS" H 7140 3085 50  0000 R CNN
 F 2 "Parts:RFSOLUTIONS_CON-SMA-EDGE-S" H 7300 3000 50  0001 L BNN
 F 3 "" H 7300 3000 50  0001 L BNN
@@
 Wire Wire Line
 	6900 2900 7200 2900
+Wire Wire Line
+	5350 1500 5500 1500
+Connection ~ 5500 1500
+Wire Wire Line
+	5500 1500 5500 1900
+Wire Wire Line
+	5500 1500 5800 1500
+Wire Wire Line
+	6100 1500 6100 1900
+Wire Wire Line
+	5800 1500 5800 1900
+Connection ~ 5800 1500
+Wire Wire Line
+	5800 1500 6100 1500
+Text Label 6900 2900 0    50   ~ 0
+GPS_RF
 $EndSCHEMATC
