File: Recovery PCB/gps-module.sch (KiCad schematic (older format))
At the start: 6 parts, among them J9 SMA_GPS, U8 CAM-M8

Commit message: Recovery PCB: Reannotate
Reannotated schematic to fix reference numbering and keep reference
designators consistent.
Parts:
- renumbered C24 to C25, J9 to J10, R19 to R20, R20 to R22, U8 to U7
Changed lines of the file:
@@
 $EndDescr
 $Comp
-L CAM-M8:CAM-M8 U8
+L CAM-M8:CAM-M8 U7
 U 1 1 5FCE2632
 P 6000 3000
-F 0 "U8" H 6000 3000 50  0001 L BNN
+F 0 "U7" H 6000 3000 50  0001 L BNN
 F 1 "CAM-M8" H 6000 3000 50  0001 L BNN
 F 2 "Parts:CAM-M8" H 6000 3000 50  0001 L BNN
@@
 $EndComp
 $Comp
-L power:GND #PWR064
+L power:GND #PWR087
 U 1 1 5FCF463B
 P 5100 4600
-F 0 "#PWR064" H 5100 4350 50  0001 C CNN
+F 0 "#PWR087" H 5100 4350 50  0001 C CNN
 F 1 "GND" H 5105 4427 50  0000 C CNN
 F 2 "" H 5100 4600 50  0001 C CNN
@@
 Connection ~ 6300 4550
 $Comp
-L Device:C C24
+L Device:C C25
 U 1 1 5FCFD1D5
 P 5350 1650
-F 0 "C24" H 5550 1700 50  0000 C CNN
+F 0 "C25" H 5550 1700 50  0000 C CNN
 F 1 "4.7u" H 5550 1600 50  0000 C CNN
 F 2 "Capacitor_SMD:C_0603_1608Metric" H 5388 1500 50  0001 C CNN
@@
 $EndComp
 $Comp
-L power:GND #PWR063
+L power:GND #PWR082
 U 1 1 5FCFFDB2
 P 5350 1800
-F 0 "#PWR063" H 5350 1550 50  0001 C CNN
+F 0 "#PWR082" H 5350 1550 50  0001 C CNN
 F 1 "GND" H 5355 1627 50  0000 C CNN
 F 2 "" H 5350 1800 50  0001 C CNN
@@
 NoConn ~ 4600 2900
 $Comp
-L power:+3.3V #PWR065
+L power:+3.3V #PWR081
 U 1 1 5FCDA81D
 P 5500 1500
-F 0 "#PWR065" H 5500 1350 50  0001 C CNN
+F 0 "#PWR081" H 5500 1350 50  0001 C CNN
 F 1 "+3.3V" H 5515 1673 50  0000 C CNN
 F 2 "" H 5500 1500 50  0001 C CNN
@@
 $EndComp
 $Comp
-L CON-SMA-EDGE-S:CON-SMA-EDGE-S J9
+L CON-SMA-EDGE-S:CON-SMA-EDGE-S J10
 U 1 1 5FCDAE06
 P 7300 3000
-F 0 "J9" H 7140 2994 50  0000 R CNN
+F 0 "J10" H 7140 2994 50  0000 R CNN
 F 1 "SMA_GPS" H 7140 3085 50  0000 R CNN
 F 2 "Parts:RFSOLUTIONS_CON-SMA-EDGE-S" H 7300 3000 50  0001 L BNN
@@
 $EndComp
 $Comp
-L power:GND #PWR066
+L power:GND #PWR085
 U 1 1 5FCDC46C
 P 7200 3100
-F 0 "#PWR066" H 7200 2850 50  0001 C CNN
+F 0 "#PWR085" H 7200 2850 50  0001 C CNN
 F 1 "GND" H 7205 2927 50  0000 C CNN
 F 2 "" H 7200 3100 50  0001 C CNN
@@
 	7200 3100 7200 3000
 $Comp
-L power:+3.3V #PWR060
+L power:+3.3V #PWR083
 U 1 1 5FCDD8DF
 P 3750 2100
-F 0 "#PWR060" H 3750 1950 50  0001 C CNN
+F 0 "#PWR083" H 3750 1950 50  0001 C CNN
 F 1 "+3.3V" H 3765 2273 50  0000 C CNN
 F 2 "" H 3750 2100 50  0001 C CNN
@@
 $EndComp
 $Comp
-L Device:R_US R19
+L Device:R_US R20
 U 1 1 5FCDE146
 P 3750 2300
-F 0 "R19" H 3818 2346 50  0000 L CNN
+F 0 "R20" H 3818 2346 50  0000 L CNN
 F 1 "2.2k" H 3818 2255 50  0000 L CNN
 F 2 "Resistor_SMD:R_0603_1608Metric" V 3790 2290 50  0001 C CNN
@@
 	3750 2150 3750 2100
 $Comp
-L power:+3.3V #PWR062
+L power:+3.3V #PWR084
 U 1 1 5FCF559E
 P 4050 2150
-F 0 "#PWR062" H 4050 2000 50  0001 C CNN
+F 0 "#PWR084" H 4050 2000 50  0001 C CNN
 F 1 "+3.3V" H 4065 2323 50  0000 C CNN
 F 2 "" H 4050 2150 50  0001 C CNN
@@
 $EndComp
 $Comp
-L power:+3.3V #PWR061
+L power:+3.3V #PWR086
 U 1 1 5FCF68E0
 P 3750 3600
-F 0 "#PWR061" H 3750 3450 50  0001 C CNN
+F 0 "#PWR086" H 3750 3450 50  0001 C CNN
 F 1 "+3.3V" H 3765 3773 50  0000 C CNN
 F 2 "" H 3750 3600 50  0001 C CNN
@@
 $EndComp
 $Comp
-L Device:R_US R20
+L Device:R_US R22
 U 1 1 5FCF6C65
 P 3750 3750
-F 0 "R20" H 3818 3796 50  0000 L CNN
+F 0 "R22" H 3818 3796 50  0000 L CNN
 F 1 "2.2k" H 3818 3705 50  0000 L CNN
 F 2 "Resistor_SMD:R_0603_1608Metric" V 3790 3740 50  0001 C CNN

Commit message: Recovery PCB: Deleted excess pullup resistors, redid mounting holes.
Parts:
- removed R20, R21: 2.2k, Resistor_SMD:R_0603_1608Metric, symbol Device:R_US
Connections:
- wire segments 45 -> 40
Changed lines of the file:
@@
 EESchema Schematic File Version 4
+LIBS:Recovery PCB-cache
 EELAYER 30 0
 EELAYER END
@@
 Wire Wire Line
 	7200 3100 7200 3000
-$Comp
-L power:+3.3V #PWR083
-U 1 1 5FCDD8DF
-P 3750 2100
-F 0 "#PWR083" H 3750 1950 50  0001 C CNN
-F 1 "+3.3V" H 3765 2273 50  0000 C CNN
-F 2 "" H 3750 2100 50  0001 C CNN
-F 3 "" H 3750 2100 50  0001 C CNN
-	1    3750 2100
-	1    0    0    -1
-$EndComp
-$Comp
-L Device:R_US R20
-U 1 1 5FCDE146
-P 3750 2300
-F 0 "R20" H 3818 2346 50  0000 L CNN
-F 1 "2.2k" H 3818 2255 50  0000 L CNN
-F 2 "Resistor_SMD:R_0603_1608Metric" V 3790 2290 50  0001 C CNN
-F 3 "~" H 3750 2300 50  0001 C CNN
-	1    3750 2300
-	1    0    0    -1
-$EndComp
-$Comp
-L Device:R_US R21
-U 1 1 5FCDEE3F
-P 4050 2300
-F 0 "R21" H 4118 2346 50  0000 L CNN
-F 1 "2.2k" H 4118 2255 50  0000 L CNN
-F 2 "Resistor_SMD:R_0603_1608Metric" V 4090 2290 50  0001 C CNN
-F 3 "~" H 4050 2300 50  0001 C CNN
-	1    4050 2300
-	1    0    0    -1
-$EndComp
 Text HLabel 3500 2600 0    50   Output ~ 0
 GPS_SCL
 Text HLabel 3500 2700 0    50   Input ~ 0
 GPS_SDA
-Wire Wire Line
-	3500 2700 4050 2700
-Wire Wire Line
-	3500 2600 3750 2600
-Wire Wire Line
-	3750 2600 3750 2450
-Connection ~ 3750 2600
-Wire Wire Line
-	3750 2600 4600 2600
-Wire Wire Line
-	4050 2450 4050 2700
-Connection ~ 4050 2700
-Wire Wire Line
-	4050 2700 4600 2700
-Wire Wire Line
-	3750 2150 3750 2100
-$Comp
-L power:+3.3V #PWR084
-U 1 1 5FCF559E
-P 4050 2150
-F 0 "#PWR084" H 4050 2000 50  0001 C CNN
-F 1 "+3.3V" H 4065 2323 50  0000 C CNN
-F 2 "" H 4050 2150 50  0001 C CNN
-F 3 "" H 4050 2150 50  0001 C CNN
-	1    4050 2150
-	1    0    0    -1
-$EndComp
 $Comp
 L power:+3.3V #PWR086
@@
 Text Label 6900 2900 0    50   ~ 0
 GPS_RF
+Wire Wire Line
+	3500 2600 4600 2600
+Wire Wire Line
+	3500 2700 4600 2700
 $EndSCHEMATC

Commit message: Recovery PCB: Add active antenna supply circuit.
Parts:
- added C26: 47n, Capacitor_SMD:C_0603_1608Metric, symbol Device:C
- added C27: 1n, Capacitor_SMD:C_0603_1608Metric, symbol Device:C
- added L2: 47n, Inductor_SMD:L_0603_1608Metric, symbol Device:L
Connections:
- wire segments 40 -> 46
Changed lines of the file:
@@
 L CON-SMA-EDGE-S:CON-SMA-EDGE-S J10
 U 1 1 5FCDAE06
-P 7300 3000
-F 0 "J10" H 7140 2994 50  0000 R CNN
-F 1 "SMA_GPS" H 7140 3085 50  0000 R CNN
-F 2 "Parts:RFSOLUTIONS_CON-SMA-EDGE-S" H 7300 3000 50  0001 L BNN
-F 3 "" H 7300 3000 50  0001 L BNN
-F 4 "RF Solutions" H 7300 3000 50  0001 L BNN "MANUFACTURER"
-F 5 "1" H 7300 3000 50  0001 L BNN "PARTREV"
-F 6 "6.35mm" H 7300 3000 50  0001 L BNN "MAXIMUM_PACKAGE_HEIGHT"
-F 7 "Manufacturer Recommendations" H 7300 3000 50  0001 L BNN "STANDARD"
-	1    7300 3000
+P 7550 3000
+F 0 "J10" H 7390 2994 50  0000 R CNN
+F 1 "SMA_GPS" H 7390 3085 50  0000 R CNN
+F 2 "Parts:RFSOLUTIONS_CON-SMA-EDGE-S" H 7550 3000 50  0001 L BNN
+F 3 "" H 7550 3000 50  0001 L BNN
+F 4 "RF Solutions" H 7550 3000 50  0001 L BNN "MANUFACTURER"
+F 5 "1" H 7550 3000 50  0001 L BNN "PARTREV"
+F 6 "6.35mm" H 7550 3000 50  0001 L BNN "MAXIMUM_PACKAGE_HEIGHT"
+F 7 "Manufacturer Recommendations" H 7550 3000 50  0001 L BNN "STANDARD"
+	1    7550 3000
 	-1   0    0    -1
 $EndComp
@@
 L power:GND #PWR085
 U 1 1 5FCDC46C
-P 7200 3100
-F 0 "#PWR085" H 7200 2850 50  0001 C CNN
-F 1 "GND" H 7205 2927 50  0000 C CNN
-F 2 "" H 7200 3100 50  0001 C CNN
-F 3 "" H 7200 3100 50  0001 C CNN
-	1    7200 3100
+P 7450 3100
+F 0 "#PWR085" H 7450 2850 50  0001 C CNN
+F 1 "GND" H 7455 2927 50  0000 C CNN
+F 2 "" H 7450 3100 50  0001 C CNN
+F 3 "" H 7450 3100 50  0001 C CNN
+	1    7450 3100
 	1    0    0    -1
 $EndComp
 Wire Wire Line
-	7200 3100 7200 3000
+	7450 3100 7450 3000
 Text HLabel 3500 2600 0    50   Output ~ 0
 GPS_SCL
@@
 ~RST
 Wire Wire Line
-	6900 2900 7200 2900
-Wire Wire Line
 	5350 1500 5500 1500
 Connection ~ 5500 1500
@@
 Wire Wire Line
 	5800 1500 6100 1500
-Text Label 6900 2900 0    50   ~ 0
+Text Label 7150 2900 0    50   ~ 0
 GPS_RF
 Wire Wire Line
@@
 Wire Wire Line
 	3500 2700 4600 2700
+$Comp
+L Device:L L2
+U 1 1 604CED70
+P 7100 2500
+F 0 "L2" V 6919 2500 50  0000 C CNN
+F 1 "47n" V 7010 2500 50  0000 C CNN
+F 2 "Inductor_SMD:L_0603_1608Metric" H 7100 2500 50  0001 C CNN
+F 3 "~" H 7100 2500 50  0001 C CNN
+	1    7100 2500
+	1    0    0    -1
+$EndComp
+$Comp
+L Device:C C26
+U 1 1 604CFCD6
+P 7450 2400
+F 0 "C26" H 7565 2446 50  0000 L CNN
+F 1 "47n" H 7565 2355 50  0000 L CNN
+F 2 "Capacitor_SMD:C_0603_1608Metric" H 7488 2250 50  0001 C CNN
+F 3 "~" H 7450 2400 50  0001 C CNN
+	1    7450 2400
+	1    0    0    -1
+$EndComp
+$Comp
+L power:GND #PWR060
+U 1 1 604D177C
+P 7450 2550
+F 0 "#PWR060" H 7450 2300 50  0001 C CNN
+F 1 "GND" H 7455 2377 50  0000 C CNN
+F 2 "" H 7450 2550 50  0001 C CNN
+F 3 "" H 7450 2550 50  0001 C CNN
+	1    7450 2550
+	1    0    0    -1
+$EndComp
+$Comp
+L power:+3.3V #PWR059
+U 1 1 604D57DA
+P 7100 2050
+F 0 "#PWR059" H 7100 1900 50  0001 C CNN
+F 1 "+3.3V" H 7115 2223 50  0000 C CNN
+F 2 "" H 7100 2050 50  0001 C CNN
+F 3 "" H 7100 2050 50  0001 C CNN
+	1    7100 2050
+	1    0    0    -1
+$EndComp
+Wire Wire Line
+	6900 2900 7100 2900
+Wire Wire Line
+	7100 2650 7100 2900
+Connection ~ 7100 2900
+Wire Wire Line
+	7100 2900 7450 2900
+Wire Wire Line
+	7450 2250 7100 2250
+Wire Wire Line
+	7100 2250 7100 2350
+Wire Wire Line
+	7100 2050 7100 2250
+Connection ~ 7100 2250
+$Comp
+L Device:C C27
+U 1 1 604D94D9
+P 7850 2400
+F 0 "C27" H 7965 2446 50  0000 L CNN
+F 1 "1n" H 7965 2355 50  0000 L CNN
+F 2 "Capacitor_SMD:C_0603_1608Metric" H 7888 2250 50  0001 C CNN
+F 3 "~" H 7850 2400 50  0001 C CNN
+	1    7850 2400
+	1    0    0    -1
+$EndComp
+Wire Wire Line
+	7450 2250 7850 2250
+Connection ~ 7450 2250
+$Comp
+L power:GND #PWR083
+U 1 1 604DA618
+P 7850 2550
+F 0 "#PWR083" H 7850 2300 50  0001 C CNN
+F 1 "GND" H 7855 2377 50  0000 C CNN
+F 2 "" H 7850 2550 50  0001 C CNN
+F 3 "" H 7850 2550 50  0001 C CNN
+	1    7850 2550
+	1    0    0    -1
+$EndComp
 $EndSCHEMATC

Commit message: Replaced IMU, relays, and power regulator with new components. Modified schematic accordingly.
Parts:
- renumbered C25 to C23, C26 to C24, C27 to C25, J10 to J9, R22 to R16, U7 to U9
Changed lines of the file:
@@
 $EndDescr
 $Comp
-L CAM-M8:CAM-M8 U7
+L CAM-M8:CAM-M8 U9
 U 1 1 5FCE2632
 P 6000 3000
-F 0 "U7" H 6000 3000 50  0001 L BNN
+F 0 "U9" H 6000 3000 50  0001 L BNN
 F 1 "CAM-M8" H 6000 3000 50  0001 L BNN
 F 2 "Parts:CAM-M8" H 6000 3000 50  0001 L BNN
@@
 $EndComp
 $Comp
-L power:GND #PWR087
+L power:GND #PWR077
 U 1 1 5FCF463B
 P 5100 4600
-F 0 "#PWR087" H 5100 4350 50  0001 C CNN
+F 0 "#PWR077" H 5100 4350 50  0001 C CNN
 F 1 "GND" H 5105 4427 50  0000 C CNN
 F 2 "" H 5100 4600 50  0001 C CNN
@@
 Connection ~ 6300 4550
 $Comp
-L Device:C C25
+L Device:C C23
 U 1 1 5FCFD1D5
 P 5350 1650
-F 0 "C25" H 5550 1700 50  0000 C CNN
+F 0 "C23" H 5550 1700 50  0000 C CNN
 F 1 "4.7u" H 5550 1600 50  0000 C CNN
 F 2 "Capacitor_SMD:C_0603_1608Metric" H 5388 1500 50  0001 C CNN
@@
 $EndComp
 $Comp
-L power:GND #PWR082
+L power:GND #PWR071
 U 1 1 5FCFFDB2
 P 5350 1800
-F 0 "#PWR082" H 5350 1550 50  0001 C CNN
+F 0 "#PWR071" H 5350 1550 50  0001 C CNN
 F 1 "GND" H 5355 1627 50  0000 C CNN
 F 2 "" H 5350 1800 50  0001 C CNN
@@
 NoConn ~ 4600 2900
 $Comp
-L power:+3.3V #PWR081
+L power:+3.3V #PWR070
 U 1 1 5FCDA81D
 P 5500 1500
-F 0 "#PWR081" H 5500 1350 50  0001 C CNN
+F 0 "#PWR070" H 5500 1350 50  0001 C CNN
 F 1 "+3.3V" H 5515 1673 50  0000 C CNN
 F 2 "" H 5500 1500 50  0001 C CNN
@@
 $EndComp
 $Comp
-L CON-SMA-EDGE-S:CON-SMA-EDGE-S J10
+L CON-SMA-EDGE-S:CON-SMA-EDGE-S J9
 U 1 1 5FCDAE06
 P 7550 3000
-F 0 "J10" H 7390 2994 50  0000 R CNN
+F 0 "J9" H 7390 2994 50  0000 R CNN
 F 1 "SMA_GPS" H 7390 3085 50  0000 R CNN
 F 2 "Parts:RFSOLUTIONS_CON-SMA-EDGE-S" H 7550 3000 50  0001 L BNN
@@
 $EndComp
 $Comp
-L power:GND #PWR085
+L power:GND #PWR075
 U 1 1 5FCDC46C
 P 7450 3100
-F 0 "#PWR085" H 7450 2850 50  0001 C CNN
+F 0 "#PWR075" H 7450 2850 50  0001 C CNN
 F 1 "GND" H 7455 2927 50  0000 C CNN
 F 2 "" H 7450 3100 50  0001 C CNN
@@
 GPS_SDA
 $Comp
-L power:+3.3V #PWR086
+L power:+3.3V #PWR076
 U 1 1 5FCF68E0
 P 3750 3600
-F 0 "#PWR086" H 3750 3450 50  0001 C CNN
+F 0 "#PWR076" H 3750 3450 50  0001 C CNN
 F 1 "+3.3V" H 3765 3773 50  0000 C CNN
 F 2 "" H 3750 3600 50  0001 C CNN
@@
 $EndComp
 $Comp
-L Device:R_US R22
+L Device:R_US R16
 U 1 1 5FCF6C65
 P 3750 3750
-F 0 "R22" H 3818 3796 50  0000 L CNN
+F 0 "R16" H 3818 3796 50  0000 L CNN
 F 1 "2.2k" H 3818 3705 50  0000 L CNN
 F 2 "Resistor_SMD:R_0603_1608Metric" V 3790 3740 50  0001 C CNN
@@
 $EndComp
 $Comp
-L Device:C C26
+L Device:C C24
 U 1 1 604CFCD6
 P 7450 2400
-F 0 "C26" H 7565 2446 50  0000 L CNN
+F 0 "C24" H 7565 2446 50  0000 L CNN
 F 1 "47n" H 7565 2355 50  0000 L CNN
 F 2 "Capacitor_SMD:C_0603_1608Metric" H 7488 2250 50  0001 C CNN
@@
 $EndComp
 $Comp
-L power:GND #PWR060
+L power:GND #PWR073
 U 1 1 604D177C
 P 7450 2550
-F 0 "#PWR060" H 7450 2300 50  0001 C CNN
+F 0 "#PWR073" H 7450 2300 50  0001 C CNN
 F 1 "GND" H 7455 2377 50  0000 C CNN
 F 2 "" H 7450 2550 50  0001 C CNN
@@
 $EndComp
 $Comp
-L power:+3.3V #PWR059
+L power:+3.3V #PWR072
 U 1 1 604D57DA
 P 7100 2050
-F 0 "#PWR059" H 7100 1900 50  0001 C CNN
+F 0 "#PWR072" H 7100 1900 50  0001 C CNN
 F 1 "+3.3V" H 7115 2223 50  0000 C CNN
 F 2 "" H 7100 2050 50  0001 C CNN
@@
 Connection ~ 7100 2250
 $Comp
-L Device:C C27
+L Device:C C25
 U 1 1 604D94D9
 P 7850 2400
-F 0 "C27" H 7965 2446 50  0000 L CNN
+F 0 "C25" H 7965 2446 50  0000 L CNN
 F 1 "1n" H 7965 2355 50  0000 L CNN
 F 2 "Capacitor_SMD:C_0603_1608Metric" H 7888 2250 50  0001 C CNN
@@
 Connection ~ 7450 2250
 $Comp
-L power:GND #PWR083
+L power:GND #PWR074
 U 1 1 604DA618
 P 7850 2550
-F 0 "#PWR083" H 7850 2300 50  0001 C CNN
+F 0 "#PWR074" H 7850 2300 50  0001 C CNN
 F 1 "GND" H 7855 2377 50  0000 C CNN
 F 2 "" H 7850 2550 50  0001 C CNN
