File: Recovery PCB/radio-915-lora.sch (KiCad schematic (older format))
At the start: 5 parts

Commit message: Updated recovery board with new connections.
Parts:
- removed U?: RFM95W-915S2, symbol RF_AM_FM:RFM95W-915S2
- added U?: RFM95W-915S2, symbol RF_Module:RFM95W-915S2
Changed lines of the file:
@@
 EESchema Schematic File Version 4
 LIBS:Recovery PCB-cache
-EELAYER 26 0
+EELAYER 30 0
 EELAYER END
 $Descr A4 11693 8268
@@
 Comment4 ""
 $EndDescr
-$Comp
-L RF_AM_FM:RFM95W-915S2 U?
-U 1 1 5E277423
-P 4550 2900
-F 0 "U?" H 4550 3578 50  0000 C CNN
-F 1 "RFM95W-915S2" H 4550 3487 50  0000 C CNN
-F 2 "" H 1250 4550 50  0001 C CNN
-F 3 "http://www.hoperf.com/upload/rf/RFM95_96_97_98W.pdf" H 1250 4550 50  0001 C CNN
-	1    4550 2900
-	1    0    0    -1
-$EndComp
 $Comp
 L Device:C C?
@@
 NoConn ~ 5050 3100
 NoConn ~ 5050 3200
+$Comp
+L RF_Module:RFM95W-915S2 U?
+U 1 1 5E548A5D
+P 4550 2900
+F 0 "U?" H 4550 3581 50  0000 C CNN
+F 1 "RFM95W-915S2" H 4550 3490 50  0000 C CNN
+F 2 "" H 1250 4550 50  0001 C CNN
+F 3 "https://www.hoperf.com/data/upload/portal/20181127/5bfcbea20e9ef.pdf" H 1250 4550 50  0001 C CNN
+	1    4550 2900
+	1    0    0    -1
+$EndComp
 $EndSCHEMATC

Commit message: Update relays and re-annotate entire schematic. Review needed before layout.
Parts:
- gave numbers to parts that had none: 5
Changed lines of the file:
@@
 $EndDescr
 $Comp
-L Device:C C?
+L Device:C C21
 U 1 1 5E279029
 P 3650 2400
-F 0 "C?" V 3398 2400 50  0000 C CNN
+F 0 "C21" V 3398 2400 50  0000 C CNN
 F 1 "0.1u" V 3489 2400 50  0000 C CNN
 F 2 "" H 3688 2250 50  0001 C CNN
@@
 $EndComp
 $Comp
-L power:GND #PWR?
+L power:GND #PWR043
 U 1 1 5E2791B0
 P 3500 2400
-F 0 "#PWR?" H 3500 2150 50  0001 C CNN
+F 0 "#PWR043" H 3500 2150 50  0001 C CNN
 F 1 "GND" H 3505 2227 50  0000 C CNN
 F 2 "" H 3500 2400 50  0001 C CNN
@@
 $EndComp
 $Comp
-L power:+3.3V #PWR?
+L power:+3.3V #PWR044
 U 1 1 5E2795E6
 P 4050 2300
-F 0 "#PWR?" H 4050 2150 50  0001 C CNN
+F 0 "#PWR044" H 4050 2150 50  0001 C CNN
 F 1 "+3.3V" H 4065 2473 50  0000 C CNN
 F 2 "" H 4050 2300 50  0001 C CNN
@@
 $EndComp
 $Comp
-L Device:Antenna AE?
+L Device:Antenna AE1
 U 1 1 5E279E92
 P 5250 2400
-F 0 "AE?" H 5330 2391 50  0000 L CNN
+F 0 "AE1" H 5330 2391 50  0000 L CNN
 F 1 "Antenna" H 5330 2300 50  0000 L CNN
 F 2 "" H 5250 2400 50  0001 C CNN
@@
 	4550 3500 4650 3500
 $Comp
-L power:GND #PWR?
+L power:GND #PWR045
 U 1 1 5E27A0D3
 P 4550 3500
-F 0 "#PWR?" H 4550 3250 50  0001 C CNN
+F 0 "#PWR045" H 4550 3250 50  0001 C CNN
 F 1 "GND" H 4555 3327 50  0000 C CNN
 F 2 "" H 4550 3500 50  0001 C CNN
@@
 	2950 2900 3150 2900
 $Comp
-L Device:R R?
+L Device:R R15
 U 1 1 5E27AC84
 P 3150 2750
-F 0 "R?" H 3220 2796 50  0000 L CNN
+F 0 "R15" H 3220 2796 50  0000 L CNN
 F 1 "100k" H 3220 2705 50  0000 L CNN
 F 2 "" V 3080 2750 50  0001 C CNN
@@
 	3150 2900 4050 2900
 $Comp
-L power:+3.3V #PWR?
+L power:+3.3V #PWR042
 U 1 1 5E27AD48
 P 3150 2600
-F 0 "#PWR?" H 3150 2450 50  0001 C CNN
+F 0 "#PWR042" H 3150 2450 50  0001 C CNN
 F 1 "+3.3V" H 3165 2773 50  0000 C CNN
 F 2 "" H 3150 2600 50  0001 C CNN
@@
 	2150 3100 2300 3100
 $Comp
-L Device:R R?
+L Device:R R14
 U 1 1 5E27AF7C
 P 2300 2950
-F 0 "R?" H 2370 2996 50  0000 L CNN
+F 0 "R14" H 2370 2996 50  0000 L CNN
 F 1 "100k" H 2370 2905 50  0000 L CNN
 F 2 "" V 2230 2950 50  0001 C CNN
@@
 	2300 3100 4050 3100
 $Comp
-L power:+3.3V #PWR?
+L power:+3.3V #PWR041
 U 1 1 5E27AFBB
 P 2300 2800
-F 0 "#PWR?" H 2300 2650 50  0001 C CNN
+F 0 "#PWR041" H 2300 2650 50  0001 C CNN
 F 1 "+3.3V" H 2315 2973 50  0000 C CNN
 F 2 "" H 2300 2800 50  0001 C CNN
@@
 NoConn ~ 5050 3200
 $Comp
-L RF_Module:RFM95W-915S2 U?
+L RF_Module:RFM95W-915S2 U6
 U 1 1 5E548A5D
 P 4550 2900
-F 0 "U?" H 4550 3581 50  0000 C CNN
+F 0 "U6" H 4550 3581 50  0000 C CNN
 F 1 "RFM95W-915S2" H 4550 3490 50  0000 C CNN
 F 2 "" H 1250 4550 50  0001 C CNN

Commit message: Added footprints.
Added footprints for various parts. Still need to update some more and calculate some values.
Parts:
- removed AE1: Antenna, symbol Device:Antenna
- removed R14, R15: 100k, symbol Device:R
- added J7: Conn_Coaxial, symbol Connector:Conn_Coaxial
- added R16, R17: 100k, Resistor_SMD:R_0603_1608Metric, symbol Device:R_US
- C21: footprint (none) -> Capacitor_SMD:C_0603_1608Metric
Changed lines of the file:
@@
 F 0 "C21" V 3398 2400 50  0000 C CNN
 F 1 "0.1u" V 3489 2400 50  0000 C CNN
-F 2 "" H 3688 2250 50  0001 C CNN
+F 2 "Capacitor_SMD:C_0603_1608Metric" H 3688 2250 50  0001 C CNN
 F 3 "~" H 3650 2400 50  0001 C CNN
 	1    3650 2400
@@
 $EndComp
 $Comp
-L power:GND #PWR043
+L power:GND #PWR047
 U 1 1 5E2791B0
 P 3500 2400
-F 0 "#PWR043" H 3500 2150 50  0001 C CNN
+F 0 "#PWR047" H 3500 2150 50  0001 C CNN
 F 1 "GND" H 3505 2227 50  0000 C CNN
 F 2 "" H 3500 2400 50  0001 C CNN
@@
 $EndComp
 $Comp
-L power:+3.3V #PWR044
+L power:+3.3V #PWR048
 U 1 1 5E2795E6
 P 4050 2300
-F 0 "#PWR044" H 4050 2150 50  0001 C CNN
+F 0 "#PWR048" H 4050 2150 50  0001 C CNN
 F 1 "+3.3V" H 4065 2473 50  0000 C CNN
 F 2 "" H 4050 2300 50  0001 C CNN
 F 3 "" H 4050 2300 50  0001 C CNN
 	1    4050 2300
-	1    0    0    -1
-$EndComp
-$Comp
-L Device:Antenna AE1
-U 1 1 5E279E92
-P 5250 2400
-F 0 "AE1" H 5330 2391 50  0000 L CNN
-F 1 "Antenna" H 5330 2300 50  0000 L CNN
-F 2 "" H 5250 2400 50  0001 C CNN
-F 3 "~" H 5250 2400 50  0001 C CNN
-	1    5250 2400
 	1    0    0    -1
 $EndComp
@@
 	4550 3500 4650 3500
 $Comp
-L power:GND #PWR045
+L power:GND #PWR049
 U 1 1 5E27A0D3
 P 4550 3500
-F 0 "#PWR045" H 4550 3250 50  0001 C CNN
+F 0 "#PWR049" H 4550 3250 50  0001 C CNN
 F 1 "GND" H 4555 3327 50  0000 C CNN
 F 2 "" H 4550 3500 50  0001 C CNN
@@
 Text HLabel 2950 2900 0    50   Input ~ 0
 RADIO_SS
-Wire Wire Line
-	2950 2900 3150 2900
 $Comp
-L Device:R R15
-U 1 1 5E27AC84
-P 3150 2750
-F 0 "R15" H 3220 2796 50  0000 L CNN
-F 1 "100k" H 3220 2705 50  0000 L CNN
-F 2 "" V 3080 2750 50  0001 C CNN
-F 3 "~" H 3150 2750 50  0001 C CNN
-	1    3150 2750
-	1    0    0    -1
-$EndComp
-Connection ~ 3150 2900
-Wire Wire Line
-	3150 2900 4050 2900
-$Comp
-L power:+3.3V #PWR042
+L power:+3.3V #PWR046
 U 1 1 5E27AD48
 P 3150 2600
-F 0 "#PWR042" H 3150 2450 50  0001 C CNN
+F 0 "#PWR046" H 3150 2450 50  0001 C CNN
 F 1 "+3.3V" H 3165 2773 50  0000 C CNN
 F 2 "" H 3150 2600 50  0001 C CNN
@@
 Text HLabel 2150 3100 0    50   Input ~ 0
 RADIO_RESET
-Wire Wire Line
-	2150 3100 2300 3100
 $Comp
-L Device:R R14
-U 1 1 5E27AF7C
-P 2300 2950
-F 0 "R14" H 2370 2996 50  0000 L CNN
-F 1 "100k" H 2370 2905 50  0000 L CNN
-F 2 "" V 2230 2950 50  0001 C CNN
-F 3 "~" H 2300 2950 50  0001 C CNN
-	1    2300 2950
-	1    0    0    -1
-$EndComp
-Connection ~ 2300 3100
-Wire Wire Line
-	2300 3100 4050 3100
-$Comp
-L power:+3.3V #PWR041
+L power:+3.3V #PWR045
 U 1 1 5E27AFBB
 P 2300 2800
-F 0 "#PWR041" H 2300 2650 50  0001 C CNN
+F 0 "#PWR045" H 2300 2650 50  0001 C CNN
 F 1 "+3.3V" H 2315 2973 50  0000 C CNN
 F 2 "" H 2300 2800 50  0001 C CNN
@@
 	1    0    0    -1
 $EndComp
+$Comp
+L Connector:Conn_Coaxial J7
+U 1 1 5E64A4C7
+P 5450 2600
+F 0 "J7" H 5550 2575 50  0000 L CNN
+F 1 "Conn_Coaxial" H 5550 2484 50  0000 L CNN
+F 2 "" H 5450 2600 50  0001 C CNN
+F 3 " ~" H 5450 2600 50  0001 C CNN
+	1    5450 2600
+	1    0    0    -1
+$EndComp
+$Comp
+L power:GND #PWR050
+U 1 1 5E64BA69
+P 5450 2800
+F 0 "#PWR050" H 5450 2550 50  0001 C CNN
+F 1 "GND" H 5455 2627 50  0000 C CNN
+F 2 "" H 5450 2800 50  0001 C CNN
+F 3 "" H 5450 2800 50  0001 C CNN
+	1    5450 2800
+	1    0    0    -1
+$EndComp
+$Comp
+L Device:R_US R16
+U 1 1 5E64C0ED
+P 2300 2950
+F 0 "R16" H 2368 2996 50  0000 L CNN
+F 1 "100k" H 2368 2905 50  0000 L CNN
+F 2 "Resistor_SMD:R_0603_1608Metric" V 2340 2940 50  0001 C CNN
+F 3 "~" H 2300 2950 50  0001 C CNN
+	1    2300 2950
+	1    0    0    -1
+$EndComp
+$Comp
+L Device:R_US R17
+U 1 1 5E64C425
+P 3150 2750
+F 0 "R17" H 3218 2796 50  0000 L CNN
+F 1 "100k" H 3218 2705 50  0000 L CNN
+F 2 "Resistor_SMD:R_0603_1608Metric" V 3190 2740 50  0001 C CNN
+F 3 "~" H 3150 2750 50  0001 C CNN
+	1    3150 2750
+	1    0    0    -1
+$EndComp
+Wire Wire Line
+	2150 3100 2300 3100
+Wire Wire Line
+	2950 2900 3150 2900
+Connection ~ 2300 3100
+Wire Wire Line
+	2300 3100 4050 3100
+Connection ~ 3150 2900
+Wire Wire Line
+	3150 2900 4050 2900
 $EndSCHEMATC

Commit message: Updated some footprints and re-annotated schematic.
Parts:
- J8: renamed from J7; footprint (none) -> Connector_Coaxial:U.FL_Molex_MCRF_73412-0110_Vertical
- renumbered C21 to C23, R16 to R17, R17 to R18
Changed lines of the file:
@@
 EESchema Schematic File Version 4
-LIBS:Recovery PCB-cache
-EELAYER 26 0
+EELAYER 30 0
 EELAYER END
 $Descr A4 11693 8268
@@
 $EndDescr
 $Comp
-L Device:C C21
+L Device:C C23
 U 1 1 5E279029
 P 3650 2400
-F 0 "C21" V 3398 2400 50  0000 C CNN
+F 0 "C23" V 3398 2400 50  0000 C CNN
 F 1 "0.1u" V 3489 2400 50  0000 C CNN
 F 2 "Capacitor_SMD:C_0603_1608Metric" H 3688 2250 50  0001 C CNN
@@
 $EndComp
 $Comp
-L power:GND #PWR047
+L power:GND #PWR056
 U 1 1 5E2791B0
 P 3500 2400
-F 0 "#PWR047" H 3500 2150 50  0001 C CNN
+F 0 "#PWR056" H 3500 2150 50  0001 C CNN
 F 1 "GND" H 3505 2227 50  0000 C CNN
 F 2 "" H 3500 2400 50  0001 C CNN
@@
 $EndComp
 $Comp
-L power:+3.3V #PWR048
+L power:+3.3V #PWR057
 U 1 1 5E2795E6
 P 4050 2300
-F 0 "#PWR048" H 4050 2150 50  0001 C CNN
+F 0 "#PWR057" H 4050 2150 50  0001 C CNN
 F 1 "+3.3V" H 4065 2473 50  0000 C CNN
 F 2 "" H 4050 2300 50  0001 C CNN
@@
 	4550 3500 4650 3500
 $Comp
-L power:GND #PWR049
+L power:GND #PWR058
 U 1 1 5E27A0D3
 P 4550 3500
-F 0 "#PWR049" H 4550 3250 50  0001 C CNN
+F 0 "#PWR058" H 4550 3250 50  0001 C CNN
 F 1 "GND" H 4555 3327 50  0000 C CNN
 F 2 "" H 4550 3500 50  0001 C CNN
@@
 RADIO_SS
 $Comp
-L power:+3.3V #PWR046
+L power:+3.3V #PWR055
 U 1 1 5E27AD48
 P 3150 2600
-F 0 "#PWR046" H 3150 2450 50  0001 C CNN
+F 0 "#PWR055" H 3150 2450 50  0001 C CNN
 F 1 "+3.3V" H 3165 2773 50  0000 C CNN
 F 2 "" H 3150 2600 50  0001 C CNN
@@
 RADIO_RESET
 $Comp
-L power:+3.3V #PWR045
+L power:+3.3V #PWR054
 U 1 1 5E27AFBB
 P 2300 2800
-F 0 "#PWR045" H 2300 2650 50  0001 C CNN
+F 0 "#PWR054" H 2300 2650 50  0001 C CNN
 F 1 "+3.3V" H 2315 2973 50  0000 C CNN
 F 2 "" H 2300 2800 50  0001 C CNN
@@
 $EndComp
 $Comp
-L Connector:Conn_Coaxial J7
+L Connector:Conn_Coaxial J8
 U 1 1 5E64A4C7
 P 5450 2600
-F 0 "J7" H 5550 2575 50  0000 L CNN
+F 0 "J8" H 5550 2575 50  0000 L CNN
 F 1 "Conn_Coaxial" H 5550 2484 50  0000 L CNN
-F 2 "" H 5450 2600 50  0001 C CNN
+F 2 "Connector_Coaxial:U.FL_Molex_MCRF_73412-0110_Vertical" H 5450 2600 50  0001 C CNN
 F 3 " ~" H 5450 2600 50  0001 C CNN
 	1    5450 2600
@@
 $EndComp
 $Comp
-L power:GND #PWR050
+L power:GND #PWR059
 U 1 1 5E64BA69
 P 5450 2800
-F 0 "#PWR050" H 5450 2550 50  0001 C CNN
+F 0 "#PWR059" H 5450 2550 50  0001 C CNN
 F 1 "GND" H 5455 2627 50  0000 C CNN
 F 2 "" H 5450 2800 50  0001 C CNN
@@
 $EndComp
 $Comp
-L Device:R_US R16
+L Device:R_US R17
 U 1 1 5E64C0ED
 P 2300 2950
-F 0 "R16" H 2368 2996 50  0000 L CNN
+F 0 "R17" H 2368 2996 50  0000 L CNN
 F 1 "100k" H 2368 2905 50  0000 L CNN
 F 2 "Resistor_SMD:R_0603_1608Metric" V 2340 2940 50  0001 C CNN
@@
 $EndComp
 $Comp
-L Device:R_US R17
+L Device:R_US R18
 U 1 1 5E64C425
 P 3150 2750
-F 0 "R17" H 3218 2796 50  0000 L CNN
+F 0 "R18" H 3218 2796 50  0000 L CNN
 F 1 "100k" H 3218 2705 50  0000 L CNN
 F 2 "Resistor_SMD:R_0603_1608Metric" V 3190 2740 50  0001 C CNN

Commit message: Added missing footprints and replaced GPS module.
Parts:
- removed J8: Conn_Coaxial, Connector_Coaxial:U.FL_Molex_MCRF_73412-0110_Vertical, symbol Connector:Conn_Coaxial
- added J8: CON-SMA-EDGE-S, RFSOLUTIONS_CON-SMA-EDGE-S, symbol CON-SMA-EDGE-S:CON-SMA-EDGE-S
- renumbered U6 to U7
Connections:
- wire segments 10 -> 11
Changed lines of the file:
@@
 NoConn ~ 5050 3200
 $Comp
-L RF_Module:RFM95W-915S2 U6
+L RF_Module:RFM95W-915S2 U7
 U 1 1 5E548A5D
 P 4550 2900
-F 0 "U6" H 4550 3581 50  0000 C CNN
+F 0 "U7" H 4550 3581 50  0000 C CNN
 F 1 "RFM95W-915S2" H 4550 3490 50  0000 C CNN
 F 2 "" H 1250 4550 50  0001 C CNN
 F 3 "https://www.hoperf.com/data/upload/portal/20181127/5bfcbea20e9ef.pdf" H 1250 4550 50  0001 C CNN
 	1    4550 2900
-	1    0    0    -1
-$EndComp
-$Comp
-L Connector:Conn_Coaxial J8
-U 1 1 5E64A4C7
-P 5450 2600
-F 0 "J8" H 5550 2575 50  0000 L CNN
-F 1 "Conn_Coaxial" H 5550 2484 50  0000 L CNN
-F 2 "Connector_Coaxial:U.FL_Molex_MCRF_73412-0110_Vertical" H 5450 2600 50  0001 C CNN
-F 3 " ~" H 5450 2600 50  0001 C CNN
-	1    5450 2600
-	1    0    0    -1
-$EndComp
-$Comp
-L power:GND #PWR059
-U 1 1 5E64BA69
-P 5450 2800
-F 0 "#PWR059" H 5450 2550 50  0001 C CNN
-F 1 "GND" H 5455 2627 50  0000 C CNN
-F 2 "" H 5450 2800 50  0001 C CNN
-F 3 "" H 5450 2800 50  0001 C CNN
-	1    5450 2800
 	1    0    0    -1
 $EndComp
@@
 Wire Wire Line
 	3150 2900 4050 2900
+$Comp
+L CON-SMA-EDGE-S:CON-SMA-EDGE-S J8
+U 1 1 5FCE5143
+P 5350 2700
+F 0 "J8" H 5342 3007 50  0000 C CNN
+F 1 "CON-SMA-EDGE-S" H 5342 2916 50  0000 C CNN
+F 2 "RFSOLUTIONS_CON-SMA-EDGE-S" H 5350 2700 50  0001 L BNN
+F 3 "" H 5350 2700 50  0001 L BNN
+F 4 "RF Solutions" H 5350 2700 50  0001 L BNN "MANUFACTURER"
+F 5 "1" H 5350 2700 50  0001 L BNN "PARTREV"
+F 6 "6.35mm" H 5350 2700 50  0001 L BNN "MAXIMUM_PACKAGE_HEIGHT"
+F 7 "Manufacturer Recommendations" H 5350 2700 50  0001 L BNN "STANDARD"
+	1    5350 2700
+	-1   0    0    -1
+$EndComp
+$Comp
+L power:GND #PWR059
+U 1 1 5FCEC316
+P 5250 2800
+F 0 "#PWR059" H 5250 2550 50  0001 C CNN
+F 1 "GND" H 5255 2627 50  0000 C CNN
+F 2 "" H 5250 2800 50  0001 C CNN
+F 3 "" H 5250 2800 50  0001 C CNN
+	1    5250 2800
+	1    0    0    -1
+$EndComp
+Wire Wire Line
+	5250 2700 5250 2800
 $EndSCHEMATC

Commit message: Finished Revision 1 of the Recovery PCB.
Parts:
- J8: footprint RFSOLUTIONS_CON-SMA-EDGE-S -> Parts:RFSOLUTIONS_CON-SMA-EDGE-S
- U7: footprint (none) -> RF_Module:HOPERF_RFM9XW_SMD
Changed lines of the file:
@@
 F 0 "U7" H 4550 3581 50  0000 C CNN
 F 1 "RFM95W-915S2" H 4550 3490 50  0000 C CNN
-F 2 "" H 1250 4550 50  0001 C CNN
+F 2 "RF_Module:HOPERF_RFM9XW_SMD" H 1250 4550 50  0001 C CNN
 F 3 "https://www.hoperf.com/data/upload/portal/20181127/5bfcbea20e9ef.pdf" H 1250 4550 50  0001 C CNN
 	1    4550 2900
@@
 F 0 "J8" H 5342 3007 50  0000 C CNN
 F 1 "CON-SMA-EDGE-S" H 5342 2916 50  0000 C CNN
-F 2 "RFSOLUTIONS_CON-SMA-EDGE-S" H 5350 2700 50  0001 L BNN
+F 2 "Parts:RFSOLUTIONS_CON-SMA-EDGE-S" H 5350 2700 50  0001 L BNN
 F 3 "" H 5350 2700 50  0001 L BNN
 F 4 "RF Solutions" H 5350 2700 50  0001 L BNN "MANUFACTURER"

Commit message: Recovery PCB: Redraw schematics
Redrew Recover PCB schematics to be more easily readable and fixed board
outline, adding netclasses to ease trace placement.
Parts:
- J8: value CON-SMA-EDGE-S -> SMA_LORA
Connections:
- net labels added: LoRa_RF
- wire segments 11 -> 13
Changed lines of the file:
@@
 L Device:C C23
 U 1 1 5E279029
-P 3650 2400
-F 0 "C23" V 3398 2400 50  0000 C CNN
-F 1 "0.1u" V 3489 2400 50  0000 C CNN
-F 2 "Capacitor_SMD:C_0603_1608Metric" H 3688 2250 50  0001 C CNN
-F 3 "~" H 3650 2400 50  0001 C CNN
-	1    3650 2400
-	0    1    1    0
+P 4400 2000
+F 0 "C23" H 4148 2000 50  0000 C CNN
+F 1 "0.1u" H 4150 1900 50  0000 C CNN
+F 2 "Capacitor_SMD:C_0603_1608Metric" H 4438 1850 50  0001 C CNN
+F 3 "~" H 4400 2000 50  0001 C CNN
+	1    4400 2000
+	1    0    0    -1
 $EndComp
 $Comp
 L power:GND #PWR056
 U 1 1 5E2791B0
-P 3500 2400
-F 0 "#PWR056" H 3500 2150 50  0001 C CNN
-F 1 "GND" H 3505 2227 50  0000 C CNN
-F 2 "" H 3500 2400 50  0001 C CNN
-F 3 "" H 3500 2400 50  0001 C CNN
-	1    3500 2400
+P 4400 2150
+F 0 "#PWR056" H 4400 1900 50  0001 C CNN
+F 1 "GND" H 4405 1977 50  0000 C CNN
+F 2 "" H 4400 2150 50  0001 C CNN
+F 3 "" H 4400 2150 50  0001 C CNN
+	1    4400 2150
 	1    0    0    -1
 $EndComp
@@
 L power:+3.3V #PWR057
 U 1 1 5E2795E6
-P 4050 2300
-F 0 "#PWR057" H 4050 2150 50  0001 C CNN
-F 1 "+3.3V" H 4065 2473 50  0000 C CNN
-F 2 "" H 4050 2300 50  0001 C CNN
-F 3 "" H 4050 2300 50  0001 C CNN
-	1    4050 2300
+P 4550 1850
+F 0 "#PWR057" H 4550 1700 50  0001 C CNN
+F 1 "+3.3V" H 4565 2023 50  0000 C CNN
+F 2 "" H 4550 1850 50  0001 C CNN
+F 3 "" H 4550 1850 50  0001 C CNN
+	1    4550 1850
 	1    0    0    -1
 $EndComp
-Wire Wire Line
-	3800 2400 4050 2400
-Connection ~ 4050 2400
-Wire Wire Line
-	4050 2400 4550 2400
-Wire Wire Line
-	4050 2300 4050 2400
-Wire Wire Line
-	5250 2600 5050 2600
 Wire Wire Line
 	4450 3500 4550 3500
@@
 	1    0    0    -1
 $EndComp
-Text HLabel 4050 2600 0    50   Input ~ 0
+Text HLabel 4000 2600 0    50   Input ~ 0
 RADIO_SCK
-Text HLabel 4050 2700 0    50   Input ~ 0
+Text HLabel 4000 2700 0    50   Input ~ 0
 RADIO_MOSI
-Text HLabel 4050 2800 0    50   Output ~ 0
+Text HLabel 4000 2800 0    50   Output ~ 0
 RADIO_MISO
 Text HLabel 2950 2900 0    50   Input ~ 0
@@
 U 1 1 5E548A5D
 P 4550 2900
-F 0 "U7" H 4550 3581 50  0000 C CNN
-F 1 "RFM95W-915S2" H 4550 3490 50  0000 C CNN
+F 0 "U7" H 4900 3700 50  0000 C CNN
+F 1 "RFM95W-915S2" H 5150 3600 50  0000 C CNN
 F 2 "RF_Module:HOPERF_RFM9XW_SMD" H 1250 4550 50  0001 C CNN
 F 3 "https://www.hoperf.com/data/upload/portal/20181127/5bfcbea20e9ef.pdf" H 1250 4550 50  0001 C CNN
@@
 L CON-SMA-EDGE-S:CON-SMA-EDGE-S J8
 U 1 1 5FCE5143
-P 5350 2700
-F 0 "J8" H 5342 3007 50  0000 C CNN
-F 1 "CON-SMA-EDGE-S" H 5342 2916 50  0000 C CNN
-F 2 "Parts:RFSOLUTIONS_CON-SMA-EDGE-S" H 5350 2700 50  0001 L BNN
-F 3 "" H 5350 2700 50  0001 L BNN
-F 4 "RF Solutions" H 5350 2700 50  0001 L BNN "MANUFACTURER"
-F 5 "1" H 5350 2700 50  0001 L BNN "PARTREV"
-F 6 "6.35mm" H 5350 2700 50  0001 L BNN "MAXIMUM_PACKAGE_HEIGHT"
-F 7 "Manufacturer Recommendations" H 5350 2700 50  0001 L BNN "STANDARD"
-	1    5350 2700
+P 5550 2700
+F 0 "J8" H 5542 3007 50  0000 C CNN
+F 1 "SMA_LORA" H 5542 2916 50  0000 C CNN
+F 2 "Parts:RFSOLUTIONS_CON-SMA-EDGE-S" H 5550 2700 50  0001 L BNN
+F 3 "" H 5550 2700 50  0001 L BNN
+F 4 "RF Solutions" H 5550 2700 50  0001 L BNN "MANUFACTURER"
+F 5 "1" H 5550 2700 50  0001 L BNN "PARTREV"
+F 6 "6.35mm" H 5550 2700 50  0001 L BNN "MAXIMUM_PACKAGE_HEIGHT"
+F 7 "Manufacturer Recommendations" H 5550 2700 50  0001 L BNN "STANDARD"
+	1    5550 2700
 	-1   0    0    -1
 $EndComp
@@
 L power:GND #PWR059
 U 1 1 5FCEC316
-P 5250 2800
-F 0 "#PWR059" H 5250 2550 50  0001 C CNN
-F 1 "GND" H 5255 2627 50  0000 C CNN
-F 2 "" H 5250 2800 50  0001 C CNN
-F 3 "" H 5250 2800 50  0001 C CNN
-	1    5250 2800
+P 5450 2800
+F 0 "#PWR059" H 5450 2550 50  0001 C CNN
+F 1 "GND" H 5455 2627 50  0000 C CNN
+F 2 "" H 5450 2800 50  0001 C CNN
+F 3 "" H 5450 2800 50  0001 C CNN
+	1    5450 2800
 	1    0    0    -1
 $EndComp
 Wire Wire Line
-	5250 2700 5250 2800
+	5450 2700 5450 2800
+Wire Wire Line
+	4400 1850 4550 1850
+Wire Wire Line
+	4550 1850 4550 2400
+Connection ~ 4550 1850
+Wire Wire Line
+	4000 2600 4050 2600
+Wire Wire Line
+	4000 2700 4050 2700
+Wire Wire Line
+	4000 2800 4050 2800
+Text Label 5050 2600 0    50   ~ 0
+LoRa_RF
+Wire Wire Line
+	5050 2600 5450 2600
 $EndSCHEMATC
