File: Recovery PCB/radio-915-lora.sch (KiCad schematic (older format))
At the start: 5 parts, among them J8 SMA_LORA, U7 RFM95W-915S2

Commit message: Recovery PCB: Reannotate
Reannotated schematic to fix reference numbering and keep reference
designators consistent.
Parts:
- renumbered C23 to C24, J8 to J9, R17 to R19, U7 to U6
Changed lines of the file:
@@
 $EndDescr
 $Comp
-L Device:C C23
+L Device:C C24
 U 1 1 5E279029
 P 4400 2000
-F 0 "C23" H 4148 2000 50  0000 C CNN
+F 0 "C24" H 4148 2000 50  0000 C CNN
 F 1 "0.1u" H 4150 1900 50  0000 C CNN
 F 2 "Capacitor_SMD:C_0603_1608Metric" H 4438 1850 50  0001 C CNN
@@
 $EndComp
 $Comp
-L power:GND #PWR056
+L power:GND #PWR076
 U 1 1 5E2791B0
 P 4400 2150
-F 0 "#PWR056" H 4400 1900 50  0001 C CNN
+F 0 "#PWR076" H 4400 1900 50  0001 C CNN
 F 1 "GND" H 4405 1977 50  0000 C CNN
 F 2 "" H 4400 2150 50  0001 C CNN
@@
 $EndComp
 $Comp
-L power:+3.3V #PWR057
+L power:+3.3V #PWR075
 U 1 1 5E2795E6
 P 4550 1850
-F 0 "#PWR057" H 4550 1700 50  0001 C CNN
+F 0 "#PWR075" H 4550 1700 50  0001 C CNN
 F 1 "+3.3V" H 4565 2023 50  0000 C CNN
 F 2 "" H 4550 1850 50  0001 C CNN
@@
 	4550 3500 4650 3500
 $Comp
-L power:GND #PWR058
+L power:GND #PWR080
 U 1 1 5E27A0D3
 P 4550 3500
-F 0 "#PWR058" H 4550 3250 50  0001 C CNN
+F 0 "#PWR080" H 4550 3250 50  0001 C CNN
 F 1 "GND" H 4555 3327 50  0000 C CNN
 F 2 "" H 4550 3500 50  0001 C CNN
@@
 RADIO_SS
 $Comp
-L power:+3.3V #PWR055
+L power:+3.3V #PWR077
 U 1 1 5E27AD48
 P 3150 2600
-F 0 "#PWR055" H 3150 2450 50  0001 C CNN
+F 0 "#PWR077" H 3150 2450 50  0001 C CNN
 F 1 "+3.3V" H 3165 2773 50  0000 C CNN
 F 2 "" H 3150 2600 50  0001 C CNN
@@
 RADIO_RESET
 $Comp
-L power:+3.3V #PWR054
+L power:+3.3V #PWR078
 U 1 1 5E27AFBB
 P 2300 2800
-F 0 "#PWR054" H 2300 2650 50  0001 C CNN
+F 0 "#PWR078" H 2300 2650 50  0001 C CNN
 F 1 "+3.3V" H 2315 2973 50  0000 C CNN
 F 2 "" H 2300 2800 50  0001 C CNN
@@
 NoConn ~ 5050 3200
 $Comp
-L RF_Module:RFM95W-915S2 U7
+L RF_Module:RFM95W-915S2 U6
 U 1 1 5E548A5D
 P 4550 2900
-F 0 "U7" H 4900 3700 50  0000 C CNN
+F 0 "U6" H 4900 3700 50  0000 C CNN
 F 1 "RFM95W-915S2" H 5150 3600 50  0000 C CNN
 F 2 "RF_Module:HOPERF_RFM9XW_SMD" H 1250 4550 50  0001 C CNN
@@
 $EndComp
 $Comp
-L Device:R_US R17
+L Device:R_US R19
 U 1 1 5E64C0ED
 P 2300 2950
-F 0 "R17" H 2368 2996 50  0000 L CNN
+F 0 "R19" H 2368 2996 50  0000 L CNN
 F 1 "100k" H 2368 2905 50  0000 L CNN
 F 2 "Resistor_SMD:R_0603_1608Metric" V 2340 2940 50  0001 C CNN
@@
 	3150 2900 4050 2900
 $Comp
-L CON-SMA-EDGE-S:CON-SMA-EDGE-S J8
+L CON-SMA-EDGE-S:CON-SMA-EDGE-S J9
 U 1 1 5FCE5143
 P 5550 2700
-F 0 "J8" H 5542 3007 50  0000 C CNN
+F 0 "J9" H 5542 3007 50  0000 C CNN
 F 1 "SMA_LORA" H 5542 2916 50  0000 C CNN
 F 2 "Parts:RFSOLUTIONS_CON-SMA-EDGE-S" H 5550 2700 50  0001 L BNN
@@
 $EndComp
 $Comp
-L power:GND #PWR059
+L power:GND #PWR079
 U 1 1 5FCEC316
 P 5450 2800
-F 0 "#PWR059" H 5450 2550 50  0001 C CNN
+F 0 "#PWR079" H 5450 2550 50  0001 C CNN
 F 1 "GND" H 5455 2627 50  0000 C CNN
 F 2 "" H 5450 2800 50  0001 C CNN

Commit message: Recovery PCB: Deleted excess pullup resistors, redid mounting holes.
Other:
- note added: "Active low, do not populate"
Changed lines of the file:
@@
 EESchema Schematic File Version 4
+LIBS:Recovery PCB-cache
 EELAYER 30 0
 EELAYER END
@@
 Wire Wire Line
 	5050 2600 5450 2600
+Text Notes 2700 2350 0    50   ~ 0
+Active low, do not populate
 $EndSCHEMATC

Commit message: Replaced IMU, relays, and power regulator with new components. Modified schematic accordingly.
Parts:
- renumbered C24 to C22, J9 to J8, R18 to R14, R19 to R15, U6 to U8
Changed lines of the file:
@@
 $EndDescr
 $Comp
-L Device:C C24
+L Device:C C22
 U 1 1 5E279029
 P 4400 2000
-F 0 "C24" H 4148 2000 50  0000 C CNN
+F 0 "C22" H 4148 2000 50  0000 C CNN
 F 1 "0.1u" H 4150 1900 50  0000 C CNN
 F 2 "Capacitor_SMD:C_0603_1608Metric" H 4438 1850 50  0001 C CNN
@@
 $EndComp
 $Comp
-L power:GND #PWR076
+L power:GND #PWR065
 U 1 1 5E2791B0
 P 4400 2150
-F 0 "#PWR076" H 4400 1900 50  0001 C CNN
+F 0 "#PWR065" H 4400 1900 50  0001 C CNN
 F 1 "GND" H 4405 1977 50  0000 C CNN
 F 2 "" H 4400 2150 50  0001 C CNN
@@
 $EndComp
 $Comp
-L power:+3.3V #PWR075
+L power:+3.3V #PWR064
 U 1 1 5E2795E6
 P 4550 1850
-F 0 "#PWR075" H 4550 1700 50  0001 C CNN
+F 0 "#PWR064" H 4550 1700 50  0001 C CNN
 F 1 "+3.3V" H 4565 2023 50  0000 C CNN
 F 2 "" H 4550 1850 50  0001 C CNN
@@
 	4550 3500 4650 3500
 $Comp
-L power:GND #PWR080
+L power:GND #PWR069
 U 1 1 5E27A0D3
 P 4550 3500
-F 0 "#PWR080" H 4550 3250 50  0001 C CNN
+F 0 "#PWR069" H 4550 3250 50  0001 C CNN
 F 1 "GND" H 4555 3327 50  0000 C CNN
 F 2 "" H 4550 3500 50  0001 C CNN
@@
 RADIO_SS
 $Comp
-L power:+3.3V #PWR077
+L power:+3.3V #PWR066
 U 1 1 5E27AD48
 P 3150 2600
-F 0 "#PWR077" H 3150 2450 50  0001 C CNN
+F 0 "#PWR066" H 3150 2450 50  0001 C CNN
 F 1 "+3.3V" H 3165 2773 50  0000 C CNN
 F 2 "" H 3150 2600 50  0001 C CNN
@@
 RADIO_RESET
 $Comp
-L power:+3.3V #PWR078
+L power:+3.3V #PWR067
 U 1 1 5E27AFBB
 P 2300 2800
-F 0 "#PWR078" H 2300 2650 50  0001 C CNN
+F 0 "#PWR067" H 2300 2650 50  0001 C CNN
 F 1 "+3.3V" H 2315 2973 50  0000 C CNN
 F 2 "" H 2300 2800 50  0001 C CNN
@@
 NoConn ~ 5050 3200
 $Comp
-L RF_Module:RFM95W-915S2 U6
+L RF_Module:RFM95W-915S2 U8
 U 1 1 5E548A5D
 P 4550 2900
-F 0 "U6" H 4900 3700 50  0000 C CNN
+F 0 "U8" H 4900 3700 50  0000 C CNN
 F 1 "RFM95W-915S2" H 5150 3600 50  0000 C CNN
 F 2 "RF_Module:HOPERF_RFM9XW_SMD" H 1250 4550 50  0001 C CNN
@@
 $EndComp
 $Comp
-L Device:R_US R19
+L Device:R_US R15
 U 1 1 5E64C0ED
 P 2300 2950
-F 0 "R19" H 2368 2996 50  0000 L CNN
+F 0 "R15" H 2368 2996 50  0000 L CNN
 F 1 "100k" H 2368 2905 50  0000 L CNN
 F 2 "Resistor_SMD:R_0603_1608Metric" V 2340 2940 50  0001 C CNN
@@
 $EndComp
 $Comp
-L Device:R_US R18
+L Device:R_US R14
 U 1 1 5E64C425
 P 3150 2750
-F 0 "R18" H 3218 2796 50  0000 L CNN
+F 0 "R14" H 3218 2796 50  0000 L CNN
 F 1 "100k" H 3218 2705 50  0000 L CNN
 F 2 "Resistor_SMD:R_0603_1608Metric" V 3190 2740 50  0001 C CNN
@@
 	3150 2900 4050 2900
 $Comp
-L CON-SMA-EDGE-S:CON-SMA-EDGE-S J9
+L CON-SMA-EDGE-S:CON-SMA-EDGE-S J8
 U 1 1 5FCE5143
 P 5550 2700
-F 0 "J9" H 5542 3007 50  0000 C CNN
+F 0 "J8" H 5542 3007 50  0000 C CNN
 F 1 "SMA_LORA" H 5542 2916 50  0000 C CNN
 F 2 "Parts:RFSOLUTIONS_CON-SMA-EDGE-S" H 5550 2700 50  0001 L BNN
@@
 $EndComp
 $Comp
-L power:GND #PWR079
+L power:GND #PWR068
 U 1 1 5FCEC316
 P 5450 2800
-F 0 "#PWR079" H 5450 2550 50  0001 C CNN
+F 0 "#PWR068" H 5450 2550 50  0001 C CNN
 F 1 "GND" H 5455 2627 50  0000 C CNN
 F 2 "" H 5450 2800 50  0001 C CNN
