File: Recovery PCB/IMU.sch (KiCad schematic (older format))
At the start: 13 parts, among them J1 Conn_01x02_Male, U3 BNO055, Y1 32.768k

Commit message: Updated recovery board with new connections.
Connections:
- net labels removed: ADDR
- wire segments 61 -> 62
Changed lines of the file:
@@
 EESchema Schematic File Version 4
 LIBS:Recovery PCB-cache
-EELAYER 26 0
+EELAYER 30 0
 EELAYER END
 $Descr A4 11693 8268
 encoding utf-8
-Sheet 4 8
+Sheet 6 8
 Title ""
 Date ""
@@
 Text HLabel 5350 3050 0    50   Input ~ 0
 nRESET
-Text HLabel 5450 4050 0    50   Input ~ 0
-ADDR
 Wire Wire Line
 	5450 3950 5100 3950
@@
 	1    0    0    -1
 $EndComp
+Wire Wire Line
+	5450 4050 5350 4050
+$Comp
+L power:GND #PWR?
+U 1 1 5E5F566F
+P 5350 4050
+F 0 "#PWR?" H 5350 3800 50  0001 C CNN
+F 1 "GND" H 5355 3877 50  0000 C CNN
+F 2 "" H 5350 4050 50  0001 C CNN
+F 3 "" H 5350 4050 50  0001 C CNN
+	1    5350 4050
+	1    0    0    -1
+$EndComp

Commit message: Update relays and re-annotate entire schematic. Review needed before layout.
Parts:
- renumbered C6 to C15, C7 to C16, C8 to C17, C9 to C18, C10 to C19, C11 to C20, J1 to J7, R3 to R10, R4 to R11, R5 to R12, R6 to R13, U3 to U5, Y1 to Y2
Changed lines of the file:
@@
 $EndDescr
 $Comp
-L power:+3.3V #PWR011
+L power:+3.3V #PWR035
 U 1 1 5DF02D6F
 P 4650 2500
-F 0 "#PWR011" H 4650 2350 50  0001 C CNN
+F 0 "#PWR035" H 4650 2350 50  0001 C CNN
 F 1 "+3.3V" H 4665 2673 50  0000 C CNN
 F 2 "" H 4650 2500 50  0001 C CNN
@@
 $EndComp
 $Comp
-L power:+3.3V #PWR010
+L power:+3.3V #PWR033
 U 1 1 5DF02F5F
 P 2950 2500
-F 0 "#PWR010" H 2950 2350 50  0001 C CNN
+F 0 "#PWR033" H 2950 2350 50  0001 C CNN
 F 1 "+3.3V" H 2965 2673 50  0000 C CNN
 F 2 "" H 2950 2500 50  0001 C CNN
@@
 $EndComp
 $Comp
-L power:GND #PWR012
+L power:GND #PWR038
 U 1 1 5DF0362D
 P 5950 4600
-F 0 "#PWR012" H 5950 4350 50  0001 C CNN
+F 0 "#PWR038" H 5950 4350 50  0001 C CNN
 F 1 "GND" H 5955 4427 50  0000 C CNN
 F 2 "" H 5950 4600 50  0001 C CNN
@@
 	5950 2850 5400 2850
 $Comp
-L Device:C C6
+L Device:C C15
 U 1 1 5DF03BA1
 P 5400 2700
-F 0 "C6" H 5515 2746 50  0000 L CNN
+F 0 "C15" H 5515 2746 50  0000 L CNN
 F 1 "0.1u" H 5515 2655 50  0000 L CNN
 F 2 "Capacitor_SMD:C_0603_1608Metric" H 5438 2550 50  0001 C CNN
@@
 INT
 $Comp
-L Device:R_US R6
+L Device:R_US R13
 U 1 1 5DF05E21
 P 4950 3250
-F 0 "R6" H 5018 3296 50  0000 L CNN
+F 0 "R13" H 5018 3296 50  0000 L CNN
 F 1 "4.7k" H 5018 3205 50  0000 L CNN
 F 2 "Resistor_SMD:R_0603_1608Metric" V 4990 3240 50  0001 C CNN
@@
 $EndComp
 $Comp
-L Device:C C7
+L Device:C C16
 U 1 1 5DF0775A
 P 6750 4200
-F 0 "C7" H 6865 4246 50  0000 L CNN
+F 0 "C16" H 6865 4246 50  0000 L CNN
 F 1 "0.1u" H 6865 4155 50  0000 L CNN
 F 2 "Capacitor_SMD:C_0603_1608Metric" H 6788 4050 50  0001 C CNN
@@
 	5950 4450 5950 4600
 $Comp
-L Sensor_Motion:BNO055 U3
+L Sensor_Motion:BNO055 U5
 U 1 1 5DF00E39
 P 6050 3550
-F 0 "U3" H 6050 4431 50  0000 C CNN
+F 0 "U5" H 6050 4431 50  0000 C CNN
 F 1 "BNO055" H 6050 4340 50  0000 C CNN
 F 2 "Package_LGA:LGA-28_5.2x3.8mm_P0.5mm" H 6300 2900 50  0001 L CNN
@@
 	5450 3750 3950 3750
 $Comp
-L Device:R_US R5
+L Device:R_US R12
 U 1 1 5DF0FA82
 P 3950 3200
-F 0 "R5" H 4018 3246 50  0000 L CNN
+F 0 "R12" H 4018 3246 50  0000 L CNN
 F 1 "4.7k" H 4018 3155 50  0000 L CNN
 F 2 "Resistor_SMD:R_0603_1608Metric" V 3990 3190 50  0001 C CNN
@@
 	3950 3350 3950 3750
 $Comp
-L Device:R_US R4
+L Device:R_US R11
 U 1 1 5DF109EE
 P 3550 3200
-F 0 "R4" H 3618 3246 50  0000 L CNN
+F 0 "R11" H 3618 3246 50  0000 L CNN
 F 1 "4.7k" H 3618 3155 50  0000 L CNN
 F 2 "Resistor_SMD:R_0603_1608Metric" V 3590 3190 50  0001 C CNN
@@
 	6150 4550 7950 4550
 $Comp
-L Device:C C11
+L Device:C C20
 U 1 1 5DF140F0
 P 8400 3600
-F 0 "C11" H 8515 3646 50  0000 L CNN
+F 0 "C20" H 8515 3646 50  0000 L CNN
 F 1 "6.8n" H 8515 3555 50  0000 L CNN
 F 2 "Capacitor_SMD:C_0603_1608Metric" H 8438 3450 50  0001 C CNN
@@
 $EndComp
 $Comp
-L Device:C C10
+L Device:C C19
 U 1 1 5DF1486E
 P 7950 3600
-F 0 "C10" H 8065 3646 50  0000 L CNN
+F 0 "C19" H 8065 3646 50  0000 L CNN
 F 1 "0.12u" H 8065 3555 50  0000 L CNN
 F 2 "Capacitor_SMD:C_0603_1608Metric" H 7988 3450 50  0001 C CNN
@@
 	6700 3450 6700 3550
 $Comp
-L Device:C C8
+L Device:C C17
 U 1 1 5DEDEF8B
 P 6950 3050
-F 0 "C8" V 6698 3050 50  0000 C CNN
+F 0 "C17" V 6698 3050 50  0000 C CNN
 F 1 "22p" V 6789 3050 50  0000 C CNN
 F 2 "Capacitor_SMD:C_0603_1608Metric" H 6988 2900 50  0001 C CNN
@@
 $EndComp
 $Comp
-L Device:C C9
+L Device:C C18
 U 1 1 5DEE0132
 P 6950 3550
-F 0 "C9" V 7100 3550 50  0000 C CNN
+F 0 "C18" V 7100 3550 50  0000 C CNN
 F 1 "22p" V 7200 3550 50  0000 C CNN
 F 2 "Capacitor_SMD:C_0603_1608Metric" H 6988 3400 50  0001 C CNN
@@
 $EndComp
 $Comp
-L Device:Crystal Y1
+L Device:Crystal Y2
 U 1 1 5DF0AC45
 P 6700 3300
-F 0 "Y1" V 6654 3431 50  0000 L CNN
+F 0 "Y2" V 6654 3431 50  0000 L CNN
 F 1 "32.768k" V 6745 3431 50  0000 L CNN
 F 2 "Crystal:Crystal_SMD_0603-2Pin_6.0x3.5mm" H 6700 3300 50  0001 C CNN
@@
 	7300 3550 7300 3600
 $Comp
-L power:GND #PWR013
+L power:GND #PWR039
 U 1 1 5DEE93BA
 P 7300 3600
-F 0 "#PWR013" H 7300 3350 50  0001 C CNN
+F 0 "#PWR039" H 7300 3350 50  0001 C CNN
 F 1 "GND" H 7305 3427 50  0000 C CNN
 F 2 "" H 7300 3600 50  0001 C CNN
@@
 $EndComp
 $Comp
-L Device:R_US R3
+L Device:R_US R10
 U 1 1 5DEF58D7
 P 3100 2800
-F 0 "R3" H 3168 2846 50  0000 L CNN
+F 0 "R10" H 3168 2846 50  0000 L CNN
 F 1 "4.7k" H 3168 2755 50  0000 L CNN
 F 2 "Resistor_SMD:R_0603_1608Metric" V 3140 2790 50  0001 C CNN
@@
 	7950 4550 8400 4550
 $Comp
-L Connector:Conn_01x02_Male J1
+L Connector:Conn_01x02_Male J7
 U 1 1 5DED60FE
 P 4400 3450
-F 0 "J1" H 4508 3631 50  0000 C CNN
+F 0 "J7" H 4508 3631 50  0000 C CNN
 F 1 "Conn_01x02_Male" H 4508 3540 50  0000 C CNN
 F 2 "Connector_PinHeader_1.00mm:PinHeader_1x02_P1.00mm_Vertical" H 4400 3450 50  0001 C CNN
@@
 	3950 3050 4950 3050
 $Comp
-L power:GND #PWR014
+L power:GND #PWR034
 U 1 1 5DEF0CA0
 P 4600 3550
-F 0 "#PWR014" H 4600 3300 50  0001 C CNN
+F 0 "#PWR034" H 4600 3300 50  0001 C CNN
 F 1 "GND" H 4750 3450 50  0000 C CNN
 F 2 "" H 4600 3550 50  0001 C CNN
@@
 	2950 3050 3550 3050
 $Comp
-L power:+3.3V #PWR015
+L power:+3.3V #PWR040
 U 1 1 5DEFA7ED
 P 8700 2850
-F 0 "#PWR015" H 8700 2700 50  0001 C CNN
+F 0 "#PWR040" H 8700 2700 50  0001 C CNN
 F 1 "+3.3V" H 8715 3023 50  0000 C CNN
 F 2 "" H 8700 2850 50  0001 C CNN
@@
 Connection ~ 5100 4550
 $Comp
-L power:GND #PWR020
+L power:GND #PWR036
 U 1 1 5DF41D8E
 P 5100 4600
-F 0 "#PWR020" H 5100 4350 50  0001 C CNN
+F 0 "#PWR036" H 5100 4350 50  0001 C CNN
 F 1 "GND" H 5105 4427 50  0000 C CNN
 F 2 "" H 5100 4600 50  0001 C CNN
@@
 	5450 4050 5350 4050
 $Comp
-L power:GND #PWR?
+L power:GND #PWR037
 U 1 1 5E5F566F
 P 5350 4050
-F 0 "#PWR?" H 5350 3800 50  0001 C CNN
+F 0 "#PWR037" H 5350 3800 50  0001 C CNN
 F 1 "GND" H 5355 3877 50  0000 C CNN
 F 2 "" H 5350 4050 50  0001 C CNN

Commit message: Added footprints.
Added footprints for various parts. Still need to update some more and calculate some values.
Parts:
- Y2: footprint Crystal:Crystal_SMD_0603-2Pin_6.0x3.5mm -> (none)
- renumbered J7 to J6, R10 to R12, R11 to R13, R12 to R14, R13 to R15
Changed lines of the file:
@@
 $EndDescr
 $Comp
-L power:+3.3V #PWR035
+L power:+3.3V #PWR039
 U 1 1 5DF02D6F
 P 4650 2500
-F 0 "#PWR035" H 4650 2350 50  0001 C CNN
+F 0 "#PWR039" H 4650 2350 50  0001 C CNN
 F 1 "+3.3V" H 4665 2673 50  0000 C CNN
 F 2 "" H 4650 2500 50  0001 C CNN
@@
 $EndComp
 $Comp
-L power:+3.3V #PWR033
+L power:+3.3V #PWR037
 U 1 1 5DF02F5F
 P 2950 2500
-F 0 "#PWR033" H 2950 2350 50  0001 C CNN
+F 0 "#PWR037" H 2950 2350 50  0001 C CNN
 F 1 "+3.3V" H 2965 2673 50  0000 C CNN
 F 2 "" H 2950 2500 50  0001 C CNN
@@
 $EndComp
 $Comp
-L power:GND #PWR038
+L power:GND #PWR042
 U 1 1 5DF0362D
 P 5950 4600
-F 0 "#PWR038" H 5950 4350 50  0001 C CNN
+F 0 "#PWR042" H 5950 4350 50  0001 C CNN
 F 1 "GND" H 5955 4427 50  0000 C CNN
 F 2 "" H 5950 4600 50  0001 C CNN
@@
 INT
 $Comp
-L Device:R_US R13
+L Device:R_US R15
 U 1 1 5DF05E21
 P 4950 3250
-F 0 "R13" H 5018 3296 50  0000 L CNN
+F 0 "R15" H 5018 3296 50  0000 L CNN
 F 1 "4.7k" H 5018 3205 50  0000 L CNN
 F 2 "Resistor_SMD:R_0603_1608Metric" V 4990 3240 50  0001 C CNN
@@
 	5450 3750 3950 3750
 $Comp
-L Device:R_US R12
+L Device:R_US R14
 U 1 1 5DF0FA82
 P 3950 3200
-F 0 "R12" H 4018 3246 50  0000 L CNN
+F 0 "R14" H 4018 3246 50  0000 L CNN
 F 1 "4.7k" H 4018 3155 50  0000 L CNN
 F 2 "Resistor_SMD:R_0603_1608Metric" V 3990 3190 50  0001 C CNN
@@
 	3950 3350 3950 3750
 $Comp
-L Device:R_US R11
+L Device:R_US R13
 U 1 1 5DF109EE
 P 3550 3200
-F 0 "R11" H 3618 3246 50  0000 L CNN
+F 0 "R13" H 3618 3246 50  0000 L CNN
 F 1 "4.7k" H 3618 3155 50  0000 L CNN
 F 2 "Resistor_SMD:R_0603_1608Metric" V 3590 3190 50  0001 C CNN
@@
 F 0 "Y2" V 6654 3431 50  0000 L CNN
 F 1 "32.768k" V 6745 3431 50  0000 L CNN
-F 2 "Crystal:Crystal_SMD_0603-2Pin_6.0x3.5mm" H 6700 3300 50  0001 C CNN
+F 2 "" H 6700 3300 50  0001 C CNN
 F 3 "~" H 6700 3300 50  0001 C CNN
 	1    6700 3300
@@
 	7300 3550 7300 3600
 $Comp
-L power:GND #PWR039
+L power:GND #PWR043
 U 1 1 5DEE93BA
 P 7300 3600
-F 0 "#PWR039" H 7300 3350 50  0001 C CNN
+F 0 "#PWR043" H 7300 3350 50  0001 C CNN
 F 1 "GND" H 7305 3427 50  0000 C CNN
 F 2 "" H 7300 3600 50  0001 C CNN
@@
 $EndComp
 $Comp
-L Device:R_US R10
+L Device:R_US R12
 U 1 1 5DEF58D7
 P 3100 2800
-F 0 "R10" H 3168 2846 50  0000 L CNN
+F 0 "R12" H 3168 2846 50  0000 L CNN
 F 1 "4.7k" H 3168 2755 50  0000 L CNN
 F 2 "Resistor_SMD:R_0603_1608Metric" V 3140 2790 50  0001 C CNN
@@
 	7950 4550 8400 4550
 $Comp
-L Connector:Conn_01x02_Male J7
+L Connector:Conn_01x02_Male J6
 U 1 1 5DED60FE
 P 4400 3450
-F 0 "J7" H 4508 3631 50  0000 C CNN
+F 0 "J6" H 4508 3631 50  0000 C CNN
 F 1 "Conn_01x02_Male" H 4508 3540 50  0000 C CNN
 F 2 "Connector_PinHeader_1.00mm:PinHeader_1x02_P1.00mm_Vertical" H 4400 3450 50  0001 C CNN
@@
 	3950 3050 4950 3050
 $Comp
-L power:GND #PWR034
+L power:GND #PWR038
 U 1 1 5DEF0CA0
 P 4600 3550
-F 0 "#PWR034" H 4600 3300 50  0001 C CNN
+F 0 "#PWR038" H 4600 3300 50  0001 C CNN
 F 1 "GND" H 4750 3450 50  0000 C CNN
 F 2 "" H 4600 3550 50  0001 C CNN
@@
 	2950 3050 3550 3050
 $Comp
-L power:+3.3V #PWR040
+L power:+3.3V #PWR044
 U 1 1 5DEFA7ED
 P 8700 2850
-F 0 "#PWR040" H 8700 2700 50  0001 C CNN
+F 0 "#PWR044" H 8700 2700 50  0001 C CNN
 F 1 "+3.3V" H 8715 3023 50  0000 C CNN
 F 2 "" H 8700 2850 50  0001 C CNN
@@
 Connection ~ 5100 4550
 $Comp
-L power:GND #PWR036
+L power:GND #PWR040
 U 1 1 5DF41D8E
 P 5100 4600
-F 0 "#PWR036" H 5100 4350 50  0001 C CNN
+F 0 "#PWR040" H 5100 4350 50  0001 C CNN
 F 1 "GND" H 5105 4427 50  0000 C CNN
 F 2 "" H 5100 4600 50  0001 C CNN
@@
 	5450 4050 5350 4050
 $Comp
-L power:GND #PWR037
+L power:GND #PWR041
 U 1 1 5E5F566F
 P 5350 4050
-F 0 "#PWR037" H 5350 3800 50  0001 C CNN
+F 0 "#PWR041" H 5350 3800 50  0001 C CNN
 F 1 "GND" H 5355 3877 50  0000 C CNN
 F 2 "" H 5350 4050 50  0001 C CNN

Commit message: Updated some footprints and re-annotated schematic.
Parts:
- J7: renamed from J6; footprint Connector_PinHeader_1.00mm:PinHeader_1x02_P1.00mm_Vertical -> Connector_PinHeader_2.54mm:PinHeader_1x02_P2.54mm_Vertical
- renumbered C15 to C17, C16 to C18, C17 to C19, C18 to C20, C19 to C21, C20 to C22, R12 to R13, R13 to R14, R14 to R15, R15 to R16
Changed lines of the file:
@@
 EESchema Schematic File Version 4
-LIBS:Recovery PCB-cache
-EELAYER 26 0
+EELAYER 30 0
 EELAYER END
 $Descr A4 11693 8268
@@
 $EndDescr
 $Comp
-L power:+3.3V #PWR039
+L power:+3.3V #PWR048
 U 1 1 5DF02D6F
 P 4650 2500
-F 0 "#PWR039" H 4650 2350 50  0001 C CNN
+F 0 "#PWR048" H 4650 2350 50  0001 C CNN
 F 1 "+3.3V" H 4665 2673 50  0000 C CNN
 F 2 "" H 4650 2500 50  0001 C CNN
@@
 $EndComp
 $Comp
-L power:+3.3V #PWR037
+L power:+3.3V #PWR046
 U 1 1 5DF02F5F
 P 2950 2500
-F 0 "#PWR037" H 2950 2350 50  0001 C CNN
+F 0 "#PWR046" H 2950 2350 50  0001 C CNN
 F 1 "+3.3V" H 2965 2673 50  0000 C CNN
 F 2 "" H 2950 2500 50  0001 C CNN
@@
 $EndComp
 $Comp
-L power:GND #PWR042
+L power:GND #PWR051
 U 1 1 5DF0362D
 P 5950 4600
-F 0 "#PWR042" H 5950 4350 50  0001 C CNN
+F 0 "#PWR051" H 5950 4350 50  0001 C CNN
 F 1 "GND" H 5955 4427 50  0000 C CNN
 F 2 "" H 5950 4600 50  0001 C CNN
@@
 	5950 2850 5400 2850
 $Comp
-L Device:C C15
+L Device:C C17
 U 1 1 5DF03BA1
 P 5400 2700
-F 0 "C15" H 5515 2746 50  0000 L CNN
+F 0 "C17" H 5515 2746 50  0000 L CNN
 F 1 "0.1u" H 5515 2655 50  0000 L CNN
 F 2 "Capacitor_SMD:C_0603_1608Metric" H 5438 2550 50  0001 C CNN
@@
 INT
 $Comp
-L Device:R_US R15
+L Device:R_US R16
 U 1 1 5DF05E21
 P 4950 3250
-F 0 "R15" H 5018 3296 50  0000 L CNN
+F 0 "R16" H 5018 3296 50  0000 L CNN
 F 1 "4.7k" H 5018 3205 50  0000 L CNN
 F 2 "Resistor_SMD:R_0603_1608Metric" V 4990 3240 50  0001 C CNN
@@
 $EndComp
 $Comp
-L Device:C C16
+L Device:C C18
 U 1 1 5DF0775A
 P 6750 4200
-F 0 "C16" H 6865 4246 50  0000 L CNN
+F 0 "C18" H 6865 4246 50  0000 L CNN
 F 1 "0.1u" H 6865 4155 50  0000 L CNN
 F 2 "Capacitor_SMD:C_0603_1608Metric" H 6788 4050 50  0001 C CNN
@@
 	5450 3750 3950 3750
 $Comp
-L Device:R_US R14
+L Device:R_US R15
 U 1 1 5DF0FA82
 P 3950 3200
-F 0 "R14" H 4018 3246 50  0000 L CNN
+F 0 "R15" H 4018 3246 50  0000 L CNN
 F 1 "4.7k" H 4018 3155 50  0000 L CNN
 F 2 "Resistor_SMD:R_0603_1608Metric" V 3990 3190 50  0001 C CNN
@@
 	3950 3350 3950 3750
 $Comp
-L Device:R_US R13
+L Device:R_US R14
 U 1 1 5DF109EE
 P 3550 3200
-F 0 "R13" H 3618 3246 50  0000 L CNN
+F 0 "R14" H 3618 3246 50  0000 L CNN
 F 1 "4.7k" H 3618 3155 50  0000 L CNN
 F 2 "Resistor_SMD:R_0603_1608Metric" V 3590 3190 50  0001 C CNN
@@
 	6150 4550 7950 4550
 $Comp
-L Device:C C20
+L Device:C C22
 U 1 1 5DF140F0
 P 8400 3600
-F 0 "C20" H 8515 3646 50  0000 L CNN
+F 0 "C22" H 8515 3646 50  0000 L CNN
 F 1 "6.8n" H 8515 3555 50  0000 L CNN
 F 2 "Capacitor_SMD:C_0603_1608Metric" H 8438 3450 50  0001 C CNN
@@
 $EndComp
 $Comp
-L Device:C C19
+L Device:C C21
 U 1 1 5DF1486E
 P 7950 3600
-F 0 "C19" H 8065 3646 50  0000 L CNN
+F 0 "C21" H 8065 3646 50  0000 L CNN
 F 1 "0.12u" H 8065 3555 50  0000 L CNN
 F 2 "Capacitor_SMD:C_0603_1608Metric" H 7988 3450 50  0001 C CNN
@@
 	6700 3450 6700 3550
 $Comp
-L Device:C C17
+L Device:C C19
 U 1 1 5DEDEF8B
 P 6950 3050
-F 0 "C17" V 6698 3050 50  0000 C CNN
+F 0 "C19" V 6698 3050 50  0000 C CNN
 F 1 "22p" V 6789 3050 50  0000 C CNN
 F 2 "Capacitor_SMD:C_0603_1608Metric" H 6988 2900 50  0001 C CNN
@@
 $EndComp
 $Comp
-L Device:C C18
+L Device:C C20
 U 1 1 5DEE0132
 P 6950 3550
-F 0 "C18" V 7100 3550 50  0000 C CNN
+F 0 "C20" V 7100 3550 50  0000 C CNN
 F 1 "22p" V 7200 3550 50  0000 C CNN
 F 2 "Capacitor_SMD:C_0603_1608Metric" H 6988 3400 50  0001 C CNN
@@
 	7300 3550 7300 3600
 $Comp
-L power:GND #PWR043
+L power:GND #PWR052
 U 1 1 5DEE93BA
 P 7300 3600
-F 0 "#PWR043" H 7300 3350 50  0001 C CNN
+F 0 "#PWR052" H 7300 3350 50  0001 C CNN
 F 1 "GND" H 7305 3427 50  0000 C CNN
 F 2 "" H 7300 3600 50  0001 C CNN
@@
 $EndComp
 $Comp
-L Device:R_US R12
+L Device:R_US R13
 U 1 1 5DEF58D7
 P 3100 2800
-F 0 "R12" H 3168 2846 50  0000 L CNN
+F 0 "R13" H 3168 2846 50  0000 L CNN
 F 1 "4.7k" H 3168 2755 50  0000 L CNN
 F 2 "Resistor_SMD:R_0603_1608Metric" V 3140 2790 50  0001 C CNN
@@
 	7950 4550 8400 4550
 $Comp
-L Connector:Conn_01x02_Male J6
+L Connector:Conn_01x02_Male J7
 U 1 1 5DED60FE
 P 4400 3450
-F 0 "J6" H 4508 3631 50  0000 C CNN
+F 0 "J7" H 4508 3631 50  0000 C CNN
 F 1 "Conn_01x02_Male" H 4508 3540 50  0000 C CNN
-F 2 "Connector_PinHeader_1.00mm:PinHeader_1x02_P1.00mm_Vertical" H 4400 3450 50  0001 C CNN
+F 2 "Connector_PinHeader_2.54mm:PinHeader_1x02_P2.54mm_Vertical" H 4400 3450 50  0001 C CNN
 F 3 "~" H 4400 3450 50  0001 C CNN
 	1    4400 3450
@@
 	3950 3050 4950 3050
 $Comp
-L power:GND #PWR038
+L power:GND #PWR047
 U 1 1 5DEF0CA0
 P 4600 3550
-F 0 "#PWR038" H 4600 3300 50  0001 C CNN
+F 0 "#PWR047" H 4600 3300 50  0001 C CNN
 F 1 "GND" H 4750 3450 50  0000 C CNN
 F 2 "" H 4600 3550 50  0001 C CNN
@@
 	2950 3050 3550 3050
 $Comp
-L power:+3.3V #PWR044
+L power:+3.3V #PWR053
 U 1 1 5DEFA7ED
 P 8700 2850
-F 0 "#PWR044" H 8700 2700 50  0001 C CNN
+F 0 "#PWR053" H 8700 2700 50  0001 C CNN
 F 1 "+3.3V" H 8715 3023 50  0000 C CNN
 F 2 "" H 8700 2850 50  0001 C CNN
@@
 Connection ~ 5100 4550
 $Comp
-L power:GND #PWR040
+L power:GND #PWR049
 U 1 1 5DF41D8E
 P 5100 4600
-F 0 "#PWR040" H 5100 4350 50  0001 C CNN
+F 0 "#PWR049" H 5100 4350 50  0001 C CNN
 F 1 "GND" H 5105 4427 50  0000 C CNN
 F 2 "" H 5100 4600 50  0001 C CNN
@@
 	5450 4050 5350 4050
 $Comp
-L power:GND #PWR041
+L power:GND #PWR050
 U 1 1 5E5F566F
 P 5350 4050
-F 0 "#PWR041" H 5350 3800 50  0001 C CNN
+F 0 "#PWR050" H 5350 3800 50  0001 C CNN
 F 1 "GND" H 5355 3877 50  0000 C CNN
 F 2 "" H 5350 4050 50  0001 C CNN

Commit message: Added missing footprints and replaced GPS module.
Parts:
- Y2: footprint (none) -> Crystal:Crystal_SMD_3215-2Pin_3.2x1.5mm
- renumbered U5 to U6
Changed lines of the file:
@@
 	5950 4450 5950 4600
 $Comp
-L Sensor_Motion:BNO055 U5
+L Sensor_Motion:BNO055 U6
 U 1 1 5DF00E39
 P 6050 3550
-F 0 "U5" H 6050 4431 50  0000 C CNN
+F 0 "U6" H 6050 4431 50  0000 C CNN
 F 1 "BNO055" H 6050 4340 50  0000 C CNN
 F 2 "Package_LGA:LGA-28_5.2x3.8mm_P0.5mm" H 6300 2900 50  0001 L CNN
@@
 F 0 "Y2" V 6654 3431 50  0000 L CNN
 F 1 "32.768k" V 6745 3431 50  0000 L CNN
-F 2 "" H 6700 3300 50  0001 C CNN
+F 2 "Crystal:Crystal_SMD_3215-2Pin_3.2x1.5mm" H 6700 3300 50  0001 C CNN
 F 3 "~" H 6700 3300 50  0001 C CNN
 	1    6700 3300

Commit message: Recovery PCB: Redraw schematics
Redrew Recover PCB schematics to be more easily readable and fixed board
outline, adding netclasses to ease trace placement.
Parts:
- C19, C20: symbol Device:C -> Device:C_Small
- J7: value Conn_01x02_Male -> BLD
- Y2: symbol Device:Crystal -> Device:Crystal_Small
Connections:
- net labels added: +3V3, GND1
- net labels removed: +3.3V
- wire segments 62 -> 44

Commit message: Rev 3 of Recovery PCB. Fixed decoupling caps and finalized power/ground.
Connections:
- net labels added: GNDD
- net labels removed: GND1
Changed lines of the file:
@@
-	1    0    0    -1
-$EndComp
-$Comp
-L Sensor_Motion:BNO055 U6
-U 1 1 5DF00E39
-P 6050 3550
-F 0 "U6" H 5600 2900 50  0000 C CNN
-F 1 "BNO055" H 5700 2800 50  0000 C CNN
-F 2 "Package_LGA:LGA-28_5.2x3.8mm_P0.5mm" H 6300 2900 50  0001 L CNN
-F 3 "https://www.bosch-sensortec.com/media/boschsensortec/downloads/datasheets/bst-bno055-ds000.pdf" H 6050 3750 50  0001 C CNN
-	1    6050 3550
 	1    0    0    -1
 $EndComp
@@
 Wire Wire Line
 	6150 2300 6150 2850
-$Comp
-L power:GND1 #PWR0106
-U 1 1 6009086D
-P 6300 2600
-F 0 "#PWR0106" H 6300 2350 50  0001 C CNN
-F 1 "GND1" H 6305 2427 50  0000 C CNN
-F 2 "" H 6300 2600 50  0001 C CNN
-F 3 "" H 6300 2600 50  0001 C CNN
-	1    6300 2600
-	1    0    0    -1
-$EndComp
-$Comp
-L power:GND1 #PWR0107
-U 1 1 600911FB
-P 6750 2600
-F 0 "#PWR0107" H 6750 2350 50  0001 C CNN
-F 1 "GND1" H 6755 2427 50  0000 C CNN
-F 2 "" H 6750 2600 50  0001 C CNN
-F 3 "" H 6750 2600 50  0001 C CNN
-	1    6750 2600
-	1    0    0    -1
-$EndComp
-$Comp
-L power:GND1 #PWR0108
-U 1 1 60093023
-P 6150 4350
-F 0 "#PWR0108" H 6150 4100 50  0001 C CNN
-F 1 "GND1" H 6155 4177 50  0000 C CNN
-F 2 "" H 6150 4350 50  0001 C CNN
-F 3 "" H 6150 4350 50  0001 C CNN
-	1    6150 4350
-	1    0    0    -1
-$EndComp
 Wire Wire Line
 	5950 4250 6150 4250
 Wire Wire Line
 	5950 4250 5950 4350
-Connection ~ 5950 4250
 Wire Wire Line
 	6150 4250 6150 4350
-Connection ~ 6150 4250
-$Comp
-L power:GND1 #PWR0109
-U 1 1 6009C1C9
-P 5200 4350
-F 0 "#PWR0109" H 5200 4100 50  0001 C CNN
-F 1 "GND1" H 5205 4177 50  0000 C CNN
-F 2 "" H 5200 4350 50  0001 C CNN
-F 3 "" H 5200 4350 50  0001 C CNN
-	1    5200 4350
-	1    0    0    -1
-$EndComp
 Wire Wire Line
 	5400 2600 5400 2650
@@
 Wire Wire Line
 	6800 3550 6850 3550
-$Comp
-L power:GND1 #PWR0119
-U 1 1 6010A6D0
+Wire Wire Line
+	5200 3950 5200 4350
+Wire Wire Line
+	5450 4350 5450 4050
+Wire Wire Line
+	4150 3750 4600 3750
+Connection ~ 4600 3750
+Wire Wire Line
+	4300 3850 4150 3850
+Connection ~ 4300 3850
+Connection ~ 6150 4250
+Connection ~ 5950 4250
+$Comp
+L power:GNDD #PWR0106
+U 1 1 60051BF6
+P 6300 2600
+F 0 "#PWR0106" H 6300 2350 50  0001 C CNN
+F 1 "GNDD" H 6304 2445 50  0000 C CNN
+F 2 "" H 6300 2600 50  0001 C CNN
+F 3 "" H 6300 2600 50  0001 C CNN
+	1    6300 2600
+	1    0    0    -1
+$EndComp
+$Comp
+L Sensor_Motion:BNO055 U6
+U 1 1 5DF00E39
+P 6050 3550
+F 0 "U6" H 5600 2900 50  0000 C CNN
+F 1 "BNO055" H 5700 2800 50  0000 C CNN
+F 2 "Package_LGA:LGA-28_5.2x3.8mm_P0.5mm" H 6300 2900 50  0001 L CNN
+F 3 "https://www.bosch-sensortec.com/media/boschsensortec/downloads/datasheets/bst-bno055-ds000.pdf" H 6050 3750 50  0001 C CNN
+	1    6050 3550
+	1    0    0    -1
+$EndComp
+$Comp
+L power:GNDD #PWR0107
+U 1 1 6005A0DB
+P 6750 2600
+F 0 "#PWR0107" H 6750 2350 50  0001 C CNN
+F 1 "GNDD" H 6754 2445 50  0000 C CNN
+F 2 "" H 6750 2600 50  0001 C CNN
+F 3 "" H 6750 2600 50  0001 C CNN
+	1    6750 2600
+	1    0    0    -1
+$EndComp
+$Comp
+L power:GNDD #PWR0108
+U 1 1 6005B1A1
+P 5200 4350
+F 0 "#PWR0108" H 5200 4100 50  0001 C CNN
+F 1 "GNDD" H 5204 4195 50  0000 C CNN
+F 2 "" H 5200 4350 50  0001 C CNN
+F 3 "" H 5200 4350 50  0001 C CNN
+	1    5200 4350
+	1    0    0    -1
+$EndComp
+$Comp
+L power:GNDD #PWR0109
+U 1 1 6005BAE2
 P 5450 4350
-F 0 "#PWR0119" H 5450 4100 50  0001 C CNN
-F 1 "GND1" H 5455 4177 50  0000 C CNN
+F 0 "#PWR0109" H 5450 4100 50  0001 C CNN
+F 1 "GNDD" H 5454 4195 50  0000 C CNN
 F 2 "" H 5450 4350 50  0001 C CNN
 F 3 "" H 5450 4350 50  0001 C CNN
@@
 	1    0    0    -1
 $EndComp
-Wire Wire Line
-	5200 3950 5200 4350
-Wire Wire Line
-	5450 4350 5450 4050
-Wire Wire Line
-	4150 3750 4600 3750
-Connection ~ 4600 3750
-Wire Wire Line
-	4300 3850 4150 3850
-Connection ~ 4300 3850
+$Comp
+L power:GNDD #PWR0119
+U 1 1 6005C5A6
+P 6150 4350
+F 0 "#PWR0119" H 6150 4100 50  0001 C CNN
+F 1 "GNDD" H 6154 4195 50  0000 C CNN
+F 2 "" H 6150 4350 50  0001 C CNN
+F 3 "" H 6150 4350 50  0001 C CNN
+	1    6150 4350
+	1    0    0    -1
+$EndComp
 $EndSCHEMATC
