File: Recovery PCB/Accelerometer.sch (KiCad schematic (older format))
At the start: 5 parts, among them U2 ADXL377

Commit message: Update relays and re-annotate entire schematic. Review needed before layout.
Parts:
- renumbered C2 to C11, C3 to C12, C4 to C13, C5 to C14, U2 to U3
Changed lines of the file:
@@
 $EndDescr
 $Comp
-L ADXL377:ADXL377 U2
+L ADXL377:ADXL377 U3
 U 1 1 5DEED3C1
 P 5900 3300
-F 0 "U2" H 5900 3767 50  0000 C CNN
+F 0 "U3" H 5900 3767 50  0000 C CNN
 F 1 "ADXL377" H 5900 3676 50  0000 C CNN
 F 2 "LFCSP-16-3X3" H 5900 3300 50  0001 L BNN
@@
 	6400 3100 6750 3100
 $Comp
-L Device:C C3
+L Device:C C12
 U 1 1 5DEEED1E
 P 6750 3250
-F 0 "C3" H 6865 3296 50  0000 L CNN
+F 0 "C12" H 6865 3296 50  0000 L CNN
 F 1 "0.01u" H 6865 3205 50  0000 L CNN
 F 2 "Capacitor_SMD:C_0603_1608Metric" H 6788 3100 50  0001 C CNN
@@
 Xout
 $Comp
-L power:GND #PWR07
+L power:GND #PWR020
 U 1 1 5DEEF1C3
 P 6750 3400
-F 0 "#PWR07" H 6750 3150 50  0001 C CNN
+F 0 "#PWR020" H 6750 3150 50  0001 C CNN
 F 1 "GND" H 6755 3227 50  0000 C CNN
 F 2 "" H 6750 3400 50  0001 C CNN
@@
 $EndComp
 $Comp
-L Device:C C4
+L Device:C C13
 U 1 1 5DEEF59F
 P 6750 3900
-F 0 "C4" H 6865 3946 50  0000 L CNN
+F 0 "C13" H 6865 3946 50  0000 L CNN
 F 1 "0.01u" H 6865 3855 50  0000 L CNN
 F 2 "Capacitor_SMD:C_0603_1608Metric" H 6788 3750 50  0001 C CNN
@@
 	6400 3300 6500 3300
 $Comp
-L power:GND #PWR08
+L power:GND #PWR021
 U 1 1 5DEF02B6
 P 6750 4050
-F 0 "#PWR08" H 6750 3800 50  0001 C CNN
+F 0 "#PWR021" H 6750 3800 50  0001 C CNN
 F 1 "GND" H 6755 3877 50  0000 C CNN
 F 2 "" H 6750 4050 50  0001 C CNN
@@
 $EndComp
 $Comp
-L power:GND #PWR06
+L power:GND #PWR019
 U 1 1 5DEF056E
 P 6400 3500
-F 0 "#PWR06" H 6400 3250 50  0001 C CNN
+F 0 "#PWR019" H 6400 3250 50  0001 C CNN
 F 1 "GND" H 6405 3327 50  0000 C CNN
 F 2 "" H 6400 3500 50  0001 C CNN
@@
 	6500 3300 6500 4350
 $Comp
-L Device:C C5
+L Device:C C14
 U 1 1 5DEF0B71
 P 6750 4500
-F 0 "C5" H 6865 4546 50  0000 L CNN
+F 0 "C14" H 6865 4546 50  0000 L CNN
 F 1 "0.01u" H 6865 4455 50  0000 L CNN
 F 2 "Capacitor_SMD:C_0603_1608Metric" H 6788 4350 50  0001 C CNN
@@
 $EndComp
 $Comp
-L power:GND #PWR09
+L power:GND #PWR022
 U 1 1 5DEF0EB0
 P 6750 4650
-F 0 "#PWR09" H 6750 4400 50  0001 C CNN
+F 0 "#PWR022" H 6750 4400 50  0001 C CNN
 F 1 "GND" H 6755 4477 50  0000 C CNN
 F 2 "" H 6750 4650 50  0001 C CNN
@@
 	5400 3200 5350 3200
 $Comp
-L Device:C C2
+L Device:C C11
 U 1 1 5DEF330A
 P 5050 3300
-F 0 "C2" H 5165 3346 50  0000 L CNN
+F 0 "C11" H 5165 3346 50  0000 L CNN
 F 1 "0.1u" H 5165 3255 50  0000 L CNN
 F 2 "Capacitor_SMD:C_0603_1608Metric" H 5088 3150 50  0001 C CNN
@@
 	5350 3100 5400 3100
 $Comp
-L power:+3.3V #PWR02
+L power:+3.3V #PWR017
 U 1 1 5DEF43DF
 P 5350 2950
-F 0 "#PWR02" H 5350 2800 50  0001 C CNN
+F 0 "#PWR017" H 5350 2800 50  0001 C CNN
 F 1 "+3.3V" H 5365 3123 50  0000 C CNN
 F 2 "" H 5350 2950 50  0001 C CNN
@@
 $EndComp
 $Comp
-L power:GND #PWR03
+L power:GND #PWR018
 U 1 1 5DEF4B6B
 P 5350 3650
-F 0 "#PWR03" H 5350 3400 50  0001 C CNN
+F 0 "#PWR018" H 5350 3400 50  0001 C CNN
 F 1 "GND" H 5355 3477 50  0000 C CNN
 F 2 "" H 5350 3650 50  0001 C CNN

Commit message: Updated some footprints and re-annotated schematic.
Parts:
- renumbered C11 to C13, C12 to C14, C13 to C15, C14 to C16
Changed lines of the file:
@@
 EESchema Schematic File Version 4
-LIBS:Recovery PCB-cache
-EELAYER 26 0
+EELAYER 30 0
 EELAYER END
 $Descr A4 11693 8268
@@
 	6400 3100 6750 3100
 $Comp
-L Device:C C12
+L Device:C C14
 U 1 1 5DEEED1E
 P 6750 3250
-F 0 "C12" H 6865 3296 50  0000 L CNN
+F 0 "C14" H 6865 3296 50  0000 L CNN
 F 1 "0.01u" H 6865 3205 50  0000 L CNN
 F 2 "Capacitor_SMD:C_0603_1608Metric" H 6788 3100 50  0001 C CNN
@@
 Xout
 $Comp
-L power:GND #PWR020
+L power:GND #PWR029
 U 1 1 5DEEF1C3
 P 6750 3400
-F 0 "#PWR020" H 6750 3150 50  0001 C CNN
+F 0 "#PWR029" H 6750 3150 50  0001 C CNN
 F 1 "GND" H 6755 3227 50  0000 C CNN
 F 2 "" H 6750 3400 50  0001 C CNN
@@
 $EndComp
 $Comp
-L Device:C C13
+L Device:C C15
 U 1 1 5DEEF59F
 P 6750 3900
-F 0 "C13" H 6865 3946 50  0000 L CNN
+F 0 "C15" H 6865 3946 50  0000 L CNN
 F 1 "0.01u" H 6865 3855 50  0000 L CNN
 F 2 "Capacitor_SMD:C_0603_1608Metric" H 6788 3750 50  0001 C CNN
@@
 	6400 3300 6500 3300
 $Comp
-L power:GND #PWR021
+L power:GND #PWR030
 U 1 1 5DEF02B6
 P 6750 4050
-F 0 "#PWR021" H 6750 3800 50  0001 C CNN
+F 0 "#PWR030" H 6750 3800 50  0001 C CNN
 F 1 "GND" H 6755 3877 50  0000 C CNN
 F 2 "" H 6750 4050 50  0001 C CNN
@@
 $EndComp
 $Comp
-L power:GND #PWR019
+L power:GND #PWR028
 U 1 1 5DEF056E
 P 6400 3500
-F 0 "#PWR019" H 6400 3250 50  0001 C CNN
+F 0 "#PWR028" H 6400 3250 50  0001 C CNN
 F 1 "GND" H 6405 3327 50  0000 C CNN
 F 2 "" H 6400 3500 50  0001 C CNN
@@
 	6500 3300 6500 4350
 $Comp
-L Device:C C14
+L Device:C C16
 U 1 1 5DEF0B71
 P 6750 4500
-F 0 "C14" H 6865 4546 50  0000 L CNN
+F 0 "C16" H 6865 4546 50  0000 L CNN
 F 1 "0.01u" H 6865 4455 50  0000 L CNN
 F 2 "Capacitor_SMD:C_0603_1608Metric" H 6788 4350 50  0001 C CNN
@@
 $EndComp
 $Comp
-L power:GND #PWR022
+L power:GND #PWR031
 U 1 1 5DEF0EB0
 P 6750 4650
-F 0 "#PWR022" H 6750 4400 50  0001 C CNN
+F 0 "#PWR031" H 6750 4400 50  0001 C CNN
 F 1 "GND" H 6755 4477 50  0000 C CNN
 F 2 "" H 6750 4650 50  0001 C CNN
@@
 	5400 3200 5350 3200
 $Comp
-L Device:C C11
+L Device:C C13
 U 1 1 5DEF330A
 P 5050 3300
-F 0 "C11" H 5165 3346 50  0000 L CNN
+F 0 "C13" H 5165 3346 50  0000 L CNN
 F 1 "0.1u" H 5165 3255 50  0000 L CNN
 F 2 "Capacitor_SMD:C_0603_1608Metric" H 5088 3150 50  0001 C CNN
@@
 	5350 3100 5400 3100
 $Comp
-L power:+3.3V #PWR017
+L power:+3.3V #PWR026
 U 1 1 5DEF43DF
 P 5350 2950
-F 0 "#PWR017" H 5350 2800 50  0001 C CNN
+F 0 "#PWR026" H 5350 2800 50  0001 C CNN
 F 1 "+3.3V" H 5365 3123 50  0000 C CNN
 F 2 "" H 5350 2950 50  0001 C CNN
@@
 $EndComp
 $Comp
-L power:GND #PWR018
+L power:GND #PWR027
 U 1 1 5DEF4B6B
 P 5350 3650
-F 0 "#PWR018" H 5350 3400 50  0001 C CNN
+F 0 "#PWR027" H 5350 3400 50  0001 C CNN
 F 1 "GND" H 5355 3477 50  0000 C CNN
 F 2 "" H 5350 3650 50  0001 C CNN

Commit message: Added missing footprints and replaced GPS module.
Parts:
- renumbered U3 to U4
Changed lines of the file:
@@
 $EndDescr
 $Comp
-L ADXL377:ADXL377 U3
+L ADXL377:ADXL377 U4
 U 1 1 5DEED3C1
 P 5900 3300
-F 0 "U3" H 5900 3767 50  0000 C CNN
+F 0 "U4" H 5900 3767 50  0000 C CNN
 F 1 "ADXL377" H 5900 3676 50  0000 C CNN
 F 2 "LFCSP-16-3X3" H 5900 3300 50  0001 L BNN

Commit message: Recovery PCB: Redraw schematics
Redrew Recover PCB schematics to be more easily readable and fixed board
outline, adding netclasses to ease trace placement.
Connections:
- wire segments 22 -> 19
Changed lines of the file:
@@
 L Device:C C13
 U 1 1 5DEF330A
-P 5050 3300
-F 0 "C13" H 5165 3346 50  0000 L CNN
-F 1 "0.1u" H 5165 3255 50  0000 L CNN
-F 2 "Capacitor_SMD:C_0603_1608Metric" H 5088 3150 50  0001 C CNN
-F 3 "~" H 5050 3300 50  0001 C CNN
-	1    5050 3300
+P 5100 2800
+F 0 "C13" H 4800 2850 50  0000 L CNN
+F 1 "0.1u" H 4800 2750 50  0000 L CNN
+F 2 "Capacitor_SMD:C_0603_1608Metric" H 5138 2650 50  0001 C CNN
+F 3 "~" H 5100 2800 50  0001 C CNN
+	1    5100 2800
 	1    0    0    -1
 $EndComp
@@
 L power:+3.3V #PWR026
 U 1 1 5DEF43DF
-P 5350 2950
-F 0 "#PWR026" H 5350 2800 50  0001 C CNN
-F 1 "+3.3V" H 5365 3123 50  0000 C CNN
-F 2 "" H 5350 2950 50  0001 C CNN
-F 3 "" H 5350 2950 50  0001 C CNN
-	1    5350 2950
+P 5350 2650
+F 0 "#PWR026" H 5350 2500 50  0001 C CNN
+F 1 "+3.3V" H 5365 2823 50  0000 C CNN
+F 2 "" H 5350 2650 50  0001 C CNN
+F 3 "" H 5350 2650 50  0001 C CNN
+	1    5350 2650
 	1    0    0    -1
 $EndComp
@@
 	5350 3500 5350 3650
 Connection ~ 5350 3500
+$Comp
+L power:GND #PWR0124
+U 1 1 6039DB62
+P 5100 2950
+F 0 "#PWR0124" H 5100 2700 50  0001 C CNN
+F 1 "GND" H 5105 2777 50  0000 C CNN
+F 2 "" H 5100 2950 50  0001 C CNN
+F 3 "" H 5100 2950 50  0001 C CNN
+	1    5100 2950
+	1    0    0    -1
+$EndComp
 Wire Wire Line
-	5350 3100 5350 2950
+	5100 2650 5350 2650
 Wire Wire Line
-	5050 3150 5050 3100
-Wire Wire Line
-	5050 3100 5350 3100
-Wire Wire Line
-	5050 3450 5050 3500
-Wire Wire Line
-	5050 3500 5350 3500
+	5350 2650 5350 3100
+Connection ~ 5350 2650
 $EndSCHEMATC

Commit message: Recovery PCB: Reannotate
Reannotated schematic to fix reference numbering and keep reference
designators consistent.
Parts:
- renumbered C13 to C14, C14 to C15, C15 to C16, C16 to C17
Changed lines of the file:
@@
 	6400 3100 6750 3100
 $Comp
-L Device:C C14
+L Device:C C15
 U 1 1 5DEEED1E
 P 6750 3250
-F 0 "C14" H 6865 3296 50  0000 L CNN
+F 0 "C15" H 6865 3296 50  0000 L CNN
 F 1 "0.01u" H 6865 3205 50  0000 L CNN
 F 2 "Capacitor_SMD:C_0603_1608Metric" H 6788 3100 50  0001 C CNN
@@
 Xout
 $Comp
-L power:GND #PWR029
+L power:GND #PWR037
 U 1 1 5DEEF1C3
 P 6750 3400
-F 0 "#PWR029" H 6750 3150 50  0001 C CNN
+F 0 "#PWR037" H 6750 3150 50  0001 C CNN
 F 1 "GND" H 6755 3227 50  0000 C CNN
 F 2 "" H 6750 3400 50  0001 C CNN
@@
 $EndComp
 $Comp
-L Device:C C15
+L Device:C C16
 U 1 1 5DEEF59F
 P 6750 3900
-F 0 "C15" H 6865 3946 50  0000 L CNN
+F 0 "C16" H 6865 3946 50  0000 L CNN
 F 1 "0.01u" H 6865 3855 50  0000 L CNN
 F 2 "Capacitor_SMD:C_0603_1608Metric" H 6788 3750 50  0001 C CNN
@@
 	6400 3300 6500 3300
 $Comp
-L power:GND #PWR030
+L power:GND #PWR040
 U 1 1 5DEF02B6
 P 6750 4050
-F 0 "#PWR030" H 6750 3800 50  0001 C CNN
+F 0 "#PWR040" H 6750 3800 50  0001 C CNN
 F 1 "GND" H 6755 3877 50  0000 C CNN
 F 2 "" H 6750 4050 50  0001 C CNN
@@
 $EndComp
 $Comp
-L power:GND #PWR028
+L power:GND #PWR038
 U 1 1 5DEF056E
 P 6400 3500
-F 0 "#PWR028" H 6400 3250 50  0001 C CNN
+F 0 "#PWR038" H 6400 3250 50  0001 C CNN
 F 1 "GND" H 6405 3327 50  0000 C CNN
 F 2 "" H 6400 3500 50  0001 C CNN
@@
 	6500 3300 6500 4350
 $Comp
-L Device:C C16
+L Device:C C17
 U 1 1 5DEF0B71
 P 6750 4500
-F 0 "C16" H 6865 4546 50  0000 L CNN
+F 0 "C17" H 6865 4546 50  0000 L CNN
 F 1 "0.01u" H 6865 4455 50  0000 L CNN
 F 2 "Capacitor_SMD:C_0603_1608Metric" H 6788 4350 50  0001 C CNN
@@
 $EndComp
 $Comp
-L power:GND #PWR031
+L power:GND #PWR041
 U 1 1 5DEF0EB0
 P 6750 4650
-F 0 "#PWR031" H 6750 4400 50  0001 C CNN
+F 0 "#PWR041" H 6750 4400 50  0001 C CNN
 F 1 "GND" H 6755 4477 50  0000 C CNN
 F 2 "" H 6750 4650 50  0001 C CNN
@@
 	5400 3200 5350 3200
 $Comp
-L Device:C C13
+L Device:C C14
 U 1 1 5DEF330A
 P 5100 2800
-F 0 "C13" H 4800 2850 50  0000 L CNN
+F 0 "C14" H 4800 2850 50  0000 L CNN
 F 1 "0.1u" H 4800 2750 50  0000 L CNN
 F 2 "Capacitor_SMD:C_0603_1608Metric" H 5138 2650 50  0001 C CNN
@@
 	5350 3100 5400 3100
 $Comp
-L power:+3.3V #PWR026
+L power:+3.3V #PWR035
 U 1 1 5DEF43DF
 P 5350 2650
-F 0 "#PWR026" H 5350 2500 50  0001 C CNN
+F 0 "#PWR035" H 5350 2500 50  0001 C CNN
 F 1 "+3.3V" H 5365 2823 50  0000 C CNN
 F 2 "" H 5350 2650 50  0001 C CNN
@@
 $EndComp
 $Comp
-L power:GND #PWR027
+L power:GND #PWR039
 U 1 1 5DEF4B6B
 P 5350 3650
-F 0 "#PWR027" H 5350 3400 50  0001 C CNN
+F 0 "#PWR039" H 5350 3400 50  0001 C CNN
 F 1 "GND" H 5355 3477 50  0000 C CNN
 F 2 "" H 5350 3650 50  0001 C CNN
@@
 Connection ~ 5350 3500
 $Comp
-L power:GND #PWR0124
+L power:GND #PWR036
 U 1 1 6039DB62
 P 5100 2950
-F 0 "#PWR0124" H 5100 2700 50  0001 C CNN
+F 0 "#PWR036" H 5100 2700 50  0001 C CNN
 F 1 "GND" H 5105 2777 50  0000 C CNN
 F 2 "" H 5100 2950 50  0001 C CNN

Commit message: Recovery PCB: Tweak Motion Axes
Reconciled IMU and accelerometer motion axes and added models for edge
connectors.
Connections:
- wire segments 19 -> 14
Changed lines of the file:
@@
 U 1 1 5DEED3C1
 P 5900 3300
-F 0 "U4" H 5900 3767 50  0000 C CNN
-F 1 "ADXL377" H 5900 3676 50  0000 C CNN
+F 0 "U4" H 6000 3700 50  0000 C CNN
+F 1 "ADXL377" H 6100 3600 50  0000 C CNN
 F 2 "LFCSP-16-3X3" H 5900 3300 50  0001 L BNN
 F 3 "Unavailable" H 5900 3300 50  0001 L BNN
@@
 $EndComp
 Wire Wire Line
-	6400 3100 6750 3100
+	6250 3150 6600 3150
 $Comp
 L Device:C C15
 U 1 1 5DEEED1E
-P 6750 3250
-F 0 "C15" H 6865 3296 50  0000 L CNN
-F 1 "0.01u" H 6865 3205 50  0000 L CNN
-F 2 "Capacitor_SMD:C_0603_1608Metric" H 6788 3100 50  0001 C CNN
-F 3 "~" H 6750 3250 50  0001 C CNN
-	1    6750 3250
+P 6600 3300
+F 0 "C15" H 6715 3346 50  0000 L CNN
+F 1 "0.01u" H 6715 3255 50  0000 L CNN
+F 2 "Capacitor_SMD:C_0603_1608Metric" H 6638 3150 50  0001 C CNN
+F 3 "~" H 6600 3300 50  0001 C CNN
+	1    6600 3300
 	1    0    0    -1
 $EndComp
-Text HLabel 7000 3100 2    50   Output ~ 0
+Text HLabel 6850 3150 2    50   Output ~ 0
 Xout
 $Comp
 L power:GND #PWR037
 U 1 1 5DEEF1C3
-P 6750 3400
-F 0 "#PWR037" H 6750 3150 50  0001 C CNN
-F 1 "GND" H 6755 3227 50  0000 C CNN
-F 2 "" H 6750 3400 50  0001 C CNN
-F 3 "" H 6750 3400 50  0001 C CNN
-	1    6750 3400
+P 6600 3450
+F 0 "#PWR037" H 6600 3200 50  0001 C CNN
+F 1 "GND" H 6605 3277 50  0000 C CNN
+F 2 "" H 6600 3450 50  0001 C CNN
+F 3 "" H 6600 3450 50  0001 C CNN
+	1    6600 3450
 	1    0    0    -1
 $EndComp
@@
 L Device:C C16
 U 1 1 5DEEF59F
-P 6750 3900
-F 0 "C16" H 6865 3946 50  0000 L CNN
-F 1 "0.01u" H 6865 3855 50  0000 L CNN
-F 2 "Capacitor_SMD:C_0603_1608Metric" H 6788 3750 50  0001 C CNN
-F 3 "~" H 6750 3900 50  0001 C CNN
-	1    6750 3900
+P 6600 3950
+F 0 "C16" H 6715 3996 50  0000 L CNN
+F 1 "0.01u" H 6715 3905 50  0000 L CNN
+F 2 "Capacitor_SMD:C_0603_1608Metric" H 6638 3800 50  0001 C CNN
+F 3 "~" H 6600 3950 50  0001 C CNN
+	1    6600 3950
 	1    0    0    -1
 $EndComp
-Text HLabel 7000 3750 2    50   Output ~ 0
+Text HLabel 6850 3800 2    50   Output ~ 0
 Yout
 Wire Wire Line
-	6400 3300 6500 3300
+	6250 3350 6350 3350
 $Comp
 L power:GND #PWR040
 U 1 1 5DEF02B6
-P 6750 4050
-F 0 "#PWR040" H 6750 3800 50  0001 C CNN
-F 1 "GND" H 6755 3877 50  0000 C CNN
-F 2 "" H 6750 4050 50  0001 C CNN
-F 3 "" H 6750 4050 50  0001 C CNN
-	1    6750 4050
+P 6600 4100
+F 0 "#PWR040" H 6600 3850 50  0001 C CNN
+F 1 "GND" H 6605 3927 50  0000 C CNN
+F 2 "" H 6600 4100 50  0001 C CNN
+F 3 "" H 6600 4100 50  0001 C CNN
+	1    6600 4100
 	1    0    0    -1
 $EndComp
@@
 L power:GND #PWR038
 U 1 1 5DEF056E
-P 6400 3500
-F 0 "#PWR038" H 6400 3250 50  0001 C CNN
-F 1 "GND" H 6405 3327 50  0000 C CNN
-F 2 "" H 6400 3500 50  0001 C CNN
-F 3 "" H 6400 3500 50  0001 C CNN
-	1    6400 3500
+P 5550 3600
+F 0 "#PWR038" H 5550 3350 50  0001 C CNN
+F 1 "GND" H 5555 3427 50  0000 C CNN
+F 2 "" H 5550 3600 50  0001 C CNN
+F 3 "" H 5550 3600 50  0001 C CNN
+	1    5550 3600
 	1    0    0    -1
 $EndComp
 Wire Wire Line
-	6600 3200 6600 3750
+	6450 3250 6450 3800
 Wire Wire Line
-	6400 3200 6600 3200
+	6250 3250 6450 3250
 Wire Wire Line
-	6600 3750 6750 3750
+	6450 3800 6600 3800
 Wire Wire Line
-	6500 4350 6750 4350
+	6350 4400 6600 4400
 Wire Wire Line
-	6500 3300 6500 4350
+	6350 3350 6350 4400
 $Comp
 L Device:C C17
 U 1 1 5DEF0B71
-P 6750 4500
-F 0 "C17" H 6865 4546 50  0000 L CNN
-F 1 "0.01u" H 6865 4455 50  0000 L CNN
-F 2 "Capacitor_SMD:C_0603_1608Metric" H 6788 4350 50  0001 C CNN
-F 3 "~" H 6750 4500 50  0001 C CNN
-	1    6750 4500
+P 6600 4550
+F 0 "C17" H 6715 4596 50  0000 L CNN
+F 1 "0.01u" H 6715 4505 50  0000 L CNN
+F 2 "Capacitor_SMD:C_0603_1608Metric" H 6638 4400 50  0001 C CNN
+F 3 "~" H 6600 4550 50  0001 C CNN
+	1    6600 4550
 	1    0    0    -1
 $EndComp
@@
 L power:GND #PWR041
 U 1 1 5DEF0EB0
-P 6750 4650
-F 0 "#PWR041" H 6750 4400 50  0001 C CNN
-F 1 "GND" H 6755 4477 50  0000 C CNN
-F 2 "" H 6750 4650 50  0001 C CNN
-F 3 "" H 6750 4650 50  0001 C CNN
-	1    6750 4650
+P 6600 4700
+F 0 "#PWR041" H 6600 4450 50  0001 C CNN
+F 1 "GND" H 6605 4527 50  0000 C CNN
+F 2 "" H 6600 4700 50  0001 C CNN
+F 3 "" H 6600 4700 50  0001 C CNN
+	1    6600 4700
 	1    0    0    -1
 $EndComp
 Wire Wire Line
-	6750 4350 7000 4350
-Connection ~ 6750 4350
-Text HLabel 7000 4350 2    50   Output ~ 0
+	6600 4400 6850 4400
+Connection ~ 6600 4400
+Text HLabel 6850 4400 2    50   Output ~ 0
 Zout
 Wire Wire Line
-	6750 3100 7000 3100
-Connection ~ 6750 3100
+	6600 3150 6850 3150
+Connection ~ 6600 3150
 Wire Wire Line
-	6750 3750 7000 3750
-Connection ~ 6750 3750
-Wire Wire Line
-	5400 3200 5350 3200
+	6600 3800 6850 3800
+Connection ~ 6600 3800
 $Comp
 L Device:C C14
 U 1 1 5DEF330A
-P 5100 2800
-F 0 "C14" H 4800 2850 50  0000 L CNN
-F 1 "0.1u" H 4800 2750 50  0000 L CNN
-F 2 "Capacitor_SMD:C_0603_1608Metric" H 5138 2650 50  0001 C CNN
-F 3 "~" H 5100 2800 50  0001 C CNN
-	1    5100 2800
+P 5650 2600
+F 0 "C14" H 5350 2650 50  0000 L CNN
+F 1 "0.1u" H 5350 2550 50  0000 L CNN
+F 2 "Capacitor_SMD:C_0603_1608Metric" H 5688 2450 50  0001 C CNN
+F 3 "~" H 5650 2600 50  0001 C CNN
+	1    5650 2600
 	1    0    0    -1
 $EndComp
-Wire Wire Line
-	5350 3200 5350 3100
-Connection ~ 5350 3100
-Wire Wire Line
-	5350 3100 5400 3100
 $Comp
 L power:+3.3V #PWR035
 U 1 1 5DEF43DF
-P 5350 2650
-F 0 "#PWR035" H 5350 2500 50  0001 C CNN
-F 1 "+3.3V" H 5365 2823 50  0000 C CNN
-F 2 "" H 5350 2650 50  0001 C CNN
-F 3 "" H 5350 2650 50  0001 C CNN
-	1    5350 2650
+P 5900 2450
+F 0 "#PWR035" H 5900 2300 50  0001 C CNN
+F 1 "+3.3V" H 5915 2623 50  0000 C CNN
+F 2 "" H 5900 2450 50  0001 C CNN
+F 3 "" H 5900 2450 50  0001 C CNN
+	1    5900 2450
 	1    0    0    -1
 $EndComp
@@
 L power:GND #PWR039
 U 1 1 5DEF4B6B
-P 5350 3650
-F 0 "#PWR039" H 5350 3400 50  0001 C CNN
-F 1 "GND" H 5355 3477 50  0000 C CNN
-F 2 "" H 5350 3650 50  0001 C CNN
-F 3 "" H 5350 3650 50  0001 C CNN
-	1    5350 3650
+P 5900 3600
+F 0 "#PWR039" H 5900 3350 50  0001 C CNN
+F 1 "GND" H 5905 3427 50  0000 C CNN
+F 2 "" H 5900 3600 50  0001 C CNN
+F 3 "" H 5900 3600 50  0001 C CNN
+	1    5900 3600
+	1    0    0    -1
+$EndComp
+$Comp
+L power:GND #PWR036
+U 1 1 6039DB62
+P 5650 2750
+F 0 "#PWR036" H 5650 2500 50  0001 C CNN
+F 1 "GND" H 5655 2577 50  0000 C CNN
+F 2 "" H 5650 2750 50  0001 C CNN
+F 3 "" H 5650 2750 50  0001 C CNN
+	1    5650 2750
 	1    0    0    -1
 $EndComp
 Wire Wire Line
-	5400 3400 5350 3400
+	5650 2450 5900 2450
+Connection ~ 5900 2450
 Wire Wire Line
-	5350 3400 5350 3500
+	5900 2450 5900 2950
 Wire Wire Line
-	5350 3500 5400 3500
+	5550 3600 5550 3150
 Wire Wire Line
-	5350 3500 5350 3650
-Connection ~ 5350 3500
-$Comp
-L power:GND #PWR036
-U 1 1 6039DB62
-P 5100 2950
-F 0 "#PWR036" H 5100 2700 50  0001 C CNN
-F 1 "GND" H 5105 2777 50  0000 C CNN
-F 2 "" H 5100 2950 50  0001 C CNN
-F 3 "" H 5100 2950 50  0001 C CNN
-	1    5100 2950
-	1    0    0    -1
-$EndComp
-Wire Wire Line
-	5100 2650 5350 2650
-Wire Wire Line
-	5350 2650 5350 3100
-Connection ~ 5350 2650
+	5900 3600 5900 3550
 $EndSCHEMATC
