File: Recovery PCB/PressureSensor.sch (KiCad schematic (older format))
At the start: 4 parts, among them U1 MS5607-02BA

Commit message: Update relays and re-annotate entire schematic. Review needed before layout.
Parts:
- renumbered C1 to C10, R1 to R5, R2 to R6, U1 to U2
Changed lines of the file:
@@
 $EndDescr
 $Comp
-L power:GND #PWR05
+L power:GND #PWR016
 U 1 1 5DEC1237
 P 6400 4100
-F 0 "#PWR05" H 6400 3850 50  0001 C CNN
+F 0 "#PWR016" H 6400 3850 50  0001 C CNN
 F 1 "GND" H 6405 3927 50  0000 C CNN
 F 2 "" H 6400 4100 50  0001 C CNN
@@
 $EndComp
 $Comp
-L Device:C C1
+L Device:C C10
 U 1 1 5DEC14F2
 P 6400 3800
-F 0 "C1" H 6515 3846 50  0000 L CNN
+F 0 "C10" H 6515 3846 50  0000 L CNN
 F 1 "0.1u" H 6515 3755 50  0000 L CNN
 F 2 "Capacitor_SMD:C_0603_1608Metric" H 6438 3650 50  0001 C CNN
@@
 	6400 3300 6400 3650
 $Comp
-L power:+3.3V #PWR04
+L power:+3.3V #PWR015
 U 1 1 5DECB6BD
 P 6400 3300
-F 0 "#PWR04" H 6400 3150 50  0001 C CNN
+F 0 "#PWR015" H 6400 3150 50  0001 C CNN
 F 1 "+3.3V" H 6415 3473 50  0000 C CNN
 F 2 "" H 6400 3300 50  0001 C CNN
@@
 	4450 3800 4450 3700
 $Comp
-L Device:R_US R1
+L Device:R_US R5
 U 1 1 5DECC67C
 P 4450 3550
-F 0 "R1" H 4518 3596 50  0000 L CNN
+F 0 "R5" H 4518 3596 50  0000 L CNN
 F 1 "4.7k" H 4518 3505 50  0000 L CNN
 F 2 "Resistor_SMD:R_0603_1608Metric" V 4490 3540 50  0001 C CNN
@@
 $EndComp
 $Comp
-L power:+3.3V #PWR01
+L power:+3.3V #PWR014
 U 1 1 5DECCB19
 P 4450 3400
-F 0 "#PWR01" H 4450 3250 50  0001 C CNN
+F 0 "#PWR014" H 4450 3250 50  0001 C CNN
 F 1 "+3.3V" H 4465 3573 50  0000 C CNN
 F 2 "" H 4450 3400 50  0001 C CNN
@@
 Connection ~ 6400 3300
 $Comp
-L Sensor_Pressure:MS5607-02BA U1
+L Sensor_Pressure:MS5607-02BA U2
 U 1 1 5DEDE483
 P 5950 3700
-F 0 "U1" H 5900 4250 50  0000 L CNN
+F 0 "U2" H 5900 4250 50  0000 L CNN
 F 1 "MS5607-02BA" H 5700 4150 50  0000 L CNN
 F 2 "Package_LGA:LGA-8_3x5mm_P1.25mm" H 5950 3700 50  0001 C CNN
@@
 Connection ~ 4450 3400
 $Comp
-L Device:R_US R2
+L Device:R_US R6
 U 1 1 5DEE447F
 P 4800 3550
-F 0 "R2" H 4868 3596 50  0000 L CNN
+F 0 "R6" H 4868 3596 50  0000 L CNN
 F 1 "4.7k" H 4868 3505 50  0000 L CNN
 F 2 "Capacitor_SMD:C_0603_1608Metric" V 4840 3540 50  0001 C CNN

Commit message: Updated some footprints and re-annotated schematic.
Parts:
- renumbered C10 to C12, R5 to R6, R6 to R7
Changed lines of the file:
@@
 EESchema Schematic File Version 4
-LIBS:Recovery PCB-cache
-EELAYER 26 0
+EELAYER 30 0
 EELAYER END
 $Descr A4 11693 8268
@@
 $EndDescr
 $Comp
-L power:GND #PWR016
+L power:GND #PWR025
 U 1 1 5DEC1237
 P 6400 4100
-F 0 "#PWR016" H 6400 3850 50  0001 C CNN
+F 0 "#PWR025" H 6400 3850 50  0001 C CNN
 F 1 "GND" H 6405 3927 50  0000 C CNN
 F 2 "" H 6400 4100 50  0001 C CNN
@@
 $EndComp
 $Comp
-L Device:C C10
+L Device:C C12
 U 1 1 5DEC14F2
 P 6400 3800
-F 0 "C10" H 6515 3846 50  0000 L CNN
+F 0 "C12" H 6515 3846 50  0000 L CNN
 F 1 "0.1u" H 6515 3755 50  0000 L CNN
 F 2 "Capacitor_SMD:C_0603_1608Metric" H 6438 3650 50  0001 C CNN
@@
 	6400 3300 6400 3650
 $Comp
-L power:+3.3V #PWR015
+L power:+3.3V #PWR024
 U 1 1 5DECB6BD
 P 6400 3300
-F 0 "#PWR015" H 6400 3150 50  0001 C CNN
+F 0 "#PWR024" H 6400 3150 50  0001 C CNN
 F 1 "+3.3V" H 6415 3473 50  0000 C CNN
 F 2 "" H 6400 3300 50  0001 C CNN
@@
 	4450 3800 4450 3700
 $Comp
-L Device:R_US R5
+L Device:R_US R6
 U 1 1 5DECC67C
 P 4450 3550
-F 0 "R5" H 4518 3596 50  0000 L CNN
+F 0 "R6" H 4518 3596 50  0000 L CNN
 F 1 "4.7k" H 4518 3505 50  0000 L CNN
 F 2 "Resistor_SMD:R_0603_1608Metric" V 4490 3540 50  0001 C CNN
@@
 $EndComp
 $Comp
-L power:+3.3V #PWR014
+L power:+3.3V #PWR023
 U 1 1 5DECCB19
 P 4450 3400
-F 0 "#PWR014" H 4450 3250 50  0001 C CNN
+F 0 "#PWR023" H 4450 3250 50  0001 C CNN
 F 1 "+3.3V" H 4465 3573 50  0000 C CNN
 F 2 "" H 4450 3400 50  0001 C CNN
@@
 Connection ~ 4450 3400
 $Comp
-L Device:R_US R6
+L Device:R_US R7
 U 1 1 5DEE447F
 P 4800 3550
-F 0 "R6" H 4868 3596 50  0000 L CNN
+F 0 "R7" H 4868 3596 50  0000 L CNN
 F 1 "4.7k" H 4868 3505 50  0000 L CNN
 F 2 "Capacitor_SMD:C_0603_1608Metric" V 4840 3540 50  0001 C CNN

Commit message: Added missing footprints and replaced GPS module.
Parts:
- renumbered U2 to U3
Changed lines of the file:
@@
 Connection ~ 6400 3300
 $Comp
-L Sensor_Pressure:MS5607-02BA U2
+L Sensor_Pressure:MS5607-02BA U3
 U 1 1 5DEDE483
 P 5950 3700
-F 0 "U2" H 5900 4250 50  0000 L CNN
+F 0 "U3" H 5900 4250 50  0000 L CNN
 F 1 "MS5607-02BA" H 5700 4150 50  0000 L CNN
 F 2 "Package_LGA:LGA-8_3x5mm_P1.25mm" H 5950 3700 50  0001 C CNN

Commit message: Recovery PCB: Redraw schematics
Redrew Recover PCB schematics to be more easily readable and fixed board
outline, adding netclasses to ease trace placement.
Connections:
- net labels added: +3V3
- wire segments 14 -> 13
Changed lines of the file:
@@
 L power:GND #PWR025
 U 1 1 5DEC1237
-P 6400 4100
-F 0 "#PWR025" H 6400 3850 50  0001 C CNN
-F 1 "GND" H 6405 3927 50  0000 C CNN
-F 2 "" H 6400 4100 50  0001 C CNN
-F 3 "" H 6400 4100 50  0001 C CNN
-	1    6400 4100
+P 5950 4150
+F 0 "#PWR025" H 5950 3900 50  0001 C CNN
+F 1 "GND" H 5955 3977 50  0000 C CNN
+F 2 "" H 5950 4150 50  0001 C CNN
+F 3 "" H 5950 4150 50  0001 C CNN
+	1    5950 4150
 	1    0    0    -1
 $EndComp
@@
 L Device:C C12
 U 1 1 5DEC14F2
-P 6400 3800
-F 0 "C12" H 6515 3846 50  0000 L CNN
-F 1 "0.1u" H 6515 3755 50  0000 L CNN
-F 2 "Capacitor_SMD:C_0603_1608Metric" H 6438 3650 50  0001 C CNN
-F 3 "~" H 6400 3800 50  0001 C CNN
-	1    6400 3800
+P 6150 2950
+F 0 "C12" H 6265 2996 50  0000 L CNN
+F 1 "0.1u" H 6265 2905 50  0000 L CNN
+F 2 "Capacitor_SMD:C_0603_1608Metric" H 6188 2800 50  0001 C CNN
+F 3 "~" H 6150 2950 50  0001 C CNN
+	1    6150 2950
+	1    0    0    -1
+$EndComp
+$Comp
+L power:+3.3V #PWR024
+U 1 1 5DECB6BD
+P 5950 2800
+F 0 "#PWR024" H 5950 2650 50  0001 C CNN
+F 1 "+3.3V" H 5965 2973 50  0000 C CNN
+F 2 "" H 5950 2800 50  0001 C CNN
+F 3 "" H 5950 2800 50  0001 C CNN
+	1    5950 2800
+	1    0    0    -1
+$EndComp
+$Comp
+L Sensor_Pressure:MS5607-02BA U3
+U 1 1 5DEDE483
+P 5950 3700
+F 0 "U3" H 6100 3350 50  0000 L CNN
+F 1 "MS5607-02BA" H 6100 3250 50  0000 L CNN
+F 2 "Package_LGA:LGA-8_3x5mm_P1.25mm" H 5950 3700 50  0001 C CNN
+F 3 "https://www.te.com/commerce/DocumentDelivery/DDEController?Action=showdoc&DocId=Data+Sheet%7FMS5607-02BA03%7FB2%7Fpdf%7FEnglish%7FENG_DS_MS5607-02BA03_B2.pdf%7FCAT-BLPS0035" H 5950 3700 50  0001 C CNN
+	1    5950 3700
+	1    0    0    -1
+$EndComp
+NoConn ~ 5550 3600
+Wire Wire Line
+	5950 4100 5950 4150
+$Comp
+L power:GND #PWR0101
+U 1 1 6003E2FC
+P 5550 4150
+F 0 "#PWR0101" H 5550 3900 50  0001 C CNN
+F 1 "GND" H 5555 3977 50  0000 C CNN
+F 2 "" H 5550 4150 50  0001 C CNN
+F 3 "" H 5550 4150 50  0001 C CNN
+	1    5550 4150
 	1    0    0    -1
 $EndComp
 Wire Wire Line
-	5950 4100 6150 4100
-Wire Wire Line
-	5950 3300 6400 3300
-Wire Wire Line
-	6400 3300 6400 3650
+	5550 3900 5550 4150
 $Comp
-L power:+3.3V #PWR024
-U 1 1 5DECB6BD
-P 6400 3300
-F 0 "#PWR024" H 6400 3150 50  0001 C CNN
-F 1 "+3.3V" H 6415 3473 50  0000 C CNN
-F 2 "" H 6400 3300 50  0001 C CNN
-F 3 "" H 6400 3300 50  0001 C CNN
-	1    6400 3300
+L power:GND #PWR0102
+U 1 1 600415A4
+P 6150 3100
+F 0 "#PWR0102" H 6150 2850 50  0001 C CNN
+F 1 "GND" H 6155 2927 50  0000 C CNN
+F 2 "" H 6150 3100 50  0001 C CNN
+F 3 "" H 6150 3100 50  0001 C CNN
+	1    6150 3100
 	1    0    0    -1
 $EndComp
-Text HLabel 5200 3700 1    50   Input ~ 0
-SDA
 Wire Wire Line
-	4450 3800 4450 3700
+	5950 2800 5950 3300
+Wire Wire Line
+	5950 2800 6150 2800
+Connection ~ 5950 2800
+$Comp
+L power:+3V3 #PWR0103
+U 1 1 60043DAC
+P 5550 2800
+F 0 "#PWR0103" H 5550 2650 50  0001 C CNN
+F 1 "+3V3" H 5565 2973 50  0000 C CNN
+F 2 "" H 5550 2800 50  0001 C CNN
+F 3 "" H 5550 2800 50  0001 C CNN
+	1    5550 2800
+	1    0    0    -1
+$EndComp
+Wire Wire Line
+	5550 2800 5550 3500
 $Comp
 L Device:R_US R6
 U 1 1 5DECC67C
-P 4450 3550
-F 0 "R6" H 4518 3596 50  0000 L CNN
-F 1 "4.7k" H 4518 3505 50  0000 L CNN
-F 2 "Resistor_SMD:R_0603_1608Metric" V 4490 3540 50  0001 C CNN
-F 3 "~" H 4450 3550 50  0001 C CNN
-	1    4450 3550
+P 4850 3400
+F 0 "R6" H 4918 3446 50  0000 L CNN
+F 1 "4.7k" H 4918 3355 50  0000 L CNN
+F 2 "Resistor_SMD:R_0603_1608Metric" V 4890 3390 50  0001 C CNN
+F 3 "~" H 4850 3400 50  0001 C CNN
+	1    4850 3400
 	1    0    0    -1
 $EndComp
@@
 L power:+3.3V #PWR023
 U 1 1 5DECCB19
-P 4450 3400
-F 0 "#PWR023" H 4450 3250 50  0001 C CNN
-F 1 "+3.3V" H 4465 3573 50  0000 C CNN
-F 2 "" H 4450 3400 50  0001 C CNN
-F 3 "" H 4450 3400 50  0001 C CNN
-	1    4450 3400
+P 4850 3200
+F 0 "#PWR023" H 4850 3050 50  0001 C CNN
+F 1 "+3.3V" H 4865 3373 50  0000 C CNN
+F 2 "" H 4850 3200 50  0001 C CNN
+F 3 "" H 4850 3200 50  0001 C CNN
+	1    4850 3200
 	1    0    0    -1
 $EndComp
-Text HLabel 5200 3800 3    50   Input ~ 0
-SCL
-Connection ~ 6400 3300
-$Comp
-L Sensor_Pressure:MS5607-02BA U3
-U 1 1 5DEDE483
-P 5950 3700
-F 0 "U3" H 5900 4250 50  0000 L CNN
-F 1 "MS5607-02BA" H 5700 4150 50  0000 L CNN
-F 2 "Package_LGA:LGA-8_3x5mm_P1.25mm" H 5950 3700 50  0001 C CNN
-F 3 "https://www.te.com/commerce/DocumentDelivery/DDEController?Action=showdoc&DocId=Data+Sheet%7FMS5607-02BA03%7FB2%7Fpdf%7FEnglish%7FENG_DS_MS5607-02BA03_B2.pdf%7FCAT-BLPS0035" H 5950 3700 50  0001 C CNN
-	1    5950 3700
-	1    0    0    -1
-$EndComp
-Connection ~ 4450 3400
 $Comp
 L Device:R_US R7
 U 1 1 5DEE447F
-P 4800 3550
-F 0 "R7" H 4868 3596 50  0000 L CNN
-F 1 "4.7k" H 4868 3505 50  0000 L CNN
-F 2 "Capacitor_SMD:C_0603_1608Metric" V 4840 3540 50  0001 C CNN
-F 3 "~" H 4800 3550 50  0001 C CNN
-	1    4800 3550
+P 5200 3400
+F 0 "R7" H 5268 3446 50  0000 L CNN
+F 1 "4.7k" H 5268 3355 50  0000 L CNN
+F 2 "Capacitor_SMD:C_0603_1608Metric" V 5240 3390 50  0001 C CNN
+F 3 "~" H 5200 3400 50  0001 C CNN
+	1    5200 3400
 	1    0    0    -1
 $EndComp
+$Comp
+L power:+3.3V #PWR0104
+U 1 1 60046089
+P 5200 3200
+F 0 "#PWR0104" H 5200 3050 50  0001 C CNN
+F 1 "+3.3V" H 5215 3373 50  0000 C CNN
+F 2 "" H 5200 3200 50  0001 C CNN
+F 3 "" H 5200 3200 50  0001 C CNN
+	1    5200 3200
+	1    0    0    -1
+$EndComp
+Text HLabel 4600 3700 0    50   Input ~ 0
+SDA
+Text HLabel 4600 3800 0    50   Input ~ 0
+SCL
 Wire Wire Line
-	4450 3400 4800 3400
+	4600 3700 5200 3700
 Wire Wire Line
-	4800 3700 5550 3700
+	5200 3550 5200 3700
+Connection ~ 5200 3700
 Wire Wire Line
-	4450 3800 5550 3800
+	5200 3700 5550 3700
 Wire Wire Line
-	6400 3950 6400 4100
-Connection ~ 6400 4100
+	4850 3550 4850 3800
 Wire Wire Line
-	5550 3900 5550 4200
+	4850 3800 4600 3800
 Wire Wire Line
-	5550 4200 6150 4200
+	4850 3800 5550 3800
+Connection ~ 4850 3800
 Wire Wire Line
-	6150 4200 6150 4100
-Connection ~ 6150 4100
+	4850 3200 4850 3250
 Wire Wire Line
-	6150 4100 6400 4100
-NoConn ~ 5550 3600
-Wire Wire Line
-	5550 3500 5550 3300
-Wire Wire Line
-	5550 3300 5950 3300
-Connection ~ 5950 3300
+	5200 3200 5200 3250
 $EndSCHEMATC

Commit message: Recovery PCB: Reannotate
Reannotated schematic to fix reference numbering and keep reference
designators consistent.
Parts:
- renumbered C12 to C13, R6 to R5, R7 to R6
Changed lines of the file:
@@
 $EndDescr
 $Comp
-L power:GND #PWR025
+L power:GND #PWR034
 U 1 1 5DEC1237
 P 5950 4150
-F 0 "#PWR025" H 5950 3900 50  0001 C CNN
+F 0 "#PWR034" H 5950 3900 50  0001 C CNN
 F 1 "GND" H 5955 3977 50  0000 C CNN
 F 2 "" H 5950 4150 50  0001 C CNN
@@
 $EndComp
 $Comp
-L Device:C C12
+L Device:C C13
 U 1 1 5DEC14F2
 P 6150 2950
-F 0 "C12" H 6265 2996 50  0000 L CNN
+F 0 "C13" H 6265 2996 50  0000 L CNN
 F 1 "0.1u" H 6265 2905 50  0000 L CNN
 F 2 "Capacitor_SMD:C_0603_1608Metric" H 6188 2800 50  0001 C CNN
@@
 $EndComp
 $Comp
-L power:+3.3V #PWR024
+L power:+3.3V #PWR029
 U 1 1 5DECB6BD
 P 5950 2800
-F 0 "#PWR024" H 5950 2650 50  0001 C CNN
+F 0 "#PWR029" H 5950 2650 50  0001 C CNN
 F 1 "+3.3V" H 5965 2973 50  0000 C CNN
 F 2 "" H 5950 2800 50  0001 C CNN
@@
 	5950 4100 5950 4150
 $Comp
-L power:GND #PWR0101
+L power:GND #PWR033
 U 1 1 6003E2FC
 P 5550 4150
-F 0 "#PWR0101" H 5550 3900 50  0001 C CNN
+F 0 "#PWR033" H 5550 3900 50  0001 C CNN
 F 1 "GND" H 5555 3977 50  0000 C CNN
 F 2 "" H 5550 4150 50  0001 C CNN
@@
 	5550 3900 5550 4150
 $Comp
-L power:GND #PWR0102
+L power:GND #PWR030
 U 1 1 600415A4
 P 6150 3100
-F 0 "#PWR0102" H 6150 2850 50  0001 C CNN
+F 0 "#PWR030" H 6150 2850 50  0001 C CNN
 F 1 "GND" H 6155 2927 50  0000 C CNN
 F 2 "" H 6150 3100 50  0001 C CNN
@@
 Connection ~ 5950 2800
 $Comp
-L power:+3V3 #PWR0103
+L power:+3V3 #PWR028
 U 1 1 60043DAC
 P 5550 2800
-F 0 "#PWR0103" H 5550 2650 50  0001 C CNN
+F 0 "#PWR028" H 5550 2650 50  0001 C CNN
 F 1 "+3V3" H 5565 2973 50  0000 C CNN
 F 2 "" H 5550 2800 50  0001 C CNN
@@
 	5550 2800 5550 3500
 $Comp
-L Device:R_US R6
+L Device:R_US R5
 U 1 1 5DECC67C
 P 4850 3400
-F 0 "R6" H 4918 3446 50  0000 L CNN
+F 0 "R5" H 4918 3446 50  0000 L CNN
 F 1 "4.7k" H 4918 3355 50  0000 L CNN
 F 2 "Resistor_SMD:R_0603_1608Metric" V 4890 3390 50  0001 C CNN
@@
 $EndComp
 $Comp
-L power:+3.3V #PWR023
+L power:+3.3V #PWR031
 U 1 1 5DECCB19
 P 4850 3200
-F 0 "#PWR023" H 4850 3050 50  0001 C CNN
+F 0 "#PWR031" H 4850 3050 50  0001 C CNN
 F 1 "+3.3V" H 4865 3373 50  0000 C CNN
 F 2 "" H 4850 3200 50  0001 C CNN
@@
 $EndComp
 $Comp
-L Device:R_US R7
+L Device:R_US R6
 U 1 1 5DEE447F
 P 5200 3400
-F 0 "R7" H 5268 3446 50  0000 L CNN
+F 0 "R6" H 5268 3446 50  0000 L CNN
 F 1 "4.7k" H 5268 3355 50  0000 L CNN
 F 2 "Capacitor_SMD:C_0603_1608Metric" V 5240 3390 50  0001 C CNN
@@
 $EndComp
 $Comp
-L power:+3.3V #PWR0104
+L power:+3.3V #PWR032
 U 1 1 60046089
 P 5200 3200
-F 0 "#PWR0104" H 5200 3050 50  0001 C CNN
+F 0 "#PWR032" H 5200 3050 50  0001 C CNN
 F 1 "+3.3V" H 5215 3373 50  0000 C CNN
 F 2 "" H 5200 3200 50  0001 C CNN

Commit message: Recovery PCB: Fix relay
Replaced unavailable relay with a correct part and replaced voltage
regulator with an easier to solder alternative.
Changed lines of the file:
@@
 	1    0    0    -1
 $EndComp
-Text HLabel 4600 3700 0    50   Input ~ 0
+Text HLabel 4600 3700 0    50   BiDi ~ 0
 SDA
 Text HLabel 4600 3800 0    50   Input ~ 0
