File: Recovery PCB/PressureSensor.sch (KiCad schematic (older format))
At the start: 4 parts, among them U3 MS5607-02BA

Commit message: Recovery PCB: Minor changes to layout.
Parts:
- R6: footprint Capacitor_SMD:C_0603_1608Metric -> Resistor_SMD:R_0603_1608Metric
Changed lines of the file:
@@
 F 0 "R6" H 5268 3446 50  0000 L CNN
 F 1 "4.7k" H 5268 3355 50  0000 L CNN
-F 2 "Capacitor_SMD:C_0603_1608Metric" V 5240 3390 50  0001 C CNN
+F 2 "Resistor_SMD:R_0603_1608Metric" V 5240 3390 50  0001 C CNN
 F 3 "~" H 5200 3400 50  0001 C CNN
 	1    5200 3400
