File: Recovery PCB/microSD.sch (KiCad schematic (older format))
At the start: 3 parts, among them J5 MEM2075-00-140-01-A, J6 Conn_01x07_Male

Commit message: Update relays and re-annotate entire schematic. Review needed before layout.
Parts:
- renumbered R11 to R9
Changed lines of the file:
@@
 	7350 3900 7350 4000
 $Comp
-L power:GND #PWR026
+L power:GND #PWR032
 U 1 1 5DF52C47
 P 7350 4000
-F 0 "#PWR026" H 7350 3750 50  0001 C CNN
+F 0 "#PWR032" H 7350 3750 50  0001 C CNN
 F 1 "GND" H 7355 3827 50  0000 C CNN
 F 2 "" H 7350 4000 50  0001 C CNN
@@
 Connection ~ 3200 4150
 $Comp
-L power:GND #PWR022
+L power:GND #PWR030
 U 1 1 5DF793E4
 P 3200 4250
-F 0 "#PWR022" H 3200 4000 50  0001 C CNN
+F 0 "#PWR030" H 3200 4000 50  0001 C CNN
 F 1 "GND" H 3205 4077 50  0000 C CNN
 F 2 "" H 3200 4250 50  0001 C CNN
@@
 	3250 3550 3150 3550
 $Comp
-L power:+3.3V #PWR021
+L power:+3.3V #PWR029
 U 1 1 5DF7A4AA
 P 3150 2900
-F 0 "#PWR021" H 3150 2750 50  0001 C CNN
+F 0 "#PWR029" H 3150 2750 50  0001 C CNN
 F 1 "+3.3V" H 3165 3073 50  0000 C CNN
 F 2 "" H 3150 2900 50  0001 C CNN
@@
 	4700 3650 4700 3450
 $Comp
-L Device:R_US R11
+L Device:R_US R9
 U 1 1 5DF951A8
 P 5150 3100
-F 0 "R11" H 5218 3146 50  0000 L CNN
+F 0 "R9" H 5218 3146 50  0000 L CNN
 F 1 "100k" H 5218 3055 50  0000 L CNN
 F 2 "Resistor_SMD:R_0603_1608Metric" V 5190 3090 50  0001 C CNN
@@
 $EndComp
 $Comp
-L power:+3.3V #PWR?
+L power:+3.3V #PWR031
 U 1 1 5E3F408D
 P 7350 3200
-F 0 "#PWR?" H 7350 3050 50  0001 C CNN
+F 0 "#PWR031" H 7350 3050 50  0001 C CNN
 F 1 "+3.3V" H 7365 3373 50  0000 C CNN
 F 2 "" H 7350 3200 50  0001 C CNN

Commit message: Added footprints.
Added footprints for various parts. Still need to update some more and calculate some values.
Parts:
- removed J6: Conn_01x07_Male, symbol Connector:Conn_01x07_Male
- renumbered R9 to R11
Connections:
- wire segments 38 -> 13
Changed lines of the file:
@@
 Comment4 ""
 $EndDescr
-$Comp
-L Connector:Conn_01x07_Male J6
-U 1 1 5DF4BC1A
-P 7650 3600
-F 0 "J6" H 7622 3624 50  0000 R CNN
-F 1 "Conn_01x07_Male" H 7622 3533 50  0000 R CNN
-F 2 "" H 7650 3600 50  0001 C CNN
-F 3 "~" H 7650 3600 50  0001 C CNN
-	1    7650 3600
-	-1   0    0    -1
-$EndComp
-Wire Wire Line
-	7450 3300 7350 3300
-Wire Wire Line
-	7350 3300 7350 3200
-Wire Wire Line
-	7450 3900 7350 3900
-Wire Wire Line
-	7350 3900 7350 4000
-$Comp
-L power:GND #PWR032
-U 1 1 5DF52C47
-P 7350 4000
-F 0 "#PWR032" H 7350 3750 50  0001 C CNN
-F 1 "GND" H 7355 3827 50  0000 C CNN
-F 2 "" H 7350 4000 50  0001 C CNN
-F 3 "" H 7350 4000 50  0001 C CNN
-	1    7350 4000
-	1    0    0    -1
-$EndComp
-Text HLabel 7200 3800 3    50   Input ~ 0
-SD_CS
-Wire Wire Line
-	7450 3500 6450 3500
-Wire Wire Line
-	6450 3500 6450 3450
-Wire Wire Line
-	7450 3600 6450 3600
-Wire Wire Line
-	6450 3600 6450 3650
-Wire Wire Line
-	7450 3400 6500 3400
-Wire Wire Line
-	6500 3400 6500 3250
-Wire Wire Line
-	7450 3700 6500 3700
-Wire Wire Line
-	6500 3700 6500 3850
 Wire Wire Line
 	3250 4050 3200 4050
@@
 Connection ~ 3200 4150
 $Comp
-L power:GND #PWR030
+L power:GND #PWR036
 U 1 1 5DF793E4
 P 3200 4250
-F 0 "#PWR030" H 3200 4000 50  0001 C CNN
+F 0 "#PWR036" H 3200 4000 50  0001 C CNN
 F 1 "GND" H 3205 4077 50  0000 C CNN
 F 2 "" H 3200 4250 50  0001 C CNN
@@
 	3250 3550 3150 3550
 $Comp
-L power:+3.3V #PWR029
+L power:+3.3V #PWR035
 U 1 1 5DF7A4AA
 P 3150 2900
-F 0 "#PWR029" H 3150 2750 50  0001 C CNN
+F 0 "#PWR035" H 3150 2750 50  0001 C CNN
 F 1 "+3.3V" H 3165 3073 50  0000 C CNN
 F 2 "" H 3150 2900 50  0001 C CNN
@@
 NoConn ~ 4650 3950
 NoConn ~ 4650 4050
-Wire Wire Line
-	4750 3650 4750 3550
-Wire Wire Line
-	4750 3550 4650 3550
-Wire Wire Line
-	4650 3650 4700 3650
-Wire Wire Line
-	4700 3650 4700 3450
 $Comp
-L Device:R_US R9
+L Device:R_US R11
 U 1 1 5DF951A8
 P 5150 3100
-F 0 "R9" H 5218 3146 50  0000 L CNN
+F 0 "R11" H 5218 3146 50  0000 L CNN
 F 1 "100k" H 5218 3055 50  0000 L CNN
 F 2 "Resistor_SMD:R_0603_1608Metric" V 5190 3090 50  0001 C CNN
@@
 	3150 2950 3150 2900
 Connection ~ 3150 2950
-Wire Wire Line
-	5150 3250 5000 3250
-Wire Wire Line
-	5000 3250 5000 4150
-Wire Wire Line
-	5000 4150 4650 4150
-Connection ~ 5150 3250
 $Comp
 L MEM2075-00-140-01-A:MEM2075-00-140-01-A J5
@@
 	-1   0    0    -1
 $EndComp
-$Comp
-L power:+3.3V #PWR031
-U 1 1 5E3F408D
-P 7350 3200
-F 0 "#PWR031" H 7350 3050 50  0001 C CNN
-F 1 "+3.3V" H 7365 3373 50  0000 C CNN
-F 2 "" H 7350 3200 50  0001 C CNN
-F 3 "" H 7350 3200 50  0001 C CNN
-	1    7350 3200
-	1    0    0    -1
-$EndComp
+Text HLabel 4750 3550 2    50   Input ~ 0
+SD_CLK
+Text HLabel 4750 3650 2    50   Input ~ 0
+SD_DI
+Text HLabel 4750 3850 2    50   Input ~ 0
+SD_DO
+Text HLabel 3250 3850 0    50   Input ~ 0
+SD_CS
 Wire Wire Line
-	5150 3250 6500 3250
+	4650 3550 4750 3550
 Wire Wire Line
-	4700 3450 6250 3450
+	4650 3650 4750 3650
 Wire Wire Line
-	4750 3650 6250 3650
+	4650 3850 4750 3850
 Wire Wire Line
-	4650 3850 6250 3850
+	5150 3250 5150 4150
 Wire Wire Line
-	7450 3800 7050 3800
-Text Label 7050 3800 2    50   ~ 0
-SD_CS
-Text Label 3250 3850 2    50   ~ 0
-SD_CS
-Text HLabel 6250 3700 0    50   Input ~ 0
-SD_CLK
-Wire Wire Line
-	6250 3700 6250 3650
-Connection ~ 6250 3650
-Wire Wire Line
-	6250 3650 6450 3650
-Text HLabel 6250 3500 0    50   Input ~ 0
-SD_DI
-Wire Wire Line
-	6250 3500 6250 3450
-Connection ~ 6250 3450
-Wire Wire Line
-	6250 3450 6450 3450
-Text HLabel 6250 3900 0    50   Input ~ 0
-SD_DO
-Wire Wire Line
-	6250 3900 6250 3850
-Connection ~ 6250 3850
-Wire Wire Line
-	6250 3850 6500 3850
+	4650 4150 5150 4150
 $EndSCHEMATC

Commit message: Updated some footprints and re-annotated schematic.
Parts:
- renumbered J5 to J6, R11 to R12
Changed lines of the file:
@@
 EESchema Schematic File Version 4
-LIBS:Recovery PCB-cache
-EELAYER 26 0
+EELAYER 30 0
 EELAYER END
 $Descr A4 11693 8268
@@
 Connection ~ 3200 4150
 $Comp
-L power:GND #PWR036
+L power:GND #PWR045
 U 1 1 5DF793E4
 P 3200 4250
-F 0 "#PWR036" H 3200 4000 50  0001 C CNN
+F 0 "#PWR045" H 3200 4000 50  0001 C CNN
 F 1 "GND" H 3205 4077 50  0000 C CNN
 F 2 "" H 3200 4250 50  0001 C CNN
@@
 	3250 3550 3150 3550
 $Comp
-L power:+3.3V #PWR035
+L power:+3.3V #PWR044
 U 1 1 5DF7A4AA
 P 3150 2900
-F 0 "#PWR035" H 3150 2750 50  0001 C CNN
+F 0 "#PWR044" H 3150 2750 50  0001 C CNN
 F 1 "+3.3V" H 3165 3073 50  0000 C CNN
 F 2 "" H 3150 2900 50  0001 C CNN
@@
 NoConn ~ 4650 4050
 $Comp
-L Device:R_US R11
+L Device:R_US R12
 U 1 1 5DF951A8
 P 5150 3100
-F 0 "R11" H 5218 3146 50  0000 L CNN
+F 0 "R12" H 5218 3146 50  0000 L CNN
 F 1 "100k" H 5218 3055 50  0000 L CNN
 F 2 "Resistor_SMD:R_0603_1608Metric" V 5190 3090 50  0001 C CNN
@@
 Connection ~ 3150 2950
 $Comp
-L MEM2075-00-140-01-A:MEM2075-00-140-01-A J5
+L MEM2075-00-140-01-A:MEM2075-00-140-01-A J6
 U 1 1 5DF6E6EE
 P 3950 3850
-F 0 "J5" H 3950 4417 50  0000 C CNN
+F 0 "J6" H 3950 4417 50  0000 C CNN
 F 1 "MEM2075-00-140-01-A" H 3950 4326 50  0000 C CNN
 F 2 "GCT_MEM2075-00-140-01-A" H 3950 3850 50  0001 L BNN

Commit message: Recovery PCB: Redraw schematics
Redrew Recover PCB schematics to be more easily readable and fixed board
outline, adding netclasses to ease trace placement.
Connections:
- net labels added: +3V3
- wire segments 13 -> 10
Changed lines of the file:
@@
 $EndComp
 Wire Wire Line
-	3250 3550 3150 3550
+	3250 3550 3200 3550
 $Comp
 L power:+3.3V #PWR044
 U 1 1 5DF7A4AA
-P 3150 2900
-F 0 "#PWR044" H 3150 2750 50  0001 C CNN
-F 1 "+3.3V" H 3165 3073 50  0000 C CNN
-F 2 "" H 3150 2900 50  0001 C CNN
-F 3 "" H 3150 2900 50  0001 C CNN
-	1    3150 2900
+P 3200 3450
+F 0 "#PWR044" H 3200 3300 50  0001 C CNN
+F 1 "+3.3V" H 3215 3623 50  0000 C CNN
+F 2 "" H 3200 3450 50  0001 C CNN
+F 3 "" H 3200 3450 50  0001 C CNN
+	1    3200 3450
 	1    0    0    -1
 $EndComp
@@
 L Device:R_US R12
 U 1 1 5DF951A8
-P 5150 3100
-F 0 "R12" H 5218 3146 50  0000 L CNN
-F 1 "100k" H 5218 3055 50  0000 L CNN
-F 2 "Resistor_SMD:R_0603_1608Metric" V 5190 3090 50  0001 C CNN
-F 3 "~" H 5150 3100 50  0001 C CNN
-	1    5150 3100
+P 5150 4000
+F 0 "R12" H 5218 4046 50  0000 L CNN
+F 1 "100k" H 5218 3955 50  0000 L CNN
+F 2 "Resistor_SMD:R_0603_1608Metric" V 5190 3990 50  0001 C CNN
+F 3 "~" H 5150 4000 50  0001 C CNN
+	1    5150 4000
 	1    0    0    -1
 $EndComp
-Wire Wire Line
-	5150 2950 3150 2950
-Wire Wire Line
-	3150 2950 3150 3550
-Wire Wire Line
-	3150 2950 3150 2900
-Connection ~ 3150 2950
 $Comp
 L MEM2075-00-140-01-A:MEM2075-00-140-01-A J6
@@
 	4650 3850 4750 3850
 Wire Wire Line
-	5150 3250 5150 4150
+	4650 4150 5150 4150
+$Comp
+L power:+3V3 #PWR0125
+U 1 1 60396F84
+P 5150 3850
+F 0 "#PWR0125" H 5150 3700 50  0001 C CNN
+F 1 "+3V3" H 5165 4023 50  0000 C CNN
+F 2 "" H 5150 3850 50  0001 C CNN
+F 3 "" H 5150 3850 50  0001 C CNN
+	1    5150 3850
+	1    0    0    -1
+$EndComp
 Wire Wire Line
-	4650 4150 5150 4150
+	3200 3450 3200 3550
 $EndSCHEMATC

Commit message: Recovery PCB: Reannotate
Reannotated schematic to fix reference numbering and keep reference
designators consistent.
Parts:
- renumbered J6 to J7, R12 to R13
Changed lines of the file:
@@
 Connection ~ 3200 4150
 $Comp
-L power:GND #PWR045
+L power:GND #PWR056
 U 1 1 5DF793E4
 P 3200 4250
-F 0 "#PWR045" H 3200 4000 50  0001 C CNN
+F 0 "#PWR056" H 3200 4000 50  0001 C CNN
 F 1 "GND" H 3205 4077 50  0000 C CNN
 F 2 "" H 3200 4250 50  0001 C CNN
@@
 	3250 3550 3200 3550
 $Comp
-L power:+3.3V #PWR044
+L power:+3.3V #PWR054
 U 1 1 5DF7A4AA
 P 3200 3450
-F 0 "#PWR044" H 3200 3300 50  0001 C CNN
+F 0 "#PWR054" H 3200 3300 50  0001 C CNN
 F 1 "+3.3V" H 3215 3623 50  0000 C CNN
 F 2 "" H 3200 3450 50  0001 C CNN
@@
 NoConn ~ 4650 4050
 $Comp
-L Device:R_US R12
+L Device:R_US R13
 U 1 1 5DF951A8
 P 5150 4000
-F 0 "R12" H 5218 4046 50  0000 L CNN
+F 0 "R13" H 5218 4046 50  0000 L CNN
 F 1 "100k" H 5218 3955 50  0000 L CNN
 F 2 "Resistor_SMD:R_0603_1608Metric" V 5190 3990 50  0001 C CNN
@@
 $EndComp
 $Comp
-L MEM2075-00-140-01-A:MEM2075-00-140-01-A J6
+L MEM2075-00-140-01-A:MEM2075-00-140-01-A J7
 U 1 1 5DF6E6EE
 P 3950 3850
-F 0 "J6" H 3950 4417 50  0000 C CNN
+F 0 "J7" H 3950 4417 50  0000 C CNN
 F 1 "MEM2075-00-140-01-A" H 3950 4326 50  0000 C CNN
 F 2 "GCT_MEM2075-00-140-01-A" H 3950 3850 50  0001 L BNN
@@
 	4650 4150 5150 4150
 $Comp
-L power:+3V3 #PWR0125
+L power:+3V3 #PWR055
 U 1 1 60396F84
 P 5150 3850
-F 0 "#PWR0125" H 5150 3700 50  0001 C CNN
+F 0 "#PWR055" H 5150 3700 50  0001 C CNN
 F 1 "+3V3" H 5165 4023 50  0000 C CNN
 F 2 "" H 5150 3850 50  0001 C CNN
